File: 7-seg-clock/7-seg-clock.kicad_sch (KiCad schematic)
At the start: 30 parts, among them J1 USB_C_Receptacle_USB2.0_16P, J2 JWT, SW1 BOOT_MD, SW2 RST, U1 LD1117S33TR_SOT223, U10 HDSP-7501, U11 HDSP-7501, U12 MAX7221xWG, U2 APDS-9960, U3 FT232RL, U4 STM32C071C8Tx, U5 HDSP-7501, U6 HDSP-7501, U7 WIZFI360-PA, U8 HDSP-7501, U9 HDSP-7501

Commit message: Better library
Parts:
- removed C1, C2, C3, C4: 1 uF, Capacitor_SMD:C_1206_3216Metric, symbol Device:C_Small
- removed C5: 10 uF, Capacitor_SMD:C_1206_3216Metric, symbol Device:C_Small
- removed D1: SD05_SOD323, Diode_SMD:D_SOD-323, symbol Diode:SD05_SOD323
- removed D2: ZEN065V130A24LS, Diode_SMD:Littelfuse_PolyZen-LS, symbol Power_Protection:ZEN065V130A24LS
- removed J1: USB_C_Receptacle_USB2.0_16P, Connector_USB:USB_C_Receptacle_HRO_TYPE-C-31-M-12, symbol Connector:USB_C_Receptacle_USB2.0_16P
- removed J2: JWT, Connector_PinHeader_2.54mm:PinHeader_1x03_P2.54mm_Vertical, symbol Connector:Conn_01x03_Pin
- removed R2: 5.1k, Resistor_SMD:R_1206_3216Metric, symbol Device:R_Small
- removed SW1: BOOT_MD, Button_Switch_SMD:SW_SPDT_PCM12, symbol Switch:SW_SPDT
- removed SW2: RST, Button_Switch_THT:SW_PUSH_6mm, symbol Switch:SW_Push
- removed U1: LD1117S33TR_SOT223, Package_TO_SOT_SMD:SOT-223-3_TabPin2, symbol Regulator_Linear:LD1117S33TR_SOT223
- removed U3: FT232RL, Package_SO:SSOP-28_5.3x10.2mm_P0.65mm, symbol Interface_USB:FT232RL
- removed U4: STM32C071C8Tx, Package_QFP:LQFP-48_7x7mm_P0.5mm, symbol MCU_ST_STM32C0:STM32C071C8Tx
- removed U7: WIZFI360-PA, WIZFI360-PA:XCVR_WIZFI360-PA, symbol WIZFI360-PA:WIZFI360-PA
- added C12: 22 uF, Capacitor_SMD:C_0805_2012Metric, symbol Device:C_Small
- added C2: 100nF, Capacitor_SMD:C_0805_2012Metric, symbol Device:C
- added D12: 3.3V LED, LED_SMD:LED_0805_2012Metric, symbol Device:LED
- added D4: 5V LED, LED_SMD:LED_0805_2012Metric, symbol Device:LED
- added F1: 500 mA, Fuse:Fuse_1206_3216Metric, symbol Device:Polyfuse
- added J1: USB_C_Receptacle_USB2.0, Connector_USB:USB_C_Receptacle_HRO_TYPE-C-31-M-12, symbol Connector:USB_C_Receptacle_USB2.0
- added J3: Conn_01x12_Pin, Connector_PinHeader_2.54mm:PinHeader_1x12_P2.54mm_Vertical, symbol Connector:Conn_01x12_Pin
- added J4: Conn_01x01_Pin, Connector_PinHeader_2.54mm:PinHeader_1x01_P2.54mm_Vertical, symbol Connector:Conn_01x01_Pin
- added J5, J6, J8: Conn_01x02_Pin, Connector_PinHeader_2.54mm:PinHeader_1x02_P2.54mm_Vertical, symbol Connector:Conn_01x02_Pin
- added J7: Conn_01x06_Pin, Connector_PinHeader_2.54mm:PinHeader_1x06_P2.54mm_Vertical, symbol Connector:Conn_01x06_Pin
- added L1: 2.2 uH, footprints:IND_PA4332.222NLT, symbol Device:L
- added R11: 100k, Resistor_SMD:R_0805_2012Metric, symbol Device:R_Small
- added R12: 562kΩ, Resistor_SMD:R_0805_2012Metric, symbol Device:R_Small
- added R13: 180kΩ, Resistor_SMD:R_0805_2012Metric, symbol Device:R_Small
- added R20: 150, Resistor_SMD:R_0805_2012Metric, symbol Device:R
- added R21: 330, Resistor_SMD:R_0805_2012Metric, symbol Device:R
- added R5: 10k, Resistor_SMD:R_0805_2012Metric, symbol Device:R_Small
- added R6, R7: 5.1k, Resistor_SMD:R_0805_2012Metric, symbol Device:R
- added R8, R9: 22, Resistor_SMD:R_0805_2012Metric, symbol Device:R
- added SW2: EN, footprints:KH-6X6X5H-STM_SKE, symbol 2026-02-17_13-05-37:KH-6X6X5H-STM
- added SW3: SLW-66527511-SMT-TR, footprints:SLW-66527511-SMT-TR_CUD, symbol 2026-02-17_12-53-48:SLW-66527511-SMT-TR
- added U1: ESP32-S3-MINI-1, RF_Module:ESP32-S2-MINI-1, symbol RF_Module:ESP32-S3-MINI-1
- added U3: PRTR5V0U2X, Package_TO_SOT_SMD:SOT-143, symbol Power_Protection:PRTR5V0U2X
- added U4: TPS62160DSG, Package_SON:WSON-8-1EP_2x2mm_P0.5mm_EP0.9x1.6mm_ThermalVias, symbol Regulator_Switching:TPS62160DSG
- C7: footprint Capacitor_SMD:C_1206_3216Metric -> Capacitor_SMD:C_0805_2012Metric; LCSC Part # (none) -> C15850
- R1: value 5.1k -> 10k; footprint Resistor_SMD:R_1206_3216Metric -> Resistor_SMD:R_0805_2012Metric; LCSC Part # (none) -> C17414
Connections:
- net +3.3V: now also C12.1, L1.2, R11.1, R12.1, R5.2, U4.6 (VOS); no longer C7.1
- net +5V: now also C7.1, C2.1, F1.2, R21.2, U3.4 (VCC), U4.2 (VIN), U4.3 (EN)
- net D+: now also R9.2, U1.24 (USB_D+), U3.3 (I/O2)
- net D-: now also R8.2, U1.23 (USB_D-), U3.2 (I/O1)
- net GND: now also C12.2, C2.2, D12.2 (A), D4.2 (A), R13.2, R6.1, R7.2, SW2.C, SW3.3, U1.1 (GND), U1.2 (GND), U1.42 (GND), U1.43 (GND), U1.44 (IO46), U1.46 (GND), U1.47 (GND), U1.48 (GND), U1.49 (GND), U1.50 (GND), U1.51 (GND), U1.52 (GND), U1.53 (GND), U1.54 (GND), U1.55 (GND), U1.56 (GND), U1.57 (GND), U1.58 (GND), U1.59 (GND), U1.60 (GND), U1.61 (GND), U1.62 (GND), U1.63 (GND), U1.64 (GND), U1.65 (GND), U3.1 (GND), U4.1 (PGND), U4.4 (AGND), U4.9 (PAD); no longer R1.2
- net SPI1_MOSI: now also U1.11 (IO7)
- net VBUS: now also F1.1, J1.A4 (VBUS), J1.A9 (VBUS), J1.B4 (VBUS), J1.B9 (VBUS)
- net +3V3: now reaches R1.1
- net +3V3: now also R20.2, SW3.1, U1.3 (3V3)
- net SPI1_MISO: now reaches U12.24 (DOUT)
- net SPI1_MISO: now also U1.6 (IO2)
- net SCL renamed I2C1_SCL
- net I2C1_SCL: now also U1.21 (IO17)
- net SDA renamed I2C1_SDA
- net I2C1_SDA: now also U1.22 (IO18)
- net SPI1_NSS renamed SPI1_CS
- net SPI1_CS: now also U1.14 (IO10)
- net SPI1_SCK renamed SPI1_CLK
- net SPI1_CLK: now also U1.10 (IO6)
- new net: D12.1 (K), R20.1
- new net: R1.2, SW2.B, U1.45 (EN)
- new net: J1.A1 (GND), J1.A12 (GND), J1.B1 (GND), J1.B12 (GND), J1.S1 (SHIELD)
- new net: J1.A5 (CC1), R6.2
- new net: J1.A6 (D+), J1.B6 (D+), R9.1
- new net: J1.A7 (D-), J1.B7 (D-), R8.1
- new net: J1.B5 (CC2), R7.1
- new net: D4.1 (K), R21.1
- new net: R12.2, R13.1, U4.5 (FB)
- new net: J4.1 (Pin_1), U1.5 (IO1)
- new net: J7.1 (Pin_1), U1.15 (IO11)
- new net: J7.2 (Pin_2), U1.16 (IO12)
- new net: J7.3 (Pin_3), U1.17 (IO13)
- new net: J7.4 (Pin_4), U1.18 (IO14)
- new net: J7.5 (Pin_5), U1.19 (IO15)
- new net: J7.6 (Pin_6), U1.20 (IO16)
- new net: J8.1 (Pin_1), U1.30 (IO48)
- new net: J8.2 (Pin_2), U1.27 (IO47)
- new net: R5.1, U1.41 (IO45)
- new net: J5.1 (Pin_1), U1.8 (IO4)
- new net: J5.2 (Pin_2), U1.9 (IO5)
- new net: L1.1, U4.7 (SW)
- new net: R11.2, U4.8 (PG)
- new net: J6.1 (Pin_1), U1.12 (IO8)
- new net: J6.2 (Pin_2), U1.13 (IO9)
- new net: J3.1 (Pin_1), U1.25 (IO21)
- new net: J3.10 (Pin_10), U1.36 (IO40)
- new net: J3.11 (Pin_11), U1.37 (IO41)
- new net: J3.12 (Pin_12), U1.38 (IO42)
- new net: J3.2 (Pin_2), U1.26 (IO26)
- new net: J3.3 (Pin_3), U1.28 (IO33)
- new net: J3.4 (Pin_4), U1.29 (IO34)
- new net: J3.5 (Pin_5), U1.31 (IO35)
- new net: J3.6 (Pin_6), U1.32 (IO36)
- new net: J3.7 (Pin_7), U1.33 (IO37)
- new net: J3.8 (Pin_8), U1.34 (IO38)
- new net: J3.9 (Pin_9), U1.35 (IO39)
- new net BOOTMODE: SW3.2, U1.4 (IO0)
- no-connect marks 36 -> 7
Other:
- moved on the sheet: C6, C8, R3, R4, U10, U11, U2, U5, U6, U8, U9
