File: 1A-17V-4Motor-Driver/1A-17V-4Motor-Driver.kicad_sch (KiCad schematic)
At the start: 38 parts, among them J1 OUT2, J12 OUT1, J2 OUT3, J3 OUT4, J4 18V, J5 MUX, Q2 AOD4185, U1 TPM8837C-SO1R, U2 TPM8837C-SO1R, U3 TPM8837C-SO1R, U4 TPM8837C-SO1R, U5 MCP23017_ML, U6 TPS54227DDAR

Commit message: You slongoid
Parts:
- removed C12: 1 uF, Capacitor_SMD:C_0805_2012Metric, symbol Device:C_Small
- removed C13: 3.3 nF, Capacitor_SMD:C_0805_2012Metric, symbol Device:C_Small
- removed C14, C19: 10 uF, Capacitor_SMD:C_0805_2012Metric, symbol Device:C_Small
- removed C15: 100nF, Capacitor_SMD:C_0805_2012Metric, symbol Device:C_Small
- removed C16: 10 pF, Capacitor_SMD:C_0805_2012Metric, symbol Device:C_Small
- removed C17, C18: 22 uF, Capacitor_SMD:C_0805_2012Metric, symbol Device:C_Small
- removed L1: SRP7028A-4R7M, IND_SRP7028A-4R7M_BRN, symbol 2026-02-19_16-15-38:SRP7028A-4R7M
- removed R3: 10k, Resistor_SMD:R_0805_2012Metric, symbol Device:R_Small
- removed R4: 133k, Resistor_SMD:R_0805_2012Metric, symbol Device:R_Small
- removed R5: 24k, Resistor_SMD:R_0805_2012Metric, symbol Device:R_Small
- removed U6: TPS54227DDAR, TPS54227DDAR:VREG_LM5017MR_NOPB, symbol TPS54227DDAR:TPS54227DDAR
- added C20, C23, C25, C27: 220 uF, Capacitor_SMD:CP_Elec_8x10.5, symbol Device:C_Small
- added C21, C22, C24, C26: 0.1 uF, Capacitor_SMD:C_0805_2012Metric, symbol Device:C_Small
- added D12: LED, LED_SMD:LED_0805_2012Metric, symbol Device:LED
- added F1: 4A Fuse, Fuse:Fuse_1206_3216Metric, symbol Device:Fuse
- added J6: Conn_01x04_Pin, Connector_PinHeader_2.54mm:PinHeader_1x04_P2.54mm_Horizontal, symbol Connector:Conn_01x04_Pin
- added R4: 330, Resistor_SMD:R_0805_2012Metric, symbol Device:R
- added R6: 10k, Resistor_SMD:R_0805_2012Metric, symbol Device:R_Small
- Q2: footprint ul_AOD4185:TO252_AOS -> footprints:TO252_AOS
- U1, U2, U3, U4: footprint ul_TPM8837C-SO1R:SOP-8_TPK -> footprints:SOP-8_TPK
Connections:
- net +5V is gone; now on net VCC: C1.1, C10.1, C11.1, C2.1, C3.1, C4.1, C5.1, C6.1, C7.1, C8.1, C9.1, U1.7 (NSLEEP), U1.8 (VCC), U2.7 (NSLEEP), U2.8 (VCC), U3.7 (NSLEEP), U3.8 (VCC), U4.7 (NSLEEP), U4.8 (VCC), U5.5 (VDD)
- net GND: now also C20.1, C21.1, C22.1, C23.1, C24.1, C25.1, C26.1, C27.1, D12.2 (A), J6.4 (Pin_4); no longer R1.1
- net SCK: now also J6.2 (Pin_2)
- net SDA: now also J6.1 (Pin_1)
- net VCC: now also R1.1, R2.2, J6.3 (Pin_3), R4.2, R6.1; no longer Q2.3 (S), U1.1 (VM), U2.1 (VM), U3.1 (VM), U4.1 (VM)
- net at U5.14 (~{RESET}): now also R6.2
- new net: D12.1 (K), R4.1
- new net: F1.1, Q2.3 (S)
- new net +VDC: C20.2, C21.2, C22.2, C23.2, C24.2, C25.2, C26.2, C27.2, F1.2, U1.1 (VM), U2.1 (VM), U3.1 (VM), U4.1 (VM)
- no-connect marks 3 -> 2
Other:
- moved on the sheet: C5, J4, J5, Q2, R1, R2, U5
