File: HighEffNixiPSU/nixi_driver.kicad_sch (KiCad schematic)
At the start: 8 parts, among them U4 HV5622PG, U5 HV5622PG

Commit message: fha
Parts:
- U4, U5: LCSC Part # (none) -> C220637
Changed lines of the file:
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@@
+			)
+		)
+		(property "LCSC Part #" "C220637"
+			(at 52.07 118.11 0)
+			(effects
+				(font
+					(size 1.27 1.27)
+				)
+				(hide yes)
 			)
 		)
@@
 			)
 		)
+		(property "LCSC Part #" "C220637"
+			(at 52.07 151.13 0)
+			(effects
+				(font
+					(size 1.27 1.27)
+				)
+				(hide yes)
+			)
+		)
 		(pin "33"
 		)
@@
 			)
 		)
+		(property "LCSC Part #" "C220637"
+			(at 195.58 80.01 0)
+			(effects
+				(font
+					(size 1.27 1.27)
+				)
+				(hide yes)
+			)
+		)
 		(pin "13"
 		)
@@
 		(property "Description" "32-Channel, Serial to Parallel Converter w/ Open Drain Outputs, PQFP-44"
 			(at 196.85 144.272 0)
+			(effects
+				(font
+					(size 1.27 1.27)
+				)
+				(hide yes)
+			)
+		)
+		(property "LCSC Part #" "C220637"
+			(at 196.85 119.38 0)
 			(effects
 				(font
@@
 			)
 		)
+		(property "LCSC Part #" "C220637"
+			(at 52.07 87.63 0)
+			(effects
+				(font
+					(size 1.27 1.27)
+				)
+				(hide yes)
+			)
+		)
 		(pin "13"
 		)
@@
 		(property "Description" "32-Channel, Serial to Parallel Converter w/ Open Drain Outputs, PQFP-44"
 			(at 46.99 66.802 0)
+			(effects
+				(font
+					(size 1.27 1.27)
+				)
+				(hide yes)
+			)
+		)
+		(property "LCSC Part #" "C220637"
+			(at 46.99 41.91 0)
 			(effects
 				(font
@@
 			)
 		)
+		(property "LCSC Part #" "C220637"
+			(at 196.85 151.13 0)
+			(effects
+				(font
+					(size 1.27 1.27)
+				)
+				(hide yes)
+			)
+		)
 		(pin "33"
 		)
@@
 			(effects
 				(font
+					(size 1.27 1.27)
+				)
+				(hide yes)
+			)
+		)
+		(property "LCSC Part #" "C220637"
+			(at 190.5 40.64 0)
+			(effects
+				(font

Commit message: shivers got timbered
Parts:
- removed N1, N2, N3, N4, N5, N6: IN-14, nixies-us:nixies-us-IN-14, symbol nixies-us:IN-14
- added Br1, Br2, Br3, Br4, Br5, Br6: 33k Ohm, Resistor_SMD:R_1210_3225Metric, symbol Device:R
- added N1, N2, N3, N4, N5, N6: IN-16, nixies-us:nixies-us-IN-16, symbol nixies-us:IN-16
Connections:
- net GND: now also N1.LHDP, N1.RHDP, N2.LHDP, N3.LHDP, N3.RHDP, N4.LHDP, N5.LHDP, N5.RHDP, N6.LHDP, N6.RHDP
- net VCC: now also Br1.2, Br2.2, Br3.2, Br4.2, Br5.2, Br6.2
- net at U4.1 (HVOUT22): now also N3.2
- net at U4.2 (HVOUT21): now also N3.1
- net at U4.3 (HVOUT20): now also N2.0
- net at U4.4 (HVOUT19): now also N2.9
- net at U4.43 (HVOUT24): now also N3.4
- net at U4.44 (HVOUT23): now also N3.3
- net at U4.5 (HVOUT18): now also N2.8
- net at U4.6 (HVOUT17): now also N2.7
- net at U4.37 (HVOUT30): now also N3.0
- net at U4.38 (HVOUT29): now also N3.9
- net at U4.39 (HVOUT28): now also N3.8
- net at U4.40 (HVOUT27): now also N3.7
- net at U4.41 (HVOUT26): now also N3.6
- net at U4.42 (HVOUT25): now also N3.5
- net at U5.13 (HVOUT10): now also N4.0
- net at U5.22 (HVOUT1): now also N4.1
- net at U5.21 (HVOUT2): now also N4.2
- net at U5.20 (HVOUT3): now also N4.3
- net at U5.19 (HVOUT4): now also N4.4
- net at U5.18 (HVOUT5): now also N4.5
- net at U5.17 (HVOUT6): now also N4.6
- net at U5.16 (HVOUT7): now also N4.7
- net at U5.15 (HVOUT8): now also N4.8
- net at U5.14 (HVOUT9): now also N4.9
- net at U4.13 (HVOUT10): now also N1.0
- net at U4.22 (HVOUT1): now also N1.1
- net at U4.21 (HVOUT2): now also N1.2
- net at U4.20 (HVOUT3): now also N1.3
- net at U4.19 (HVOUT4): now also N1.4
- net at U4.18 (HVOUT5): now also N1.5
- net at U4.17 (HVOUT6): now also N1.6
- net at U4.16 (HVOUT7): now also N1.7
- net at U4.15 (HVOUT8): now also N1.8
- net at U4.14 (HVOUT9): now also N1.9
- net at U5.10 (HVOUT13): now also N5.3
- net at U5.11 (HVOUT12): now also N5.2
- net at U5.12 (HVOUT11): now also N5.1
- net at U5.7 (HVOUT16): now also N5.6
- net at U5.8 (HVOUT15): now also N5.5
- net at U5.9 (HVOUT14): now also N5.4
- net at U4.12 (HVOUT11): now also N2.1
- net at U4.11 (HVOUT12): now also N2.2
- net at U4.10 (HVOUT13): now also N2.3
- net at U4.9 (HVOUT14): now also N2.4
- net at U4.8 (HVOUT15): now also N2.5
- net at U4.7 (HVOUT16): now also N2.6
- net at U5.1 (HVOUT22): now also N6.2
- net at U5.2 (HVOUT21): now also N6.1
- net at U5.3 (HVOUT20): now also N5.0
- net at U5.4 (HVOUT19): now also N5.9
- net at U5.43 (HVOUT24): now also N6.4
- net at U5.44 (HVOUT23): now also N6.3
- net at U5.5 (HVOUT18): now also N5.8
- net at U5.6 (HVOUT17): now also N5.7
- net at U5.37 (HVOUT30): now also N6.0
- net at U5.42 (HVOUT25): now also N6.5
- net at U5.41 (HVOUT26): now also N6.6
- net at U5.40 (HVOUT27): now also N6.7
- net at U5.39 (HVOUT28): now also N6.8
- net at U5.38 (HVOUT29): now also N6.9
- net at U5.35 (HVOUT32): now also N4.RHDP
- net at U5.36 (HVOUT31): now also N2.RHDP
- new net: Br6.1, N6.A
- new net: Br5.1, N5.A
- new net: Br3.1, N3.A
- new net: Br2.1, N2.A
- new net: Br4.1, N4.A
- new net: Br1.1, N1.A
- no-connect marks 4 -> 2
