File: HighEffNixiPSU/HighEffNixiPSU.kicad_pcb (KiCad board)
At the start: 4 copper layers, 79.9 x 139.9 mm, 74 parts, among them IC1 AZ1117CH-3.3TRG1, J1 Jack-DC, J2 USB_C_Receptacle_USB2.0, Q1 FQD16N25CTM, Q10 2N2219, Q11 2N2219, Q2 2N2219, Q3 2N2219, Q4 2N2219, Q5 2N2219, Q6 2N2219, Q7 2N2219, Q8 2N2219, Q9 2N2219, SW2 EN, U1 LM3478MM, U2 ESP32-S3-MINI-1, U4 HV5622PG, U5 HV5622PG

Commit message: afawj
Parts:
- removed Q11: 2N2219, Package_TO_SOT_THT:TO-39-3
- added Q12: MMBTA06, Package_TO_SOT_SMD:SOT-23, F.Cu at (175.8, 37.0)
- Q10, Q2, Q3, Q4, Q5, Q6, Q7, Q8, Q9: value 2N2219 -> MMBTA06; footprint Package_TO_SOT_THT:TO-39-3 -> Package_TO_SOT_SMD:SOT-23
- moved R11 113.1 mm to (166.1, 63.4)
- moved GND1 98.5 mm to (201.7, 135.5), turned to 0 degrees
- moved R2 84.2 mm to (181.5, 112.8), turned to 0 degrees
- moved R27 78.2 mm to (189.4, 48.3)
- moved R25 76.3 mm to (187.0, 44.9), turned to -90 degrees
- moved R15 75.1 mm to (166.6, 116.2), turned to 0 degrees
- moved R26 72.4 mm to (186.3, 48.1), turned to 0 degrees
- moved R16 72.3 mm to (198.0, 138.0), turned to 90 degrees
- moved Ccomp2 71.8 mm to (154.7, 93.1)
- moved Q7 67.8 mm to (177.4, 114.0), turned to 180 degrees
- moved Q10 66.0 mm to (192.8, 47.3), turned to 180 degrees
- moved R21 57.8 mm to (172.4, 114.3), turned to 0 degrees
- moved R18 56.1 mm to (170.9, 111.9)
- moved R23 52.9 mm to (175.7, 107.5), turned to 180 degrees
- moved Q5 52.4 mm to (167.4, 100.1), turned to 0 degrees
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Connections:
- Q10 pad 1: GND -> Net-(Q10-B)
- Q10 pad 2: Net-(Q10-B) -> GND
- Q10 pad 3: Net-(Q10-C) -> /mcu/BL
- Q2 pad 1: GND -> Net-(Q2-B)
- Q2 pad 2: Net-(Q2-B) -> GND
- Q2 pad 3: Net-(Q2-C) -> /mcu/CLK
- Q3 pad 1: GND -> Net-(Q3-B)
- Q3 pad 2: Net-(Q3-B) -> GND
- Q3 pad 3: /mcu/CLK -> Net-(Q3-C)
- Q4 pad 1: GND -> Net-(Q4-B)
- Q4 pad 2: Net-(Q4-B) -> GND
- Q4 pad 3: Net-(Q4-C) -> /mcu/DAT
- Q5 pad 1: GND -> Net-(Q5-B)
- Q5 pad 2: Net-(Q5-B) -> GND
- Q5 pad 3: /mcu/DAT -> Net-(Q5-C)
- Q6 pad 1: GND -> Net-(Q6-B)
- Q6 pad 2: Net-(Q6-B) -> GND
- Q6 pad 3: Net-(Q6-C) -> /mcu/LE
- Q7 pad 1: GND -> Net-(Q7-B)
- Q7 pad 2: Net-(Q7-B) -> GND
- Q8 pad 1: GND -> Net-(Q8-B)
- Q8 pad 2: Net-(Q8-B) -> GND
- Q8 pad 3: /mcu/LE -> /mcu/POL
- Q9 pad 1: GND -> Net-(Q9-B)
- Q9 pad 2: Net-(Q9-B) -> GND
- Q9 pad 3: /mcu/POL -> Net-(Q9-C)
- R11 pad 2: Net-(Q4-B) -> Net-(Q3-B)
- R12 pad 2: Net-(Q4-C) -> Net-(Q3-C)
- R13 pad 1: Net-(Q4-C) -> Net-(Q3-C)
- R13 pad 2: Net-(Q5-B) -> Net-(Q4-B)
- R15 pad 2: Net-(Q6-B) -> Net-(Q5-B)
- R17 pad 2: Net-(Q6-C) -> Net-(Q5-C)
- R19 pad 1: Net-(Q6-C) -> Net-(Q5-C)
- R19 pad 2: Net-(Q8-B) -> Net-(Q6-B)
- R2 pad 2: Net-(Q2-B) -> Net-(Q12-B)
- R21 pad 2: Net-(Q9-B) -> Net-(Q8-B)
- R24 pad 2: Net-(Q10-B) -> Net-(Q9-B)
- R25 pad 2: Net-(Q10-C) -> Net-(Q9-C)
- R26 pad 1: Net-(Q10-C) -> Net-(Q9-C)
- R26 pad 2: Net-(Q11-B) -> Net-(Q10-B)
- R3 pad 2: Net-(Q2-C) -> Net-(Q12-C)
- R4 pad 1: Net-(Q2-C) -> Net-(Q12-C)
- R4 pad 2: Net-(Q3-B) -> Net-(Q2-B)
Routing:
- net +12V: track 27.1 -> 188.1 mm, vias 13 -> 0
- net Net-(Q4-B): track 117.3 -> 2.57 mm, vias 1 -> 0
- net /mcu/CLK_OUT: track 106.5 -> 9.75 mm, vias 2 -> 0
- net GND: track 81.9 -> 0.00 mm, vias 52 -> 84
- net Net-(Q12-B): track 0.00 -> 79.8 mm, vias 0 -> 2
- net /mcu/LE_OUT: track 92.2 -> 12.6 mm, vias 2 -> 0
- net Net-(Q9-B): track 8.54 -> 66.0 mm, vias 0 -> 2
- net Net-(Ccomp1-Pad2): track 62.7 -> 17.2 mm
- net Net-(Q2-B): track 40.7 -> 4.77 mm
- net Net-(Ccomp2-Pad2): track 25.5 -> 58.4 mm, vias 0 -> 2
- net Net-(Q6-B): track 39.1 -> 6.40 mm, vias 1 -> 2
- net Net-(Q10-B): track 40.6 -> 10.1 mm
- net /mcu/POL_OUT: track 63.3 -> 32.9 mm, vias 0 -> 2
- net VCC: track 182.3 -> 157.2 mm
- net Net-(U4A-HVOUT2): track 61.0 -> 40.2 mm, vias 0 -> 1
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- added copper zone on B.Cu, net GND
- added copper zone on F.Cu, net GND
- removed copper zone on In2.Cu, net +12V
- removed copper zone on In1.Cu, net GND
Other:
- board size 79.9 x 139.9 mm -> 76.2 x 122.8 mm
- copper layers 4 -> 2

Commit message: shivers got timbered
Parts:
- added Br1: 33k Ohm, Resistor_SMD:R_1210_3225Metric, F.Cu at (2.31, 1.60)
- added Br2: 33k Ohm, Resistor_SMD:R_1210_3225Metric, F.Cu at (2.31, 5.82)
- added Br3: 33k Ohm, Resistor_SMD:R_1210_3225Metric, F.Cu at (2.31, 10.0)
- added Br4: 33k Ohm, Resistor_SMD:R_1210_3225Metric, F.Cu at (2.31, 14.2)
- added Br5: 33k Ohm, Resistor_SMD:R_1210_3225Metric, F.Cu at (2.31, 18.4)
- added Br6: 33k Ohm, Resistor_SMD:R_1210_3225Metric, F.Cu at (2.31, 22.7)
- N1, N2, N3, N4, N5, N6: value IN-14 -> IN-16; footprint nixies-us:nixies-us-IN-14 -> nixies-us:nixies-us-IN-16; moved to B.Cu
- moved Q10 151.6 mm to (41.2, 44.7)
- moved Q12 151.6 mm to (24.1, 34.4)
- moved Q2 151.6 mm to (28.0, 33.9)
- moved Q9 151.6 mm to (38.8, 41.8)
- moved R10 151.6 mm to (27.0, 37.3)
- moved R25 151.6 mm to (35.4, 42.3)
- moved R26 151.6 mm to (34.7, 45.5)
- moved R27 151.6 mm to (37.8, 45.7)
- moved R3 151.6 mm to (29.4, 40.2)
- moved R4 151.6 mm to (23.9, 38.5)
- moved U5 151.6 mm to (46.0, 63.1)
- moved VIN1 151.6 mm to (43.4, 34.6)
- moved Rcomp1 100.2 mm to (107.1, 116.0)
- moved Q6 94.0 mm to (77.2, 93.1)
- moved R15 94.0 mm to (73.1, 107.3)
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Connections:
- N1 pad A: VCC -> Net-(Br1-Pad1)
- N2 pad A: VCC -> Net-(Br2-Pad1)
- N2 pad RHDP: GND -> Net-(U5D-HVOUT31)
- N3 pad A: VCC -> Net-(Br3-Pad1)
- N4 pad A: VCC -> Net-(Br4-Pad1)
- N4 pad RHDP: GND -> Net-(U5D-HVOUT32)
- N5 pad A: VCC -> Net-(Br5-Pad1)
- N6 pad A: VCC -> Net-(Br6-Pad1)
- U5 pad 35: unconnected-(U5D-HVOUT32-Pad35) -> Net-(U5D-HVOUT32)
- U5 pad 36: unconnected-(U5D-HVOUT31-Pad36) -> Net-(U5D-HVOUT31)
Routing:
- net +12V: track 188.1 -> 0.00 mm
- net VCC: track 157.2 -> 0.00 mm
- net /mcu/CLK: track 93.1 -> 0.00 mm, vias 4 -> 0
- net /mcu/BL: track 82.9 -> 0.00 mm, vias 4 -> 0
- net /mcu/DAT: track 81.2 -> 0.00 mm, vias 2 -> 0
- net Net-(Q12-B): track 79.8 -> 0.00 mm, vias 2 -> 0
- net /mcu/LE: track 77.6 -> 0.00 mm, vias 5 -> 0
- net +3V3: track 76.8 -> 0.00 mm, vias 4 -> 0
- net /mcu/POL: track 73.1 -> 0.00 mm, vias 3 -> 0
- net /mcu/DAT_OUT: track 67.9 -> 0.00 mm, vias 2 -> 0
- net Net-(U4B-HVOUT9): track 66.8 -> 0.00 mm, vias 1 -> 0
- net Net-(Q9-B): track 66.0 -> 0.00 mm, vias 2 -> 0
- net Net-(Ccomp2-Pad2): track 58.4 -> 0.00 mm, vias 2 -> 0
- net Net-(U4A-HVOUT8): track 54.4 -> 0.00 mm, vias 1 -> 0
- net Net-(U5A-HVOUT2): track 52.3 -> 0.00 mm, vias 3 -> 0
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Other:
- board size 76.2 x 122.8 mm -> 84.9 x 97.4 mm

Commit message: The so called shenanigooner
Parts:
- added S2: TL3340AF160QG, TL3340AF160QG:TL3340, F.Cu at (150.6, 109.2)
- moved Br2 258.3 mm to (223.7, 138.9), turned to -90 degrees
- moved Br1 257.2 mm to (214.9, 146.4), turned to 180 degrees
- moved Br3 237.1 mm to (215.7, 113.4), turned to -90 degrees
- moved Br4 233.2 mm to (217.9, 103.1)
- moved Br5 224.2 mm to (217.9, 79.9), turned to 180 degrees
- moved Br6 221.3 mm to (218.7, 68.9), turned to 90 degrees
- moved Q12 217.3 mm to (209.2, 148.2), turned to 180 degrees
- moved R4 215.1 mm to (207.1, 151.2), turned to 0 degrees
- moved Q2 210.7 mm to (205.2, 148.0), turned to -90 degrees
- moved R3 210.7 mm to (207.1, 153.5)
- moved R10 208.0 mm to (202.2, 149.4), turned to 90 degrees
- moved VIN1 180.5 mm to (210.6, 102.5)
- moved R25 174.6 mm to (191.6, 120.4), turned to 0 degrees
- moved Q9 173.9 mm to (195.4, 117.5), turned to 90 degrees
- moved R26 172.9 mm to (191.6, 118.1)
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Connections:
- C1 pad 1: Net-(C1-+) -> +12V
- Cbyp1 pad 1: Net-(C1-+) -> +12V
- L1 pad 1: Net-(C1-+) -> +12V
- U1 pad 8: Net-(C1-+) -> +12V
- U2 pad 13: unconnected-(U2-IO9-Pad13) -> Net-(U2-IO9)
Routing:
- net +12V: track 0.00 -> 199.8 mm
- net VCC: track 0.00 -> 161.9 mm
- net /mcu/CLK: track 0.00 -> 89.5 mm, vias 0 -> 4
- net +3V3: track 0.00 -> 83.4 mm, vias 0 -> 4
- net /mcu/BL: track 0.00 -> 75.1 mm, vias 0 -> 7
- net /mcu/POL: track 0.00 -> 70.8 mm, vias 0 -> 6
- net /mcu/BL_OUT: track 0.00 -> 67.5 mm, vias 0 -> 2
- net Net-(Q7-B): track 0.00 -> 59.9 mm, vias 0 -> 2
- net Net-(Q12-B): track 0.00 -> 58.5 mm, vias 0 -> 2
- net Net-(Q9-B): track 0.00 -> 56.8 mm, vias 0 -> 2
- net /mcu/LE: track 0.00 -> 54.7 mm, vias 0 -> 3
- net Net-(Q5-B): track 0.00 -> 54.6 mm, vias 0 -> 2
- net Net-(U5C-HVOUT24): track 0.00 -> 50.0 mm, vias 0 -> 1
- net Net-(U4C-HVOUT23): track 0.00 -> 47.9 mm, vias 0 -> 4
- net Net-(U4C-HVOUT24): track 0.00 -> 46.7 mm, vias 0 -> 3
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
Commit message: a
Parts:
- added H1: Mount, MountingHole:MountingHole_3mm_Pad_TopOnly, F.Cu at (166.1, 63.8)
- added H2: Mount, MountingHole:MountingHole_3mm_Pad_TopOnly, F.Cu at (213.4, 63.8)
- added H3: Mount, MountingHole:MountingHole_3mm_Pad_TopOnly, F.Cu at (158.7, 104.4)
- added H4: Mount, MountingHole:MountingHole_3mm_Pad_TopOnly, F.Cu at (200.5, 131.1)

Commit message: basti
Parts:
- removed IC1: AZ1117CH-3.3TRG1, AZ1117CH-3.3TRG1:SOT230P700X180-4N
- added C12: 100nF, Capacitor_SMD:C_0805_2012Metric, F.Cu at (190.5, 89.6)
- added C13: 100nF, Capacitor_SMD:C_0805_2012Metric, F.Cu at (187.5, 88.9)
- added C14: 100nF, Capacitor_SMD:C_0805_2012Metric, F.Cu at (194.3, 87.3)
- added C15: 100nF, Capacitor_SMD:C_0603_1608Metric, F.Cu at (200.2, 139.3)
- added C16: 15 pF, Capacitor_SMD:C_0402_1005Metric, F.Cu at (203.0, 136.8)
- added C17: 100nF, Capacitor_SMD:C_0603_1608Metric, F.Cu at (205.1, 145.7)
- added C18: 10uF, Capacitor_SMD:C_0805_2012Metric, F.Cu at (208.7, 134.1)
- added C19: 10uF, Capacitor_SMD:C_0805_2012Metric, F.Cu at (201.1, 145.9)
- added C2: 10 uF, Capacitor_SMD:C_Elec_10x10.2, F.Cu at (161.2, 106.8)
- added C20: 22uF, Capacitor_SMD:C_0805_2012Metric, F.Cu at (202.3, 140.6)
- added C3: 10uF, Capacitor_SMD:C_0805_2012Metric, F.Cu at (215.6, 90.3)
- added C4: 100nF, Capacitor_SMD:C_0805_2012Metric, F.Cu at (185.6, 91.9)
- added C7: 100nF, Capacitor_SMD:C_0805_2012Metric, F.Cu at (190.5, 87.3)
- added L2: SDR0403-3R3ML, footprints:IND_BOURNS_SDR0403, F.Cu at (203.0, 150.0)
- added Rfbb1: 10 kOhm, Resistor_SMD:R_0603_1608Metric, F.Cu at (200.2, 134.7)
- added Rfbt1: 30 kOhm, Resistor_SMD:R_0805_2012Metric, F.Cu at (204.6, 141.0)
- added U3: TPS562202, Package_TO_SOT_SMD:SOT-563, F.Cu at (207.5, 146.6)
- moved H1 101.0 mm to (215.2, 152.1), turned to 90 degrees
- moved H3 68.6 mm to (213.7, 63.3), turned to 90 degrees
- moved R24 62.5 mm to (168.8, 119.3)
- moved Q4 53.2 mm to (176.5, 64.7), turned to -90 degrees
- moved Q6 53.0 mm to (160.1, 89.0), turned to -90 degrees
- moved R14 52.6 mm to (173.4, 63.8), turned to 90 degrees
- moved R16 52.1 mm to (208.3, 73.3), turned to 180 degrees
- moved R7 51.1 mm to (169.2, 78.6), turned to 0 degrees
- moved R6 50.8 mm to (170.4, 76.3), turned to 0 degrees
- moved R22 50.5 mm to (159.4, 92.3)
- moved R19 49.1 mm to (163.1, 94.2)
- moved Ccomp2 48.5 mm to (185.6, 68.0), turned to 90 degrees
- moved R13 47.6 mm to (179.5, 64.2), turned to 90 degrees
- moved Q3 47.5 mm to (178.0, 68.1)
- moved H2 47.2 mm to (166.2, 63.3), turned to 90 degrees
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Routing:
- net GND: track 0.00 -> 123.9 mm, vias 89 -> 143
- net /mcu/LE: track 54.7 -> 137.8 mm, vias 3 -> 4
- net /mcu/DAT: track 33.8 -> 101.2 mm, vias 0 -> 2
- net /mcu/BL_OUT: track 67.5 -> 10.2 mm
- net /mcu/POL_OUT: track 18.1 -> 70.0 mm, vias 0 -> 2
- net +12V: track 199.8 -> 249.1 mm
- net Net-(U5A-HVOUT2): track 29.3 -> 76.5 mm, vias 2 -> 1
- net Net-(U5B-HVOUT16): track 15.3 -> 54.2 mm, vias 1 -> 0
- net Net-(Q12-B): track 58.5 -> 21.8 mm
- net Net-(U4D-HVOUT27): track 15.7 -> 51.6 mm, vias 1 -> 3
- net Net-(Ccomp2-Pad2): track 6.37 -> 39.7 mm, vias 0 -> 2
- net /mcu/LE_OUT: track 40.8 -> 9.34 mm
- net Net-(U3-VBST): track 0.00 -> 29.1 mm
- net Net-(U2-EN): track 5.51 -> 34.2 mm
- net Net-(U5A-HVOUT8): track 22.0 -> 49.6 mm
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- added copper zone on In1.Cu, net GND
- added copper zone on In2.Cu, net GND
- removed copper zone on B.Cu, net GND
- removed copper zone on F.Cu, net GND
Other:
- board size 84.9 x 97.4 mm -> 90 x 97.4 mm
- copper layers 2 -> 4
