File: HighEffNixiPSU/HighEffNixiPSU.kicad_sch (KiCad schematic)
At the start: 19 parts, among them J1 Screw_Terminal_01x02, Q1 FQD16N25CTM, U1 LM3478MM

Commit message: You slongoid
Parts:
- removed J1: Screw_Terminal_01x02, footprints:WJ500V-5.08-2P, symbol Connector:Screw_Terminal_01x02
- added IC1: AZ1117CH-3.3TRG1, AZ1117CH-3.3TRG1:SOT230P700X180-4N, symbol Personal:AZ1117CH-3.3TRG1
- added J1: Jack-DC, Connector_BarrelJack:BarrelJack_CUI_PJ-063AH_Horizontal, symbol Connector:Jack-DC
- C1: footprint EEE1AA101SP -> footprints:EEE1AA101SP
Connections:
- net GND: now also IC1.1 (ADJ/GND), J1.2
- net at C1.1 (+), Cbyp1.1, L1.1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: no longer VIN1.1 (Pin_1)
- net VCC: now reaches D1.2 (K), Rfb2.2
- new net +12V: IC1.3 (INPUT), J1.1, VIN1.1 (Pin_1)
- new net +3V3: IC1.2 (OUTPUT), IC1.4 (VOUT)
Other:
- added sheet mcu (mcu.kicad_sch)
- added sheet nixi_driver (nixi_driver.kicad_sch)
- moved on the sheet: C1, Cbyp1, Ccomp1, Ccomp2, Ccomp3, Cfilt1, D1, GND1, L1, Q1, RFilt1, RSense1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

Commit message: fha
Parts:
- IC1: LCSC Part # (none) -> C92102
Changed lines of the file:
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@@
+			)
+		)
+		(property "LCSC Part #" "C92102"
+			(at 88.9 25.4 0)
+			(effects
+				(font
+					(size 1.27 1.27)
+				)
+				(hide yes)
 			)
 		)

Commit message: The so called shenanigooner
Connections:
- net +12V: now also C1.1 (+), Cbyp1.1, L1.1, U1.8 (V_{IN})
Changed lines of the file:
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@@
 	)
 	(junction
+		(at 46.99 62.23)
+		(diameter 0)
+		(color 0 0 0 0)
+	)
+	(junction
 		(at 102.87 62.23)
 		(diameter 0)
@@
 	(wire
 		(pts
-			(xy 222.25 49.53) (xy 191.77 49.53)
+			(xy 232.41 49.53) (xy 191.77 49.53)
 		)
 		(stroke
@@
 	(symbol
 		(lib_id "power:VCC")
-		(at 222.25 49.53 0)
+		(at 232.41 49.53 0)
 		(unit 1)
 		(exclude_from_sim no)
@@
 		(fields_autoplaced yes)
 		(property "Reference" "#PWR010"
-			(at 222.25 53.34 0)
+			(at 232.41 53.34 0)
 			(effects
 				(font
@@
 		)
 		(property "Value" "VCC"
-			(at 222.25 44.45 0)
+			(at 232.41 44.45 0)
 			(effects
 				(font
@@
 		)
 		(property "Footprint" ""
-			(at 222.25 49.53 0)
+			(at 232.41 49.53 0)
 			(effects
 				(font
@@
 		)
 		(property "Datasheet" ""
-			(at 222.25 49.53 0)
+			(at 232.41 49.53 0)
 			(effects
 				(font
@@
 		)
 		(property "Description" "Power symbol creates a global label with name \"VCC\""
-			(at 222.25 49.53 0)
+			(at 232.41 49.53 0)
 			(effects
 				(font
@@
 					(unit 1)
 				)
+			)
+		)
+	)
+	(symbol
+		(lib_id "power:+12V")
+		(at 46.99 62.23 0)
+		(unit 1)
+		(exclude_from_sim no)
+		(in_bom yes)
+		(on_board yes)
+		(dnp no)
+		(fields_autoplaced yes)
+		(property "Reference" "#PWR057"
+			(at 46.99 66.04 0)
+			(effects
+				(font
+					(size 1.27 1.27)
+				)
+				(hide yes)
+			)
+		)
+		(property "Value" "+12V"
+			(at 46.99 57.15 0)
+			(effects
+				(font
+					(size 1.27 1.27)
+				)
+			)
+		)
+		(property "Footprint" ""
+			(at 46.99 62.23 0)
+			(effects
+				(font
+					(size 1.27 1.27)
+				)
+				(hide yes)
+			)
+		)
+		(property "Datasheet" ""
+			(at 46.99 62.23 0)
+			(effects
+				(font
+					(size 1.27 1.27)
+				)
+				(hide yes)
+			)
+		)
+		(property "Description" "Power symbol creates a global label with name \"+12V\""
+			(at 46.99 62.23 0)
+			(effects
+				(font
+					(size 1.27 1.27)
+				)
+				(hide yes)
+			)
+		)
+		(pin "1"
+		)
+		(instances
+			(project "HighEffNixiPSU"
+				(path "/6358b760-01e9-45d0-9d78-5a1aba5b2ae5"
+					(reference "#PWR057")
+					(unit 1)
+				)

Commit message: a
Parts:
- added H1, H2, H3, H4: Mount, MountingHole:MountingHole_3mm_Pad_TopOnly, symbol Mechanical:MountingHole_Pad
Connections:
- net GND: now also H1.1, H2.1, H3.1, H4.1
Other:
- moved on the sheet: IC1

Commit message: basti
Parts:
- removed IC1: AZ1117CH-3.3TRG1, AZ1117CH-3.3TRG1:SOT230P700X180-4N, symbol Personal:AZ1117CH-3.3TRG1
- added C12, C13, C14, C4, C7: 100nF, Capacitor_SMD:C_0805_2012Metric, symbol Device:C
- added C2: 10 uF, Capacitor_SMD:C_Elec_10x10.2, symbol Device:C_Polarized
- added C3: 10uF, Capacitor_SMD:C_0805_2012Metric, symbol Device:C
Connections:
- net +12V: now also C12.1, C13.1, C14.1, C3.1, C4.1, C7.1
- net GND: now also C12.2, C13.2, C14.2, C2.2, C3.2, C4.2, C7.2
- net VCC: now also C2.1
