File: HighEffNixiPSU/mcu.kicad_sch (KiCad schematic)
At the start: 46 parts, among them J2 USB_C_Receptacle_USB2.0, Q10 2N2219, Q11 2N2219, Q2 2N2219, Q3 2N2219, Q4 2N2219, Q5 2N2219, Q6 2N2219, Q7 2N2219, Q8 2N2219, Q9 2N2219, SW2 EN, U2 ESP32-S3-MINI-1

Commit message: afawj
Parts:
- removed Q10, Q11, Q2, Q3, Q4, Q5, Q6, Q7, Q8, Q9: 2N2219, Package_TO_SOT_THT:TO-39-3, symbol Transistor_BJT:2N2219
- added Q10, Q12, Q2, Q3, Q4, Q5, Q6, Q7, Q8, Q9: MMBTA06, Package_TO_SOT_SMD:SOT-23, symbol Transistor_BJT:MMBTA06
Connections:
- net BL: now also Q10.3 (C)
- net CLK: now also Q2.3 (C)
- net DAT: now also Q4.3 (C)
- net GND: now also Q10.2 (E), Q12.2 (E), Q2.2 (E), Q3.2 (E), Q4.2 (E), Q5.2 (E), Q6.2 (E), Q7.2 (E), Q8.2 (E), Q9.2 (E)
- net LE: now also Q6.3 (C)
- net POL: now also Q8.3 (C)
- net at R15.2: now also Q5.1 (B)
- net at R26.2: now also Q10.1 (B)
- net at R16.2: now also Q7.1 (B)
- net at R2.2: now also Q12.1 (B)
- net at R17.2, R19.1: now also Q5.3 (C)
- net at R11.2: now also Q3.1 (B)
- net at R12.2, R13.1: now also Q3.3 (C)
- net at R18.2, R21.1: now also Q7.3 (C)
- net at R3.2, R4.1: now also Q12.3 (C)
- net at R25.2, R26.1: now also Q9.3 (C)
- net at R21.2: now also Q8.1 (B)
- net at R19.2: now also Q6.1 (B)
- net at R24.2: now also Q9.1 (B)
- net at R4.2: now also Q2.1 (B)
- net at R13.2: now also Q4.1 (B)

Commit message: fha
Parts:
- Q10, Q12, Q2, Q3, Q4, Q5, Q6, Q7, Q8, Q9: LCSC Part # (none) -> C20069139
- S1: LCSC Part # (none) -> C109335
Changed lines of the file:
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@@
 			)
 		)
+		(property "LCSC Part #" "C20069139"
+			(at 45.72 116.84 0)
+			(effects
+				(font
+					(size 1.27 1.27)
+				)
+				(hide yes)
+			)
+		)
 		(pin "1"
 		)
@@
 			)
 		)
+		(property "LCSC Part #" "C109335"
+			(at 95.25 27.94 0)
+			(effects
+				(font
+					(size 1.27 1.27)
+				)
+				(hide yes)
+			)
+		)
 		(pin "4"
 		)
@@
 			)
 		)
+		(property "LCSC Part #" "C20069139"
+			(at 45.72 148.59 0)
+			(effects
+				(font
+					(size 1.27 1.27)
+				)
+				(hide yes)
+			)
+		)
 		(pin "1"
 		)
@@
 			)
 		)
+		(property "LCSC Part #" "C20069139"
+			(at 67.31 148.59 0)
+			(effects
+				(font
+					(size 1.27 1.27)
+				)
+				(hide yes)
+			)
+		)
 		(pin "1"
 		)
@@
 			)
 		)
+		(property "LCSC Part #" "C20069139"
+			(at 45.72 85.09 0)
+			(effects
+				(font
+					(size 1.27 1.27)
+				)
+				(hide yes)
+			)
+		)
 		(pin "1"
 		)
@@
 			)
 		)
+		(property "LCSC Part #" "C20069139"
+			(at 67.31 116.84 0)
+			(effects
+				(font
+					(size 1.27 1.27)
+				)
+				(hide yes)
+			)
+		)
 		(pin "1"
 		)
@@
 			)
 		)
+		(property "LCSC Part #" "C20069139"
+			(at 123.19 180.34 0)
+			(effects
+				(font
+					(size 1.27 1.27)
+				)
+				(hide yes)
+			)
+		)
 		(pin "1"
 		)
@@
 			)
 		)
+		(property "LCSC Part #" "C20069139"
+			(at 144.78 180.34 0)
+			(effects
+				(font
+					(size 1.27 1.27)
+				)
+				(hide yes)
+			)
+		)
 		(pin "1"
 		)
@@
 			)
 		)
+		(property "LCSC Part #" "C20069139"
+			(at 67.31 180.34 0)
+			(effects
+				(font
+					(size 1.27 1.27)
+				)
+				(hide yes)
+			)
+		)
 		(pin "1"
 		)
@@
 			)
 		)
+		(property "LCSC Part #" "C20069139"
+			(at 45.72 180.34 0)
+			(effects
+				(font
+					(size 1.27 1.27)
+				)
+				(hide yes)
+			)
+		)
 		(pin "1"
 		)
@@
 			(at 67.31 85.09 0)
 			(effects
+				(font
+					(size 1.27 1.27)
+				)
+				(hide yes)
+			)
+		)
+		(property "LCSC Part #" "C20069139"
+			(at 67.31 85.09 0)
+			(effects

Commit message: The so called shenanigooner
Parts:
- added S2: TL3340AF160QG, TL3340, symbol Personal:TL3340AF160QG
Connections:
- net GND: now also S2.1, S2.3
- net at U2.13 (IO9): now also S2.2

Commit message: a
Parts:
- S2: footprint TL3340 -> TL3340AF160QG:TL3340
Changed lines of the file:
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@@
 			)
 		)
-		(property "Footprint" "TL3340"
+		(property "Footprint" "TL3340AF160QG:TL3340"
 			(at 153.67 141.91 0)
 			(effects

Commit message: basti
Parts:
- added C15, C17: 100nF, Capacitor_SMD:C_0603_1608Metric, symbol Device:C
- added C16: 15 pF, Capacitor_SMD:C_0402_1005Metric, symbol Device:C
- added C18, C19: 10uF, Capacitor_SMD:C_0805_2012Metric, symbol Device:C
- added C20: 22uF, Capacitor_SMD:C_0805_2012Metric, symbol Device:C
- added L2: SDR0403-3R3ML, footprints:IND_BOURNS_SDR0403, symbol Personal:SDR0403-3R3ML
- added Rfbb1: 10 kOhm, Resistor_SMD:R_0603_1608Metric, symbol Device:R_Small
- added Rfbt1: 30 kOhm, Resistor_SMD:R_0805_2012Metric, symbol Device:R_Small
- added U3: TPS562202, Package_TO_SOT_SMD:SOT-563, symbol Regulator_Switching:TPS562202
Connections:
- net +12V: now also C17.1, C18.1, C19.1, U3.1 (VIN), U3.5 (EN)
- net +3V3: now also C16.1, C20.1, L2.1, Rfbt1.1
- net GND: now also C17.2, C18.2, C19.2, C20.2, Rfbb1.2, U3.3 (GND)
- new net: C16.2, Rfbb1.1, Rfbt1.2, U3.6 (VFB)
- new net: C15.1, U3.4 (VBST)
- new net: C15.2, L2.2, U3.2 (SW)
