File: Psu/BuckV1/BuckV1.kicad_pcb (KiCad board)
At the start: 2 copper layers, 50 x 59.9 mm, 17 parts, among them J1 IN, J2 OUT, Q1 STD10P6F6, U1 LM2576HVS-ADJ, U2 STPS20M100SG-TR

Commit message: raaaa
Parts:
- removed Q1: STD10P6F6, footprints:STD10P6F6
- added Q2: STD10P6F6, footprints:STD10P6F6, F.Cu at (107.2, 110.1)
- moved C2 98.6 mm to (108.3, 80.5), turned to 0 degrees
- moved C1 84.6 mm to (107.7, 96.3)
- moved S1 82.7 mm to (126.9, 106.2), turned to 0 degrees
- moved U1 70.3 mm to (127.9, 95.4)
- moved C3 70.1 mm to (119.2, 102.9), turned to 0 degrees
- moved C4 69.6 mm to (119.2, 105.4), turned to 0 degrees
- moved C6 68.4 mm to (119.2, 110.4), turned to 0 degrees
- moved C5 59.8 mm to (119.2, 107.9), turned to 0 degrees
- moved J2 58.0 mm to (128.1, 111.6), turned to 0 degrees
- moved R2 55.9 mm to (134.8, 112.4), turned to 0 degrees
- moved U2 52.5 mm to (126.7, 78.2), turned to 0 degrees
- moved L1 50.3 mm to (139.9, 78.8)
- moved R1 46.8 mm to (134.8, 109.5), turned to 0 degrees
- moved J1 43.4 mm to (123.5, 111.6)
- moved F1 35.5 mm to (141.0, 95.3)
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Connections:
- C1 pad 1: Net-(U1-VIN) -> Net-(Q2-D)
- C3 pad 1: Net-(U1-VIN) -> Net-(Q2-D)
- C4 pad 1: Net-(U1-VIN) -> Net-(Q2-D)
- F1 pad 1: Net-(Q1-D) -> Net-(J1-Pin_1)
- F1 pad 2: Net-(U1-VIN) -> Net-(Q2-S)
- U1 pad 1: Net-(U1-VIN) -> Net-(Q2-D)
Routing:
- net Net-(J2-Pin_1): track 40.2 -> 0.00 mm
- net Net-(U1-OUT): track 33.8 -> 0.00 mm
- net Net-(U1-VIN): track 32.4 -> 0.00 mm
- net Net-(U1-FB): track 25.1 -> 0.00 mm, vias 1 -> 0
- net /EN: track 18.6 -> 0.00 mm, vias 2 -> 0
- net Net-(Q1-D): track 11.3 -> 0.00 mm
- net Net-(J1-Pin_1): track 7.45 -> 0.00 mm
- net Net-(R1-Pad1): track 6.62 -> 0.00 mm, vias 1 -> 0
- net GND: vias 79 -> 0
- removed copper zone on B.Cu, net GND
- removed copper zone on F.Cu, net GND

Commit message: Ra ra rasputin
Parts:
- moved C1 92.2 mm to (196.7, 72.6)
- moved Q2 89.5 mm to (196.7, 112.3), turned to -90 degrees
- moved C4 79.0 mm to (191.2, 73.0), turned to 90 degrees
- moved C3 76.9 mm to (191.0, 75.4), turned to 180 degrees
- moved S1 75.5 mm to (198.9, 83.4)
- moved J1 69.1 mm to (192.3, 118.1), turned to 90 degrees
- moved C6 64.6 mm to (178.1, 84.0), turned to 90 degrees
- moved C5 63.8 mm to (176.3, 79.3), turned to 90 degrees
- moved C2 63.6 mm to (167.7, 103.2)
- moved U1 60.5 mm to (187.7, 86.5), turned to -90 degrees
- moved J2 56.3 mm to (179.0, 87.5)
- moved R2 54.4 mm to (180.9, 83.5), turned to 90 degrees
- moved R1 52.1 mm to (178.1, 80.5), turned to 90 degrees
- moved F1 48.4 mm to (184.6, 116.2), turned to 90 degrees
- moved VR1 46.1 mm to (183.8, 95.9)
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Connections:
- S1 pad 1: +3V3 -> Net-(Q2-D)
Routing:
- net Net-(Q2-D): track 0.00 -> 55.7 mm, vias 0 -> 2
- net Net-(U1-OUT): track 0.00 -> 33.7 mm
- net Net-(J2-Pin_1): track 0.00 -> 32.8 mm
- net Net-(U1-FB): track 0.00 -> 27.5 mm, vias 0 -> 1
- net /EN: track 0.00 -> 20.0 mm
- net Net-(R1-Pad1): track 0.00 -> 17.5 mm, vias 0 -> 1
- net Net-(J1-Pin_1): track 0.00 -> 8.31 mm
- net Net-(Q2-S): track 0.00 -> 8.30 mm
- net GND: vias 0 -> 66
- added copper zone on B.Cu, net GND
- added copper zone on F.Cu, net GND

Commit message: ra
Parts:
- removed S1: SSSS811101, footprints:SSSS811101
- moved U2 39.3 mm to (201.7, 97.3), turned to -90 degrees
- moved J1 27.3 mm to (168.9, 104.1), turned to 0 degrees
- moved C2 20.8 mm to (188.2, 106.5), turned to 180 degrees
- moved VR1 17.7 mm to (198.5, 105.7)
- moved U1 15.4 mm to (202.2, 81.3), turned to 90 degrees
- moved R2 14.7 mm to (194.0, 90.3), turned to -90 degrees
- moved C5 14.5 mm to (164.4, 87.5)
- moved Q2 14.4 mm to (183.8, 118.8)
- moved L1 14.2 mm to (184.0, 91.2), turned to 90 degrees
- moved R1 14.2 mm to (166.9, 89.2), turned to 0 degrees
- moved C4 13.6 mm to (191.7, 86.5)
- moved F1 13.0 mm to (171.8, 114.0), turned to -90 degrees
- moved C3 13.0 mm to (194.8, 87.8)
- moved C6 8.60 mm to (169.6, 84.0), turned to 180 degrees
- moved C1 7.62 mm to (190.0, 76.2), turned to 90 degrees
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Connections:
- U1 pad 5: /EN -> GND
Routing:
- net Net-(R1-Pad1): track 17.5 -> 37.6 mm
- net /EN: track 20.0 -> 0.00 mm
- net Net-(J2-Pin_1): track 32.8 -> 48.5 mm
- net Net-(U1-FB): track 27.5 -> 31.3 mm, vias 1 -> 2
- net Net-(Q2-S): track 8.30 -> 9.78 mm
- net Net-(U1-OUT): track 33.7 -> 32.3 mm, vias 0 -> 2
- net Net-(Q2-D): track 55.7 -> 56.1 mm, vias 2 -> 0
- net GND: vias 66 -> 72
