File: Psu/BuckV1/BuckV1.kicad_sch (KiCad schematic)
At the start: 17 parts, among them J1 IN, J2 OUT, Q1 STD10P6F6, U1 LM2576HVS-ADJ, U2 STPS20M100SG-TR

Commit message: raaaa
Parts:
- removed Q1: STD10P6F6, STD10P6F6, symbol Personal:STD10P6F6
- added Q2: STD10P6F6, STD10P6F6, symbol Personal:STD10P6F6
Connections:
- net GND: now also Q2.1 (G)
- net at J1.1 (Pin_1): now also F1.1
- net at C1.1, C3.1, C4.1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: now also Q2.2 (D); no longer F1.2
- new net: F1.2, Q2.3 (S)
Other:
- moved on the sheet: F1

Commit message: Ra ra rasputin
Parts:
- Q2: footprint STD10P6F6 -> footprints:STD10P6F6
Connections:
- net +3V3 is gone; now on an unnamed net: S1.1
Changed lines of the file:
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@@
+	(wire
+		(pts
+			(xy 39.37 92.71) (xy 55.88 92.71)
+		)
+		(stroke
+			(width 0)
+			(type default)
+		)
+	)
+	(wire
+		(pts
+			(xy 39.37 121.92) (xy 39.37 92.71)
+		)
+		(stroke
+			(width 0)
+			(type default)
+		)
+	)
 	(wire
 		(pts
@@
 	(wire
 		(pts
-			(xy 185.42 97.79) (xy 196.85 97.79)
+			(xy 39.37 121.92) (xy 74.93 121.92)
 		)
 		(stroke
@@
 	(wire
 		(pts
-			(xy 105.41 107.95) (xy 105.41 102.87)
+			(xy 185.42 97.79) (xy 196.85 97.79)
 		)
 		(stroke
@@
 	(wire
 		(pts
-			(xy 34.29 92.71) (xy 24.13 92.71)
+			(xy 105.41 107.95) (xy 105.41 102.87)
 		)
 		(stroke
@@
 	(wire
 		(pts
-			(xy 140.97 97.79) (xy 168.91 97.79)
+			(xy 34.29 92.71) (xy 24.13 92.71)
 		)
 		(stroke
@@
 	(wire
 		(pts
-			(xy 163.83 83.82) (xy 162.56 83.82)
+			(xy 140.97 97.79) (xy 168.91 97.79)
 		)
 		(stroke
@@
 	(wire
 		(pts
-			(xy 34.29 77.47) (xy 34.29 92.71)
+			(xy 163.83 83.82) (xy 162.56 83.82)
 		)
 		(stroke
@@
 	(wire
 		(pts
-			(xy 162.56 83.82) (xy 162.56 92.71)
+			(xy 34.29 77.47) (xy 34.29 92.71)
 		)
 		(stroke
@@
 	(wire
 		(pts
-			(xy 66.04 127) (xy 74.93 127)
+			(xy 162.56 83.82) (xy 162.56 92.71)
 		)
 		(stroke
@@
 	(wire
 		(pts
-			(xy 66.04 121.92) (xy 74.93 121.92)
+			(xy 66.04 127) (xy 74.93 127)
 		)
 		(stroke
@@
 			)
 		)
-		(property "Footprint" "STD10P6F6"
+		(property "Footprint" "footprints:STD10P6F6"
 			(at 52.07 -16.18 0)
 			(effects
@@
 					(unit 1)
 				)
-			)
-		)
-	)
-	(symbol
-		(lib_id "power:+3V3")
-		(at 66.04 121.92 0)
-		(unit 1)
-		(exclude_from_sim no)
-		(in_bom yes)
-		(on_board yes)
-		(dnp no)
-		(property "Reference" "#PWR067"
-			(at 66.04 125.73 0)
-			(effects
-				(font
-					(size 1.27 1.27)
-				)
-				(hide yes)
-			)
-		)
-		(property "Value" "+3V3"
-			(at 66.04 118.11 0)
-			(effects
-				(font
-					(size 1.27 1.27)
-				)
-			)
-		)
-		(property "Footprint" ""
-			(at 66.04 121.92 0)
-			(effects
-				(font
-					(size 1.27 1.27)
-				)
-				(hide yes)
-			)
-		)
-		(property "Datasheet" ""
-			(at 66.04 121.92 0)
-			(effects
-				(font
-					(size 1.27 1.27)
-				)
-				(hide yes)
-			)
-		)
-		(property "Description" ""
-			(at 66.04 121.92 0)
-			(effects
-				(font
-					(size 1.27 1.27)
-				)
-			)
-		)
-		(pin "1"
-		)
-		(instances
-			(project "BuckV1"
-				(path "/1ea0fc8a-a46b-4318-aa68-554101b34543"
-					(reference "#PWR067")
-					(unit 1)
-				)

Commit message: ra
Parts:
- removed S1: SSSS811101, footprints:SSSS811101, symbol Personal:SSSS811101
Connections:
- net EN is gone; now on net GND: U1.5 (~{ON}/OFF)
- no-connect marks 5 -> 1
