File: Measurement/LC-Resonator/LC-Resonator.kicad_sch (KiCad schematic)
At the start: 19 parts, among them J3 USB_C_Receptacle_USB2.0, SW1 KH-6X6X5H-STM, U1 CH552G, U2 74HC04, U4 PRTR5V0U2X

Commit message: wajfawj
Parts:
- removed C1, C2: 100pF, symbol Device:C
- removed C_dec: 100nF, Capacitor_SMD:C_0402_1005Metric, symbol Device:C_Small
- removed F1: 500 mA, Fuse:Fuse_1206_3216Metric, symbol Device:Polyfuse
- removed J_L: L_unknown, symbol Connector_Generic:Conn_01x02
- removed Rf: 1M, Resistor_SMD:R_0402_1005Metric, symbol Device:R
- removed U2: 74HC04, Package_SO:SOIC-14_3.9x8.7mm_P1.27mm, symbol 74xx:74HC04
- removed U4: PRTR5V0U2X, Package_TO_SOT_SMD:SOT-143, symbol Power_Protection:PRTR5V0U2X
- added C1, C10, C12, C5: 100n, Capacitor_SMD:C_0603_1608Metric, symbol Device:C_Small
- added C11, C9: 10u, Capacitor_SMD:C_0603_1608Metric, symbol Device:C_Small
- added C2, C4: 1n, Capacitor_SMD:C_0603_1608Metric, symbol Device:C_Small
- added C8: 470n, Capacitor_SMD:C_0603_1608Metric, symbol Device:C_Small
- added J2, J3: Lx, footprints:4mm_Banana_Socket_Deltron_571, symbol Connector:Conn_01x01_Socket
- added L1: 1uH, Inductor_SMD:L_0805_2012Metric, symbol Device:L
- added M1: OLED 1.3", footprints:LCD_OLED_128X64_1.3_I2C, symbol Connector_Generic:Conn_01x04
- added Q1: 2SC3356, Package_TO_SOT_SMD:SOT-23, symbol Transistor_BJT:MMBT2222A
- added R10, R11, R12, R14, R5, R6: 10k, Resistor_SMD:R_0603_1608Metric, symbol Device:R
- added R13: 470, Resistor_SMD:R_0603_1608Metric, symbol Device:R
- added R7: 2k2, Resistor_SMD:R_0603_1608Metric, symbol Device:R
- added R9: 100k, Resistor_SMD:R_0603_1608Metric, symbol Device:R
- added SW2: KH-6X6X5H-STM, footprints:KH-6X6X5H-STM_SKE, symbol Personal:KH-6X6X5H-STM
- added U3: 74HC590, Package_SO:SOIC-16_3.9x9.9mm_P1.27mm, symbol 74xx:74HC590
- added U4: MCP6561R, Package_TO_SOT_SMD:SOT-23-5, symbol Comparator:MCP6561R
- C3: value 100nF -> 1n; footprint Capacitor_SMD:C_0805_2012Metric -> Capacitor_SMD:C_0603_1608Metric; LCSC (none) -> C309468; LCSC Part # C49678 -> (none); Package/Case (none) -> 0603; Par (none) -> 1% NP0
- renumbered C3 to C6, C4 to C7, J3 to J1, R6 to R1, R7 to R2, R8 to R3, R9 to R4, R1 to R8, U1 to U2
Connections:
- net GND: now also J1.A1 (GND), J1.A12 (GND), J1.B1 (GND), J1.B12 (GND), C1.2, C10.2, C11.2, C12.2, C5.2, C8.2, C9.2, M1.2 (Pin_2), R11.2, R6.2, R7.2, SW2.A, U3.12 (~{CE}), U3.14 (~{OE}), U3.8 (GND), U4.5 (V-)
- net VBUS: now also C7.2, SW1.C, SW1.D, U2.15 (VCC), C10.1, C11.1, C12.1, C9.1, L1.2, M1.1 (Pin_1), R10.1, R12.1, R14.1, R5.1, U3.16 (VCC), U4.2 (V+)
- net FREQ: now reaches U2.1 (P3.2)
- net FREQ: now also U3.7 (Q7)
- net SCL: now reaches U2.10 (P3.3)
- net SCL: now also M1.3 (Pin_3)
- net BTN: now reaches U2.2 (P1.4)
- net BTN: now also C8.1, R13.1
- net CLRST: now reaches U2.3 (P1.5)
- net CLRST: now also R12.2, U3.10 (~{MRC})
- removed net +5V: C3.1, C7.2, SW1.C, SW1.D, U2.15 (VCC)
- net OSC_OUT renamed SDA
- net SDA: now also M1.4 (Pin_4)
- new net: C2.2, C3.1, Q1.2 (E), R7.1
- new net: U3.11 (CPC), U3.13 (CPR), U4.1
- new net: C4.2, R9.1, U4.3 (+)
- new net: C5.1, R10.2, R11.1, R9.2, U4.4 (-)
- new net: J3.1 (Pin_1), L1.1
- new net: R13.2, R14.2, SW2.D
- new net: C2.1, C4.1, J2.1 (Pin_1), Q1.3 (C)
- new net: C1.1, Q1.1 (B), R5.2, R6.1
- no-connect marks 2 -> 12
Other:
- note removed: "Colpitts Resonator Tank Circuit f = 1/(2pi * sqrt(L * Ceq)) Ceq = C1*C2/(C1+C2) = 50pF f ~ 2.25 MHz (L=100uH, C1=C2=100pF) J1: frequency measurement (Out vs GND) J2: capacitance measurement (Mid vs GND)"
- moved on the sheet: C6, C7, R8, SW1, U2

Commit message: faw
Parts:
- L1: LCSC C1042 -> C113100
- M1: LCSC ------ -> C7465997
Changed lines of the file:
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@@
 			)
 		)
-		(property "LCSC" "C1042"
+		(property "LCSC" "C113100"
 			(at 49.53 44.45 90)
 			(effects
@@
 			)
 		)
-		(property "LCSC" "------"
+		(property "LCSC" "C7465997"
 			(at 245.11 133.35 0)
 			(effects
