File: Misc/USB-C-Fastcharger/USB-C-Fastcharger.kicad_sch (KiCad schematic)
At the start: 13 parts, among them J1 USB_C_Receptacle_USB2.0_16P, J3 VOUT, Q1 PMOS, U1 HUSB238_xxxDD

Commit message: fajhw
Parts:
- removed C2: 680 uF, Capacitor_THT:CP_Radial_D12.5mm_P5.00mm, symbol Device:C_Polarized
- added C2, C5: 100 uF, Capacitor_SMD:C_0805_2012Metric, symbol Device:C
- added C6: 10uF, Capacitor_SMD:C_0805_2012Metric, symbol Device:C
- added C7: 100nF, Capacitor_SMD:C_0805_2012Metric, symbol Device:C
- added F1: 3A 30V, Fuse:Fuse_2920_7451Metric, symbol Device:Fuse
- added J4: I2C, Connector_PinHeader_2.54mm:PinHeader_1x04_P2.54mm_Vertical, symbol Connector:Conn_01x04_Pin
- added R4: 0 Ohm, Resistor_SMD:R_0805_2012Metric, symbol Device:R_Small
- C3: footprint Capacitor_SMD:C_0603_1608Metric -> Capacitor_SMD:C_0805_2012Metric; LCSC C19702 -> C440198
- C4: footprint Capacitor_SMD:C_0603_1608Metric -> Capacitor_SMD:C_0805_2012Metric; LCSC C14663 -> C49678
- R1: value 10 ohm -> 0 Ohm; LCSC Part # C17415 -> C17477
Connections:
- net GND: now also C2.2, C5.1, C6.1, C7.1, J4.4 (Pin_4)
- net at C3.1, C4.1, J3.1 (Pin_1)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: now also C2.1
- net at J1.A4 (VBUS), J1.A9 (VBUS), J1.B4 (VBUS)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: now also F1.1; no longer Q1.1 (D), R1.1, R3.1
- net at C1.2, U1.1 (VIN): now also Q1.1 (D), R3.1, C5.2, C6.2, C7.2, F1.2; no longer R1.2
- net at U1.6 (SDA): now also J4.3 (Pin_3), R4.2
- net at U1.7 (SCL): now also R1.2, J4.2 (Pin_2)
- new net: J4.1 (Pin_1), R1.1, R4.1
- no-connect marks 6 -> 4
Other:
- moved on the sheet: J1
