File: Bluetooth Box V3/power.kicad_sch (KiCad schematic)
At the start: 8 parts, among them U10 MIC5356-SGYMME

Commit message: started pcb routing
Parts:
- renumbered C49 to C33, C50 to C34, C36 to C35, C37 to C36, CR2 to CR1, R11 to R18, R12 to R19, U10 to U6
Changed lines of the file:
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@@
 		(on_board yes)
 		(dnp no)
-		(property "Reference" "C37"
+		(property "Reference" "C36"
 			(at 113.03 83.8262 0)
 			(effects
@@
 			(project "Bluetooth Box V3"
 				(path "/c5f2915a-1379-46bf-9932-ae9df9d21574/08bbdc8c-2f8e-4da1-ab4d-f5452d4c4cd9"
-					(reference "C37")
+					(reference "C36")
 					(unit 1)
 				)
@@
 		(on_board yes)
 		(dnp no)
-		(property "Reference" "C36"
+		(property "Reference" "C35"
 			(at 104.14 82.5562 0)
 			(effects
@@
 			(project "Bluetooth Box V3"
 				(path "/c5f2915a-1379-46bf-9932-ae9df9d21574/08bbdc8c-2f8e-4da1-ab4d-f5452d4c4cd9"
-					(reference "C36")
+					(reference "C35")
 					(unit 1)
 				)
@@
 		(on_board yes)
 		(dnp no)
-		(property "Reference" "#PWR063"
+		(property "Reference" "#PWR051"
 			(at 69.85 66.04 0)
 			(effects
@@
 			(project "Bluetooth Box V3"
 				(path "/c5f2915a-1379-46bf-9932-ae9df9d21574/08bbdc8c-2f8e-4da1-ab4d-f5452d4c4cd9"
-					(reference "#PWR063")
+					(reference "#PWR051")
 					(unit 1)
 				)
@@
 		(dnp no)
 		(fields_autoplaced yes)
-		(property "Reference" "#PWR059"
+		(property "Reference" "#PWR050"
 			(at 46.99 54.61 0)
 			(effects
@@
 			(project "Bluetooth Box V3"
 				(path "/c5f2915a-1379-46bf-9932-ae9df9d21574/08bbdc8c-2f8e-4da1-ab4d-f5452d4c4cd9"
-					(reference "#PWR059")
+					(reference "#PWR050")
 					(unit 1)
 				)
@@
 		(on_board yes)
 		(dnp no)
-		(property "Reference" "#PWR061"
+		(property "Reference" "#PWR053"
 			(at 118.11 57.15 0)
 			(effects
@@
 			(project "Bluetooth Box V3"
 				(path "/c5f2915a-1379-46bf-9932-ae9df9d21574/08bbdc8c-2f8e-4da1-ab4d-f5452d4c4cd9"
-					(reference "#PWR061")
+					(reference "#PWR053")
 					(unit 1)
 				)
@@
 		(dnp no)
 		(fields_autoplaced yes)
-		(property "Reference" "R11"
+		(property "Reference" "R18"
 			(at 64.77 74.93 90)
 			(effects
@@
 			(project "Bluetooth Box V3"
 				(path "/c5f2915a-1379-46bf-9932-ae9df9d21574/08bbdc8c-2f8e-4da1-ab4d-f5452d4c4cd9"
-					(reference "R11")
+					(reference "R18")
 					(unit 1)
 				)
@@
 		(dnp no)
 		(fields_autoplaced yes)
-		(property "Reference" "#PWR062"
+		(property "Reference" "#PWR052"
 			(at 88.9 93.98 0)
 			(effects
@@
 			(project "Bluetooth Box V3"
 				(path "/c5f2915a-1379-46bf-9932-ae9df9d21574/08bbdc8c-2f8e-4da1-ab4d-f5452d4c4cd9"
-					(reference "#PWR062")
+					(reference "#PWR052")
 					(unit 1)
 				)
@@
 		(dnp no)
 		(fields_autoplaced yes)
-		(property "Reference" "C49"
+		(property "Reference" "C33"
 			(at 55.8799 50.8 0)
 			(effects
@@
 			(project "Bluetooth Box V3"
 				(path "/c5f2915a-1379-46bf-9932-ae9df9d21574/08bbdc8c-2f8e-4da1-ab4d-f5452d4c4cd9"
-					(reference "C49")
+					(reference "C33")
 					(unit 1)
 				)
@@
 		(dnp no)
 		(fields_autoplaced yes)
-		(property "Reference" "U10"
+		(property "Reference" "U6"
 			(at 88.9 69.85 0)
 			(effects
@@
 			(project "Bluetooth Box V3"
 				(path "/c5f2915a-1379-46bf-9932-ae9df9d21574/08bbdc8c-2f8e-4da1-ab4d-f5452d4c4cd9"
-					(reference "U10")
+					(reference "U6")
 					(unit 1)
 				)
@@
 		(on_board yes)
 		(dnp no)
-		(property "Reference" "C50"
+		(property "Reference" "C34"
 			(at 72.39 73.6662 0)
 			(effects
@@
 			(project ""
 				(path "/c5f2915a-1379-46bf-9932-ae9df9d21574/08bbdc8c-2f8e-4da1-ab4d-f5452d4c4cd9"
-					(reference "C50")
+					(reference "C34")
 					(unit 1)
 				)
@@
 		(dnp no)
 		(fields_autoplaced yes)
-		(property "Reference" "CR2"
+		(property "Reference" "CR1"
 			(at 86.36 44.45 0)
 			(effects
@@
 			(project "Bluetooth Box V3"
 				(path "/c5f2915a-1379-46bf-9932-ae9df9d21574/08bbdc8c-2f8e-4da1-ab4d-f5452d4c4cd9"
-					(reference "CR2")
+					(reference "CR1")
 					(unit 1)
 				)
@@
 		(dnp no)
 		(fields_autoplaced yes)
-		(property "Reference" "R12"
+		(property "Reference" "R19"
 			(at 64.77 87.63 90)
 			(effects
@@
 			(project "Bluetooth Box V3"
 				(path "/c5f2915a-1379-46bf-9932-ae9df9d21574/08bbdc8c-2f8e-4da1-ab4d-f5452d4c4cd9"
-					(reference "R12")
-					(unit 1)
-				)
+					(reference "R19")
+					(unit 1)
+				)

Commit message: Idiotencheck 1
Parts:
- removed C33: 22 uF, Capacitor_SMD:C_0805_2012Metric, symbol Device:C
- removed C36: 2.2 uF, Capacitor_SMD:C_0805_2012Metric, symbol Device:C_Small
- removed CR1: L4940D2T5-TR, ul_L4940D2T5-TR:D2PAK_STM, symbol 2026-02-19_20-19-44:L4940D2T5-TR
- removed R18, R19: 10 kΩ, Resistor_SMD:R_0805_2012Metric, symbol Device:R_Small
- removed U6: MIC5356-SGYMME, Package_SO:MSOP-8-1EP_3x3mm_P0.65mm_EP2.5x3mm_Mask1.73x2.36mm_ThermalVias, symbol Regulator_Linear:MIC5356-SGYMME
- added C31, C33: 10 uF, Capacitor_SMD:C_0805_2012Metric, symbol Device:C_Small
- added U8: AZ1117-3.3, Package_TO_SOT_SMD:TO-252-2, symbol Regulator_Linear:AZ1117-3.3
- added U9: NCP1117-1.8_SOT223, Package_TO_SOT_SMD:SOT-223-3_TabPin2, symbol Regulator_Linear:NCP1117-1.8_SOT223
- C34, C35: value 2.2 uF -> 10 uF; LCSC Part # C377773 -> C440198
Connections:
- net 1.8 V: now also C35.2, U9.2 (VO)
- net 3.3 V: now also C34.2, C33.2, U8.2 (VO), U9.3 (VI); no longer C35.1
- net 5 V: now also C31.2, U8.3 (VI); no longer C34.2
- net GND: now also C35.1, C31.1, C33.1, U8.1 (GND), U9.1 (GND); no longer C35.2

Commit message: First production
Parts:
- removed U9: NCP1117-1.8_SOT223, Package_TO_SOT_SMD:SOT-223-3_TabPin2, symbol Regulator_Linear:NCP1117-1.8_SOT223
- added U4: AMS1117-1.8, Package_TO_SOT_SMD:SOT-223-3_TabPin2, symbol Regulator_Linear:AMS1117-1.8
- U8: LCSC Part # (none) -> C362112
Connections:
- net 1.8 V: now also U4.2 (VO)
- net 3.3 V: now also U4.3 (VI)
- net GND: now also U4.1 (GND)
Changed lines of the file:
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@@
 	(paper "A4")
+	(junction
+		(at 102.87 77.47)
+		(diameter 0)
+		(color 0 0 0 0)
+	)
 	(junction
 		(at 82.55 77.47)
@@
 	(junction
 		(at 92.71 77.47)
-		(diameter 0)
-		(color 0 0 0 0)
-	)
-	(junction
-		(at 102.87 77.47)
 		(diameter 0)
 		(color 0 0 0 0)
@@
 			)
 		)
+		(property "LCSC Part #" "C362112"
+			(at 74.93 77.47 0)
+			(effects
+				(font
+					(size 1.27 1.27)
+				)
+				(hide yes)
+			)
+		)
 		(pin "2"
 		)
@@
 	)
 	(symbol
-		(lib_id "Regulator_Linear:NCP1117-1.8_SOT223")
+		(lib_id "Regulator_Linear:AMS1117-1.8")
 		(at 110.49 77.47 0)
 		(unit 1)
@@
 		(dnp no)
 		(fields_autoplaced yes)
-		(property "Reference" "U9"
+		(property "Reference" "U4"
 			(at 110.49 71.12 0)
 			(effects
@@
 			)
 		)
-		(property "Value" "NCP1117-1.8_SOT223"
+		(property "Value" "AMS1117-1.8"
 			(at 110.49 73.66 0)
 			(effects
@@
 			)
 		)
-		(property "Datasheet" "http://www.onsemi.com/pub_link/Collateral/NCP1117-D.PDF"
+		(property "Datasheet" "http://www.advanced-monolithic.com/pdf/ds1117.pdf"
 			(at 113.03 83.82 0)
 			(effects
@@
 			)
 		)
-		(property "Description" "1A Low drop-out regulator, Fixed Output 1.8V, SOT-223"
+		(property "Description" "1A Low Dropout regulator, positive, 1.8V fixed output, SOT-223"
 			(at 110.49 77.47 0)
 			(effects
@@
 			)
 		)
+		(property "LCSC Part #" "C46473009"
+			(at 110.49 77.47 0)
+			(effects
+				(font
+					(size 1.27 1.27)
+				)
+				(hide yes)
+			)
+		)
 		(pin "3"
 		)
@@
 			(project ""
 				(path "/c5f2915a-1379-46bf-9932-ae9df9d21574/08bbdc8c-2f8e-4da1-ab4d-f5452d4c4cd9"
-					(reference "U9")
-					(unit 1)
-				)
+					(reference "U4")
+					(unit 1)
+				)
