File: Bluetooth Box V3/active_dac_output_filter.kicad_sch (KiCad schematic)
At the start: 9 parts, among them U4 AD8606ARM

Commit message: started pcb routing
Parts:
- renumbered C18 to C4, C19 to C5, C21 to C6, C24 to C7, R16 to R10, R13 to R7, R14 to R8, R15 to R9, U4 to U3
Changed lines of the file:
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@@
 		(dnp no)
 		(fields_autoplaced yes)
-		(property "Reference" "#PWR038"
+		(property "Reference" "#PWR033"
 			(at 142.24 99.06 0)
 			(effects
@@
 			(project "Bluetooth Box V3"
 				(path "/c5f2915a-1379-46bf-9932-ae9df9d21574/55e88474-986a-4b71-810c-88147fedcdc0"
-					(reference "#PWR038")
-					(unit 1)
-				)
-				(path "/c5f2915a-1379-46bf-9932-ae9df9d21574/f9e0ecb5-3163-4072-a4b4-f0759403d588"
-					(reference "#PWR041")
+					(reference "#PWR033")
+					(unit 1)
+				)
+				(path "/c5f2915a-1379-46bf-9932-ae9df9d21574/f9e0ecb5-3163-4072-a4b4-f0759403d588"
+					(reference "#PWR035")
 					(unit 1)
 				)
@@
 		(dnp no)
 		(fields_autoplaced yes)
-		(property "Reference" "#PWR040"
+		(property "Reference" "#PWR034"
 			(at 180.34 92.71 0)
 			(effects
@@
 			(project "Bluetooth Box V3"
 				(path "/c5f2915a-1379-46bf-9932-ae9df9d21574/55e88474-986a-4b71-810c-88147fedcdc0"
-					(reference "#PWR040")
-					(unit 1)
-				)
-				(path "/c5f2915a-1379-46bf-9932-ae9df9d21574/f9e0ecb5-3163-4072-a4b4-f0759403d588"
-					(reference "#PWR066")
+					(reference "#PWR034")
+					(unit 1)
+				)
+				(path "/c5f2915a-1379-46bf-9932-ae9df9d21574/f9e0ecb5-3163-4072-a4b4-f0759403d588"
+					(reference "#PWR036")
 					(unit 1)
 				)
@@
 		(dnp no)
 		(fields_autoplaced yes)
-		(property "Reference" "U4"
+		(property "Reference" "U3"
 			(at 152.4 68.58 0)
 			(effects
@@
 			(project "Bluetooth Box V3"
 				(path "/c5f2915a-1379-46bf-9932-ae9df9d21574/55e88474-986a-4b71-810c-88147fedcdc0"
+					(reference "U3")
+					(unit 1)
+				)
+				(path "/c5f2915a-1379-46bf-9932-ae9df9d21574/f9e0ecb5-3163-4072-a4b4-f0759403d588"
 					(reference "U4")
-					(unit 1)
-				)
-				(path "/c5f2915a-1379-46bf-9932-ae9df9d21574/f9e0ecb5-3163-4072-a4b4-f0759403d588"
-					(reference "U7")
 					(unit 1)
 				)
@@
 		(dnp no)
 		(fields_autoplaced yes)
-		(property "Reference" "C18"
+		(property "Reference" "C4"
 			(at 146.05 87.6299 0)
 			(effects
@@
 			(project "Bluetooth Box V3"
 				(path "/c5f2915a-1379-46bf-9932-ae9df9d21574/55e88474-986a-4b71-810c-88147fedcdc0"
-					(reference "C18")
-					(unit 1)
-				)
-				(path "/c5f2915a-1379-46bf-9932-ae9df9d21574/f9e0ecb5-3163-4072-a4b4-f0759403d588"
-					(reference "C25")
+					(reference "C4")
+					(unit 1)
+				)
+				(path "/c5f2915a-1379-46bf-9932-ae9df9d21574/f9e0ecb5-3163-4072-a4b4-f0759403d588"
+					(reference "C8")
 					(unit 1)
 				)
@@
 		(dnp no)
 		(fields_autoplaced yes)
-		(property "Reference" "R16"
+		(property "Reference" "R10"
 			(at 182.88 81.2799 0)
 			(effects
@@
 			(project "Bluetooth Box V3"
 				(path "/c5f2915a-1379-46bf-9932-ae9df9d21574/55e88474-986a-4b71-810c-88147fedcdc0"
-					(reference "R16")
-					(unit 1)
-				)
-				(path "/c5f2915a-1379-46bf-9932-ae9df9d21574/f9e0ecb5-3163-4072-a4b4-f0759403d588"
-					(reference "R20")
+					(reference "R10")
+					(unit 1)
+				)
+				(path "/c5f2915a-1379-46bf-9932-ae9df9d21574/f9e0ecb5-3163-4072-a4b4-f0759403d588"
+					(reference "R14")
 					(unit 1)
 				)
@@
 		(dnp no)
 		(fields_autoplaced yes)
-		(property "Reference" "R14"
+		(property "Reference" "R8"
 			(at 137.1599 73.66 0)
 			(effects
@@
 			(project "Bluetooth Box V3"
 				(path "/c5f2915a-1379-46bf-9932-ae9df9d21574/55e88474-986a-4b71-810c-88147fedcdc0"
-					(reference "R14")
-					(unit 1)
-				)
-				(path "/c5f2915a-1379-46bf-9932-ae9df9d21574/f9e0ecb5-3163-4072-a4b4-f0759403d588"
-					(reference "R18")
+					(reference "R8")
+					(unit 1)
+				)
+				(path "/c5f2915a-1379-46bf-9932-ae9df9d21574/f9e0ecb5-3163-4072-a4b4-f0759403d588"
+					(reference "R12")
 					(unit 1)
 				)
@@
 		(dnp no)
 		(fields_autoplaced yes)
-		(property "Reference" "C21"
+		(property "Reference" "C6"
 			(at 161.6709 74.93 0)
 			(effects
@@
 			(project "Bluetooth Box V3"
 				(path "/c5f2915a-1379-46bf-9932-ae9df9d21574/55e88474-986a-4b71-810c-88147fedcdc0"
-					(reference "C21")
-					(unit 1)
-				)
-				(path "/c5f2915a-1379-46bf-9932-ae9df9d21574/f9e0ecb5-3163-4072-a4b4-f0759403d588"
-					(reference "C27")
+					(reference "C6")
+					(unit 1)
+				)
+				(path "/c5f2915a-1379-46bf-9932-ae9df9d21574/f9e0ecb5-3163-4072-a4b4-f0759403d588"
+					(reference "C10")
 					(unit 1)
 				)
@@
 		(dnp no)
 		(fields_autoplaced yes)
-		(property "Reference" "R15"
+		(property "Reference" "R9"
 			(at 170.1799 76.2 0)
 			(effects
@@
 			(project "Bluetooth Box V3"
 				(path "/c5f2915a-1379-46bf-9932-ae9df9d21574/55e88474-986a-4b71-810c-88147fedcdc0"
-					(reference "R15")
-					(unit 1)
-				)
-				(path "/c5f2915a-1379-46bf-9932-ae9df9d21574/f9e0ecb5-3163-4072-a4b4-f0759403d588"
-					(reference "R19")
+					(reference "R9")
+					(unit 1)
+				)
+				(path "/c5f2915a-1379-46bf-9932-ae9df9d21574/f9e0ecb5-3163-4072-a4b4-f0759403d588"
+					(reference "R13")
 					(unit 1)
 				)
@@
 		(dnp no)
 		(fields_autoplaced yes)
-		(property "Reference" "C19"
+		(property "Reference" "C5"
 			(at 151.1299 60.96 0)
 			(effects
@@
 			(project "Bluetooth Box V3"
 				(path "/c5f2915a-1379-46bf-9932-ae9df9d21574/55e88474-986a-4b71-810c-88147fedcdc0"
-					(reference "C19")
-					(unit 1)
-				)
-				(path "/c5f2915a-1379-46bf-9932-ae9df9d21574/f9e0ecb5-3163-4072-a4b4-f0759403d588"
-					(reference "C26")
+					(reference "C5")
+					(unit 1)
+				)
+				(path "/c5f2915a-1379-46bf-9932-ae9df9d21574/f9e0ecb5-3163-4072-a4b4-f0759403d588"
+					(reference "C9")
 					(unit 1)
 				)
@@
 		(dnp no)
 		(fields_autoplaced yes)
-		(property "Reference" "R13"
+		(property "Reference" "R7"
 			(at 129.5399 73.66 0)
 			(effects
@@
 			(project "Bluetooth Box V3"
 				(path "/c5f2915a-1379-46bf-9932-ae9df9d21574/55e88474-986a-4b71-810c-88147fedcdc0"
-					(reference "R13")
-					(unit 1)
-				)
-				(path "/c5f2915a-1379-46bf-9932-ae9df9d21574/f9e0ecb5-3163-4072-a4b4-f0759403d588"
-					(reference "R17")
+					(reference "R7")
+					(unit 1)
+				)
+				(path "/c5f2915a-1379-46bf-9932-ae9df9d21574/f9e0ecb5-3163-4072-a4b4-f0759403d588"
+					(reference "R11")
 					(unit 1)
 				)
@@
 		(dnp no)
 		(fields_autoplaced yes)
-		(property "Reference" "C24"
+		(property "Reference" "C7"
 			(at 171.45 81.2799 0)
 			(effects
@@
 			(project "Bluetooth Box V3"
 				(path "/c5f2915a-1379-46bf-9932-ae9df9d21574/55e88474-986a-4b71-810c-88147fedcdc0"
-					(reference "C24")
-					(unit 1)
-				)
-				(path "/c5f2915a-1379-46bf-9932-ae9df9d21574/f9e0ecb5-3163-4072-a4b4-f0759403d588"
-					(reference "C48")
-					(unit 1)
-				)
+					(reference "C7")
+					(unit 1)
+				)
+				(path "/c5f2915a-1379-46bf-9932-ae9df9d21574/f9e0ecb5-3163-4072-a4b4-f0759403d588"
+					(reference "C11")
+					(unit 1)
+				)

Commit message: Aux In gefixt
Parts:
- C4: footprint Capacitor_SMD:C_0201_0603Metric -> Capacitor_SMD:C_0603_1608Metric_Pad1.08x0.95mm_HandSolder
Changed lines of the file:
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@@
 			)
 		)
-		(property "Footprint" "Capacitor_SMD:C_0201_0603Metric"
+		(property "Footprint" "Capacitor_SMD:C_0603_1608Metric_Pad1.08x0.95mm_HandSolder"
 			(at 143.2052 92.71 0)
 			(effects

Commit message: Idiotencheck 1
Parts:
- U3: LCSC Part # (none) -> C459905
Changed lines of the file:
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@@
+			)
+		)
+		(property "LCSC Part #" "C459905"
+			(at 152.4 78.74 0)
+			(effects
+				(font
+					(size 1.27 1.27)
+				)
+				(hide yes)
 			)
 		)
@@
 				)
 				(path "/c5f2915a-1379-46bf-9932-ae9df9d21574/f9e0ecb5-3163-4072-a4b4-f0759403d588"
-					(reference "U4")
-					(unit 1)
+					(reference "U3")
+					(unit 2)
 				)
 			)
