File: Bluetooth Box V3/Bluetooth Box V3.kicad_pcb (KiCad board)
At the start: 2 copper layers, 64.5 x 74.8 mm, 121 parts, among them IC1 PAM8620TR, J1 USB_C_Receptacle_USB2.0, J10 GND, J2 5V Screw, J3 GND, J4 GND, J5 12V Screw, J7 Woofer, J8 Tweeter, SW1 BOOT, SW2 EN, U2 PCM1862DBT, U3 AD8606ARM, U4 AMS1117-1.8, U5 ESP32-WROOM-32E-R2, U6 CH340G, U7 ADAU1701, U8 AZ1117-3.3, Y1 Crystal_GND24, Y2 Crystal_GND24, Y3 12 MHz

Commit message: Ach basti
Routing:
- net +3V3: track 248.2 -> 250.1 mm
Changed lines of the file:
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@@
+	)
+	(segment
+		(start 75 58.3)
+		(end 75 57.39)
+		(width 0.2)
+		(layer "F.Cu")
+		(net "+3V3")
 	)
 	(segment
@@
 	)
 	(segment
+		(start 78.854448 52.83)
+		(end 79.2 52.83)
+		(width 0.2)
+		(layer "F.Cu")
+		(net "+3V3")
+	)
+	(segment
 		(start 110 97.5)
 		(end 115.25 97.5)
@@
 	)
 	(segment
+		(start 88.40741 91.5)
+		(end 90.5 93.59259)
+		(width 0.2)
+		(layer "F.Cu")
+		(net "+3V3")
+	)
+	(segment
+		(start 75 57.39)
+		(end 74.25 56.64)
+		(width 0.2)
+		(layer "F.Cu")
+		(net "+3V3")
+	)
+	(segment
+		(start 74.9 81.95)
+		(end 75.45 82.5)
+		(width 0.2)
+		(layer "F.Cu")
+		(net "+3V3")
+	)
+	(segment
+		(start 108.75 96.25)
+		(end 110 97.5)
+		(width 0.2)
+		(layer "F.Cu")
+		(net "+3V3")
+	)
+	(segment
+		(start 103 40.3375)
+		(end 94.6625 40.3375)
+		(width 0.2)
+		(layer "F.Cu")
+		(net "+3V3")
+	)
+	(segment
+		(start 85.600735 88.5)
+		(end 87.6375 88.5)
+		(width 0.2)
+		(layer "F.Cu")
+		(net "+3V3")
+	)
+	(segment
+		(start 115.25 97.5)
+		(end 115.5 97.25)
+		(width 0.2)
+		(layer "F.Cu")
+		(net "+3V3")
+	)
+	(segment
+		(start 93.4125 82.75)
+		(end 95.5 84.8375)
+		(width 0.2)
+		(layer "F.Cu")
+		(net "+3V3")
+	)
+	(segment
+		(start 85.05 41.9)
+		(end 85.05 37.72)
+		(width 0.2)
+		(layer "F.Cu")
+		(net "+3V3")
+	)
+	(segment
+		(start 75.82 78.95)
+		(end 92.2 78.95)
+		(width 0.2)
+		(layer "F.Cu")
+		(net "+3V3")
+	)
+	(segment
+		(start 108.25 85.35741)
+		(end 108.89259 86)
+		(width 0.2)
+		(layer "F.Cu")
+		(net "+3V3")
+	)
+	(segment
+		(start 98.5875 73.8375)
+		(end 98.5875 75.75)
+		(width 0.2)
+		(layer "F.Cu")
+		(net "+3V3")
+	)
+	(segment
+		(start 74.9 80.4)
+		(end 74.9 79.87)
+		(width 0.2)
+		(layer "F.Cu")
+		(net "+3V3")
+	)
+	(segment
+		(start 94.5 81.25)
+		(end 95.3406 81.25)
+		(width 0.2)
+		(layer "F.Cu")
+		(net "+3V3")
+	)
+	(segment
+		(start 90.5 95.3)
+		(end 92.5 95.3)
+		(width 0.2)
+		(layer "F.Cu")
+		(net "+3V3")
+	)
+	(segment
+		(start 75.044448 56.64)
+		(end 78.854448 52.83)
+		(width 0.2)
+		(layer "F.Cu")
+		(net "+3V3")
+	)
+	(segment
+		(start 88.40741 88.5)
+		(end 90.2 90.29259)
+		(width 0.2)
+		(layer "F.Cu")
+		(net "+3V3")
+	)
+	(segment
+		(start 98.5 73.75)
+		(end 100.25 73.75)
+		(width 0.2)
+		(layer "F.Cu")
+		(net "+3V3")
+	)
+	(segment
+		(start 81.58 52.83)
+		(end 82.5 53.75)
+		(width 0.2)
+		(layer "F.Cu")
+		(net "+3V3")
+	)
+	(segment
+		(start 92.5 95.3)
+		(end 94.5 95.3)
+		(width 0.2)
+		(layer "F.Cu")
+		(net "+3V3")
+	)
+	(segment
+		(start 82.5 53.75)
+		(end 85.2 53.75)
+		(width 0.2)
+		(layer "F.Cu")
+		(net "+3V3")
+	)
+	(segment
+		(start 87.6375 91)
+		(end 90.2 91)
+		(width 0.2)
+		(layer "F.Cu")
+		(net "+3V3")
+	)
+	(segment
+		(start 87.6375 91.5)
+		(end 88.40741 91.5)
+		(width 0.2)
+		(layer "F.Cu")
+		(net "+3V3")
+	)
+	(segment
+		(start 115.1625 86)
+		(end 116.8 86)
+		(width 0.2)
+		(layer "F.Cu")
+		(net "+3V3")
+	)
+	(segment
+		(start 92.2 78.95)
+		(end 94.5 81.25)
+		(width 0.2)
+		(layer "F.Cu")
+		(net "+3V3")
+	)
+	(segment
+		(start 74.9 80.4)
+		(end 74.9 81.95)
+		(width 0.2)
+		(layer "F.Cu")
+		(net "+3V3")
+	)
+	(segment
 		(start 74.25 56.64)
 		(end 75.044448 56.64)
 		(width 0.2)
 		(layer "F.Cu")
-		(net "+3V3")
-	)
-	(segment
-		(start 88.40741 91.5)
-		(end 90.5 93.59259)
-		(width 0.2)
-		(layer "F.Cu")
-		(net "+3V3")
-	)
-	(segment
-		(start 74.9 81.95)
-		(end 75.45 82.5)
-		(width 0.2)
-		(layer "F.Cu")
-		(net "+3V3")
-	)
-	(segment
-		(start 108.75 96.25)
-		(end 110 97.5)
-		(width 0.2)
-		(layer "F.Cu")
-		(net "+3V3")
-	)
-	(segment
-		(start 103 40.3375)
-		(end 94.6625 40.3375)
-		(width 0.2)
-		(layer "F.Cu")
-		(net "+3V3")
-	)
-	(segment
-		(start 85.600735 88.5)
-		(end 87.6375 88.5)
-		(width 0.2)
-		(layer "F.Cu")
-		(net "+3V3")
-	)
-	(segment
-		(start 115.25 97.5)
-		(end 115.5 97.25)
-		(width 0.2)
-		(layer "F.Cu")
-		(net "+3V3")
-	)
-	(segment
-		(start 93.4125 82.75)
-		(end 95.5 84.8375)
-		(width 0.2)
-		(layer "F.Cu")
-		(net "+3V3")
-	)
-	(segment
-		(start 85.05 41.9)
-		(end 85.05 37.72)
-		(width 0.2)
-		(layer "F.Cu")
-		(net "+3V3")
-	)
-	(segment
-		(start 78.854448 52.83)
-		(end 79.2 52.83)
-		(width 0.2)
-		(layer "F.Cu")
-		(net "+3V3")
-	)
-	(segment
-		(start 75.82 78.95)
-		(end 92.2 78.95)
-		(width 0.2)
-		(layer "F.Cu")
-		(net "+3V3")
-	)
-	(segment
-		(start 108.25 85.35741)
-		(end 108.89259 86)
-		(width 0.2)
-		(layer "F.Cu")
-		(net "+3V3")
-	)
-	(segment
-		(start 98.5875 73.8375)
-		(end 98.5875 75.75)
-		(width 0.2)
-		(layer "F.Cu")
-		(net "+3V3")
-	)
-	(segment
-		(start 74.9 80.4)
-		(end 74.9 79.87)
-		(width 0.2)
-		(layer "F.Cu")
-		(net "+3V3")
-	)
-	(segment
-		(start 75.044448 56.64)
-		(end 78.854448 52.83)
-		(width 0.2)
-		(layer "F.Cu")
-		(net "+3V3")
-	)
-	(segment
-		(start 94.5 81.25)
-		(end 95.3406 81.25)
-		(width 0.2)
-		(layer "F.Cu")
-		(net "+3V3")
-	)
-	(segment
-		(start 90.5 95.3)
-		(end 92.5 95.3)
-		(width 0.2)
-		(layer "F.Cu")
-		(net "+3V3")
-	)
-	(segment
-		(start 88.40741 88.5)
-		(end 90.2 90.29259)
-		(width 0.2)
-		(layer "F.Cu")
-		(net "+3V3")
-	)
-	(segment
-		(start 98.5 73.75)
-		(end 100.25 73.75)
-		(width 0.2)
-		(layer "F.Cu")
-		(net "+3V3")
-	)
-	(segment
-		(start 81.58 52.83)
-		(end 82.5 53.75)
-		(width 0.2)
-		(layer "F.Cu")
-		(net "+3V3")
-	)
-	(segment
-		(start 92.5 95.3)
-		(end 94.5 95.3)
-		(width 0.2)
-		(layer "F.Cu")
-		(net "+3V3")
-	)
-	(segment
-		(start 82.5 53.75)
-		(end 85.2 53.75)
-		(width 0.2)
-		(layer "F.Cu")
-		(net "+3V3")
-	)
-	(segment
-		(start 87.6375 91)
-		(end 90.2 91)
-		(width 0.2)
-		(layer "F.Cu")
-		(net "+3V3")
-	)
-	(segment
-		(start 87.6375 91.5)
-		(end 88.40741 91.5)
-		(width 0.2)
-		(layer "F.Cu")
-		(net "+3V3")
-	)
-	(segment
-		(start 115.1625 86)
-		(end 116.8 86)
-		(width 0.2)
-		(layer "F.Cu")
-		(net "+3V3")
-	)
-	(segment
-		(start 92.2 78.95)
-		(end 94.5 81.25)
-		(width 0.2)
-		(layer "F.Cu")
-		(net "+3V3")
-	)
-	(segment
-		(start 74.9 80.4)
-		(end 74.9 81.95)
-		(width 0.2)
-		(layer "F.Cu")

Commit message: Grrr basti, grrr
Parts:
- removed S1: SSSS811101, footprints:SSSS811101
- added Q1: SS8050, Package_TO_SOT_SMD:SOT-23, F.Cu at (90.4, 56.3)
- added R16: 10k Ohm, Resistor_SMD:R_0805_2012Metric, F.Cu at (87.3, 58.8)
- added R17: 4.7k, Resistor_SMD:R_0603_1608Metric, F.Cu at (93.3, 59.9)
- added R6: 10k Ohm, Resistor_SMD:R_0805_2012Metric, F.Cu at (87.4, 55.2)
- added SS8050: NPN, Package_TO_SOT_SMD:SOT-23, F.Cu at (90.4, 59.9)
- R5: value 10k -> 0 ohm
- moved TP6 4.32 mm to (79.7, 60.0)
- moved TP7 3.60 mm to (82.5, 50.1)
Connections:
- U5 pad 25: /BOOTMODE -> /GPIO0
- U5 pad 34: /RX -> /TX_OUT
- U5 pad 35: /TX -> /RX_IN
- U6 pad 13: unconnected-(U6-~{DTR}-Pad13) -> /UART/DTR
- U6 pad 14: unconnected-(U6-~{RTS}-Pad14) -> /UART/RTS
- U6 pad 2: /TX -> /TX_OUT
- U6 pad 3: /RX -> /RX_IN
Routing:
- net Net-(Q1-C): track 9.86 -> 41.1 mm, vias 0 -> 2
- net /UART/DTR: track 0.00 -> 22.2 mm, vias 0 -> 3
- net /UART/RTS: track 0.00 -> 18.9 mm, vias 0 -> 2
- net /RX: track 10.6 -> 0.00 mm
- net /RX_IN: track 0.00 -> 9.73 mm
- net /TX_OUT: track 0.00 -> 8.98 mm
- net /TX: track 8.83 -> 0.00 mm
- net /GPIO0: track 0.00 -> 4.58 mm
- net +3V3: track 250.1 -> 254.6 mm
- net Net-(Q1-B): track 0.00 -> 4.36 mm
- net Net-(SS8050-B): track 0.00 -> 4.32 mm
- net /BOOTMODE: track 4.08 -> 0.00 mm
- net Net-(R26-Pad1): track 2.34 -> 3.23 mm
- net GND: vias 53 -> 52
Other:
- board text removed: "BOOTMODE"

Commit message: Try fixes
Parts:
- removed R5: 0 ohm, Resistor_SMD:R_0805_2012Metric
- added C16: 1 uF, Capacitor_SMD:C_0603_1608Metric, F.Cu at (83.0, 56.8)
- added R30: 10k Ohm, Resistor_SMD:R_0805_2012Metric, F.Cu at (78.0, 82.5)
- added SW3: KH-6X6X5H-STM, footprints:KH-6X6X5H-STM_SKE, F.Cu at (76.0, 89.1)
- R17: value 4.7k -> 10k Ohm; footprint Resistor_SMD:R_0603_1608Metric -> Resistor_SMD:R_0805_2012Metric
- SW2: value EN -> KH-6X6X5H-STM
- moved SW2 58.5 mm to (92.8, 33.0), turned to -90 degrees
- moved R17 23.0 mm to (98.2, 37.5), turned to 0 degrees
- moved R16 1.18 mm to (88.3, 59.5)
- moved Q1 1.14 mm to (91.5, 56.0), turned to 0 degrees
- moved SS8050 1.13 mm to (91.5, 59.6), turned to 0 degrees
- moved R6 1.11 mm to (88.3, 55.9), turned to -90 degrees
Connections:
- net /UART/DTR renamed Net-(SS8050-E)
- net /UART/RTS renamed Net-(Q1-E)
- Q1 pad 1: Net-(Q1-C) -> /EN
- R17 pad 1: +3V3 -> Net-(R17-Pad1)
- R17 pad 2: /GPIO0 -> +3V3
- SW2 pad A: unconnected-(SW2-PadA) -> Net-(R17-Pad1)
- SW2 pad B: Net-(Q1-C) -> Net-(R17-Pad1)
- SW2 pad C: GND -> /EN
- SW2 pad D: unconnected-(SW2-PadD) -> /EN
- U5 pad 11: unconnected-(U5-IO26-Pad11) -> /SCL
- U5 pad 14: /SCL -> GND
- U5 pad 23: /I2S_LRCLK -> +3V3
- U5 pad 29: unconnected-(U5-IO5-Pad29) -> +3V3
- U5 pad 3: Net-(Q1-C) -> /EN
- U5 pad 37: unconnected-(U5-IO23-Pad37) -> /I2S_LRCLK
Routing:
- net /EN: track 0.00 -> 63.7 mm, vias 0 -> 6
- net Net-(Q1-C): track 41.1 -> 0.00 mm, vias 2 -> 0
- net /GPIO0: track 4.58 -> 40.6 mm, vias 0 -> 2
- net /I2S_LRCLK: track 48.1 -> 63.4 mm
- net +3V3: track 254.6 -> 269.8 mm
- net Net-(R30-Pad1): track 0.00 -> 15.0 mm
- net Net-(R17-Pad1): track 0.00 -> 11.2 mm
- net Net-(Q1-E): track 18.9 -> 23.7 mm
- net Net-(SS8050-E): track 22.2 -> 26.5 mm
- net /SCL: track 35.5 -> 38.5 mm, vias 2 -> 4
- net Net-(Q1-B): track 4.36 -> 2.32 mm, vias 0 -> 2
- net Net-(SS8050-B): track 4.32 -> 2.32 mm, vias 0 -> 2
- net GND: track 100.3 -> 98.3 mm, vias 52 -> 62
Other:
- board text removed: "+"
- board text removed: "-"
- board text removed: "12V"
- board text removed: "Reboot"
- board text removed: "Tweeter"
- board text removed: "Woofer"

Commit message: yarr
Parts:
- moved R17 15.2 mm to (88.1, 26.1)
- moved SW2 6.26 mm to (87.0, 30.5), turned to 0 degrees
Connections:
- IC1 pad 16: GNDA -> GND
- IC1 pad 20: GNDA -> GND
- IC1 pad 25: GNDA -> GND
- IC1 pad 32: GNDA -> GND
- IC1 pad 9: GNDA -> GND
- J4 pad 1: GNDA -> GND
- J5 pad 2: GNDA -> GND
Routing:
- net +3V3: track 269.8 -> 395.8 mm, vias 20 -> 0
- net GND: track 98.3 -> 0.00 mm, vias 62 -> 123
- net GNDA: track 36.9 -> 0.00 mm, vias 5 -> 0
- net /Amplifier/LOUTN: track 9.54 -> 23.6 mm, vias 0 -> 2
- net +1V8: track 24.5 -> 35.8 mm, vias 0 -> 2
- net /Amplifier/LOUTP: track 15.0 -> 25.1 mm
- net /Amplifier/ROUTP: track 9.49 -> 19.0 mm
- net +5V: track 39.8 -> 32.3 mm, vias 0 -> 2
- net /I2S_LRCLK: track 63.4 -> 56.3 mm, vias 3 -> 4
- net D+: track 21.3 -> 27.3 mm, vias 2 -> 0
- net /Amplifier/ROUTN: track 14.7 -> 20.1 mm
- net D-: track 22.0 -> 27.3 mm, vias 2 -> 0
- net /AUX_I2S_DATA: track 18.8 -> 13.7 mm
- net /BT_I2S_DATA: track 34.2 -> 29.4 mm
- net Net-(SS8050-E): track 26.5 -> 22.2 mm, vias 3 -> 2
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
Commit message: fj
Parts:
- added C81: 100 nF, Capacitor_SMD:C_0805_2012Metric, F.Cu at (85.3, 60.0)
- added C82: 100 nF, Capacitor_SMD:C_0805_2012Metric, F.Cu at (74.8, 60.6)
- moved C80 0.74 mm to (74.8, 58.5), turned to 0 degrees
Routing:
- net +3V3: track 395.8 -> 365.4 mm
- net GND: track 0.00 -> 13.8 mm, vias 123 -> 136

Commit message: 4 layer
Parts:
- moved C82 0.10 mm to (74.8, 60.7)
Routing:
- net +3V3: track 365.4 -> 319.3 mm
- net +12V: track 64.1 -> 71.4 mm, vias 4 -> 2
- net Net-(U2-VINL1/VIN1P): track 5.57 -> 12.7 mm, vias 2 -> 0
- net Net-(SS8050-B): track 2.89 -> 8.21 mm, vias 2 -> 0
- net /AUX_I2S_DATA: track 13.7 -> 18.3 mm
- net GND: track 13.8 -> 9.21 mm, vias 136 -> 172
- net /I2S_BCLK: track 34.0 -> 30.4 mm, vias 2 -> 3
- net D+: track 27.3 -> 24.4 mm
- net D-: track 27.3 -> 24.4 mm
- net Net-(IC1-RINP): track 9.26 -> 6.33 mm, vias 0 -> 2
- net Net-(U2-VINR1/VIN2P): track 7.93 -> 5.96 mm
- net /SDA: track 34.2 -> 35.7 mm
- net Net-(U7-~{RESET}): track 7.41 -> 6.19 mm
- net /Amplifier/LOUTN: track 23.6 -> 24.8 mm, vias 2 -> 0
- net /GPIO0: track 42.0 -> 40.9 mm
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- added copper zone on In1.Cu, net GND
- added copper zone on In2.Cu, net GND
- removed copper zone on B.Cu, net GND
- removed copper zone on F.Cu, net GND
Other:
- copper layers 2 -> 4

Commit message: basti hat drueber geguckt
Routing:
- net +12V: track 71.4 -> 69.9 mm
- net /Amplifier/ROUTN: track 20.2 -> 19.5 mm
Other:
- board text added: "+"
- board text added: "-"
- board text added: "12V"
- board text added: "Bootmode"
- board text added: "Reset"
- board text added: "Tweeter"
- board text added: "Woofer"

Commit message: fja
Routing:
- net GND: track 9.21 -> 46.2 mm, vias 172 -> 152
- net Net-(J1-CC2): track 2.71 -> 29.9 mm
- net +12V: track 69.9 -> 90.0 mm, vias 2 -> 0
- net Net-(U2-VINR1/VIN2P): track 5.96 -> 18.3 mm, vias 2 -> 0
- net /SDA: track 35.7 -> 45.8 mm, vias 4 -> 3
- net /Mute: track 26.7 -> 35.7 mm
- net Net-(J1-CC1): track 3.47 -> 11.6 mm
- net +1V8: track 35.4 -> 27.5 mm, vias 2 -> 3
- net +3V3: track 319.3 -> 327.1 mm, vias 0 -> 2
- net +5V: track 33.0 -> 40.6 mm, vias 2 -> 0
- net /EN: track 66.5 -> 73.6 mm, vias 4 -> 3
- net /SCL: track 40.4 -> 47.3 mm, vias 4 -> 3
- net Net-(U7-FILTA): track 6.42 -> 13.2 mm, vias 0 -> 2
- net /Amplifier/LOUTN: track 24.8 -> 19.1 mm
- net /Amplifier/LOUTP: track 25.2 -> 19.5 mm
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