File: AMP/AMP-V1/AMP-V1.kicad_sch (KiCad schematic)
At the start: 83 parts, among them IC1 TPA3116D2QDADRQ1, J2 L, J3 R, J4 AudioJack3_SwitchTR, J5 R, U1 NE5532, U2 NE5532, U3 LM7812_TO220

Commit message: fj
Parts:
- added VR1, VR2: 3296W-1-103LF, footprints:TRIM_3296W-1-103LF, symbol Personal:3296W-1-103LF
- U3: footprint Package_TO_SOT_THT:TO-220-3_Vertical -> Package_TO_SOT_SMD:TO-263-2; LCSC Part # C2902509 -> C7432181
Connections:
- net GND: now also VR1.1, VR2.1
- net RING-RIGHT: now also VR2.2; no longer J4.R
- net TIP-LEFT: now also VR1.2; no longer J4.T
- new net: J4.T, VR1.3
- new net: J4.R, VR2.3

Commit message: Yarr
Parts:
- IC1: value TPA3116D2QDADRQ1 -> TPA3116D2DAD; LCSC Part # C2872892 -> C2865736; Manufacturer_Part_Number TPA3116D2QDADRQ1 -> TPA3116D2DAD
- J2, J3, J5: LCSC Part # (none) -> C8465
- J4: LCSC Part # (none) -> C4991610
Changed lines of the file:
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@@
 			)
 		)
+		(property "LCSC Part #" "C8465"
+			(at 57.15 68.58 0)
+			(effects
+				(font
+					(size 1.27 1.27)
+				)
+				(hide yes)
+			)
+		)
 		(pin "1"
 		)
@@
 			)
 		)
-		(property "Value" "TPA3116D2QDADRQ1"
+		(property "Value" "TPA3116D2DAD"
 			(at 190.5 66.04 0)
 			(effects
@@
 			)
 		)
-		(property "Manufacturer_Part_Number" "TPA3116D2QDADRQ1"
+		(property "Manufacturer_Part_Number" "TPA3116D2DAD"
 			(at 204.47 866.04 0)
 			(effects
@@
 			)
 		)
-		(property "LCSC Part #" "C2872892"
+		(property "LCSC Part #" "C2865736"
 			(at 172.72 71.12 0)
 			(effects
@@
 			)
 		)
+		(property "LCSC Part #" "C8465"
+			(at 300.99 99.06 0)
+			(effects
+				(font
+					(size 1.27 1.27)
+				)
+				(hide yes)
+			)
+		)
 		(pin "1"
 		)
@@
 			)
 		)
+		(property "LCSC Part #" "C8465"
+			(at 300.99 73.66 0)
+			(effects
+				(font
+					(size 1.27 1.27)
+				)
+				(hide yes)
+			)
+		)
 		(pin "1"
 		)
@@
 			(at 25.4 26.67 0)
 			(effects
+				(font
+					(size 1.27 1.27)
+				)
+				(hide yes)
+			)
+		)
+		(property "LCSC Part #" "C4991610"
+			(at 25.4 26.67 0)
+			(effects

Commit message: LPF
Parts:
- removed C1, C2, C3, C4: 22 pF, Capacitor_SMD:C_0603_1608Metric, symbol Device:C_Small
- removed C12, C46, C6, C7: 100nF, Capacitor_SMD:C_0603_1608Metric, symbol Device:C
- removed C15, C42: 47uF, Capacitor_SMD:C_1206_3216Metric, symbol Device:C
- removed C26, C44, C45: 470 uF, Capacitor_THT:CP_Radial_D12.5mm_P5.00mm, symbol Device:C_Polarized
- removed C40, C41, C5: 10uF, Capacitor_SMD:C_0603_1608Metric, symbol Device:C
- removed C43: 220 uF, Capacitor_SMD:C_0603_1608Metric, symbol Device:C
- removed D1: LED, LED_SMD:LED_0603_1608Metric, symbol Device:LED
- removed J5: R, footprints:WJ500V-5.08-2P, symbol Connector:Screw_Terminal_01x02
- removed L8: 10 uH, Inductor_SMD:L_0603_1608Metric, symbol Device:L
- removed R1, R10, R11, R12, R17, R2, R22, R3, R5, R6, R7: 10K, Resistor_SMD:R_0603_1608Metric, symbol Device:R_Small
- removed R20: 3.3 Ohm, Resistor_SMD:R_0603_1608Metric, symbol Device:R_Small
- removed R23: 2.2 Ohm, Resistor_SMD:R_0603_1608Metric, symbol Device:R_Small
- removed R4, R8: 100K, Resistor_SMD:R_0603_1608Metric, symbol Device:R_Small
- removed U1, U2: NE5532, Package_SO:SOIC-8_3.9x4.9mm_P1.27mm, symbol Amplifier_Operational:NE5532
- removed U3: LM7812_TO220, Package_TO_SOT_SMD:TO-263-2, symbol Regulator_Linear:LM7812_TO220
Connections:
- net GND: no longer VR1.1, VR2.1
- no-connect marks 3 -> 5
Other:
- added sheet LR-Decode (lr-decode.kicad_sch)
- added sheet power (power.kicad_sch)
- moved on the sheet: C10, C11, C13, C14, C16, C17, C18, C19, C20, C21, C22, C23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
