File: FM-Radios/FM-Radio-v1/FM-Radio.kicad_pcb (KiCad board)
At the start: 2 copper layers, 50 x 57 mm, 60 parts, among them J1 L_OUT, J2 USB_C_Receptacle_USB2.0, J3 R_OUT, J4 VBUS, J5 GND, J6 BWSMA-KE-Z001, SW2 EN, U1 ESP32-S3-MINI-1U, U2 SI4702-C19-GMR, U4 PRTR5V0U2X, U5 TPS62160DSG, U6 PAM8406D, Y1 32.768 kHz

Commit message: fjaoiwe
Parts:
- added C27: 10uF, Capacitor_SMD:C_0603_1608Metric, F.Cu at (236.6, 101.7)
- added FB5: 120Ohm 2A, Resistor_SMD:R_0805_2012Metric, F.Cu at (242.2, 131.3)
- added J7: 3V3, Connector_PinHeader_2.54mm:PinHeader_1x01_P2.54mm_Vertical, F.Cu at (255.1, 137.7)
- added R14: 0 Ohm, Resistor_SMD:R_0603_1608Metric, F.Cu at (240.7, 111.7)
- moved U2 97.7 mm to (253.7, 113.6), turned to 0 degrees
- moved FB4 92.8 mm to (242.2, 128.3), turned to 0 degrees
- moved C15 89.9 mm to (245.5, 116.0), turned to 0 degrees
- moved FB1 88.7 mm to (242.2, 119.5)
- moved R11 88.3 mm to (240.7, 109.2), turned to 0 degrees
- moved U6 87.9 mm to (248.6, 132.1)
- moved J6 85.5 mm to (247.0, 110.0), turned to 0 degrees
- moved C26 84.9 mm to (236.6, 99.2)
- moved FB3 84.9 mm to (242.2, 125.4), turned to 0 degrees
- moved Y1 83.7 mm to (235.0, 136.6), turned to 0 degrees
- moved FB2 82.2 mm to (242.2, 122.4)
- moved J4 81.7 mm to (255.1, 128.5)
- moved C18 81.2 mm to (232.6, 99.2), turned to 0 degrees
- moved C19 81.1 mm to (232.6, 101.7), turned to 0 degrees
- moved R2 80.7 mm to (236.6, 106.7), turned to 0 degrees
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Connections:
- C26 pad 1: Net-(J3-Pin_1) -> Net-(J3-Pin_2)
- L1 pad 2: +3.3V -> Net-(U5-VOS)
- R1 pad 1: +3V3 -> +3.3V
- R10 pad 1: +3V3 -> +3.3V
- R22 pad 1: +3.3V -> Net-(U5-VOS)
- R3 pad 1: +3V3 -> +3.3V
- R5 pad 2: +3V3 -> +3.3V
- S1 pad 1: +3V3 -> +3.3V
- U1 pad 3: +3V3 -> +3.3V
- U2 pad 16: +5V -> Net-(U2-VA)
- U5 pad 6: +3.3V -> Net-(U5-VOS)
Routing:
- net +5V: track 78.8 -> 0.00 mm
- net +3.3V: track 74.4 -> 0.00 mm
- net +3V3: track 57.1 -> 0.00 mm, vias 2 -> 0
- net VBUS: track 37.8 -> 0.00 mm, vias 2 -> 0
- net /GPIO9: track 35.8 -> 0.00 mm, vias 2 -> 0
- net /GPIO8: track 31.6 -> 0.00 mm, vias 3 -> 0
- net Net-(J2-D--PadA7): track 30.6 -> 0.00 mm, vias 2 -> 0
- net /BOOTMODE: track 28.3 -> 0.00 mm
- net Net-(J2-D+-PadA6): track 27.6 -> 0.00 mm, vias 2 -> 0
- net /RST: track 24.2 -> 0.00 mm, vias 2 -> 0
- net Net-(U6--OUT_L): track 23.6 -> 0.00 mm, vias 2 -> 0
- net Net-(U6--OUT_R): track 18.6 -> 0.00 mm, vias 2 -> 0
- net Net-(J2-CC2): track 17.4 -> 0.00 mm
- net Net-(J1-Pin_1): track 17.0 -> 0.00 mm
- net Net-(U6-INL): track 16.1 -> 0.00 mm, vias 2 -> 0
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
Commit message: yarrr
Parts:
- removed J4: VBUS, Connector_PinHeader_2.54mm:PinHeader_1x01_P2.54mm_Vertical
- removed J7: 3V3, Connector_PinHeader_2.54mm:PinHeader_1x01_P2.54mm_Vertical
- removed L1: 2.2 uH, footprints:IND_PA4332.222NLT
- removed R12: 562kΩ, Resistor_SMD:R_0805_2012Metric
- removed R13: 180kΩ, Resistor_SMD:R_0805_2012Metric
- removed R14: 0 Ohm, Resistor_SMD:R_0603_1608Metric
- removed R22: 100k, Resistor_SMD:R_0603_1608Metric
- removed U5: TPS62160DSG, Package_SON:WSON-8-1EP_2x2mm_P0.5mm_EP0.9x1.6mm_ThermalVias
- added C28: 22 uF, Capacitor_SMD:C_0603_1608Metric, F.Cu at (101.7, 93.3)
- added IC1: TPS62160DGKR, footprints:SOP65P490X110-8N, F.Cu at (124.4, 91.8)
- added J8: 3V3, Connector_PinHeader_2.54mm:PinHeader_1x01_P2.54mm_Vertical, F.Cu at (123.8, 116.5)
- added J9: VBUS, Connector_PinHeader_2.54mm:PinHeader_1x01_P2.54mm_Vertical, F.Cu at (123.8, 121.1)
- added L2: 2.2 uH, footprints:IND_PA4332.222NLT, F.Cu at (108.2, 129.4)
- added R15: 100k, Resistor_SMD:R_0603_1608Metric, F.Cu at (105.7, 103.3)
- added R16: 562kΩ, Resistor_SMD:R_0805_2012Metric, F.Cu at (119.3, 125.8)
- added R17: 180kΩ, Resistor_SMD:R_0805_2012Metric, F.Cu at (119.3, 128.8)
- C24: value 22 uF -> 47uF; footprint Capacitor_SMD:C_0603_1608Metric -> Capacitor_SMD:C_1206_3216Metric
- moved C15 143.5 mm to (102.5, 128.2)
- moved U2 141.1 mm to (113.4, 128.8)
- moved SW2 139.6 mm to (114.4, 93.9)
- moved U6 139.6 mm to (111.9, 103.7)
- moved C26 139.3 mm to (97.7, 108.3)
- moved C25 135.4 mm to (97.7, 105.8)
- moved C27 135.4 mm to (101.7, 90.8)
- moved C1 135.2 mm to (89.7, 90.8)
- moved C10 135.2 mm to (93.7, 93.3)
- moved C11 135.2 mm to (93.7, 95.8)
- moved C12 135.2 mm to (93.7, 98.3)
- moved C13 135.2 mm to (93.7, 100.8)
- moved C14 135.2 mm to (93.7, 103.3)
- moved C16 135.2 mm to (93.7, 105.8)
- moved C17 135.2 mm to (93.7, 108.3)
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Other:
- board size 50 x 57 mm -> 45.1 x 57 mm

Commit message: yarrrr
Parts:
- moved R6 94.0 mm to (192.8, 85.3), turned to 90 degrees
- moved R5 92.2 mm to (192.8, 91.6), turned to 90 degrees
- moved R1 91.1 mm to (192.8, 96.5), turned to 90 degrees
- moved C13 89.3 mm to (182.2, 112.6), turned to 180 degrees
- moved R7 87.1 mm to (192.8, 88.4), turned to 90 degrees
- moved C19 86.4 mm to (172.3, 136.8)
- moved C4 86.2 mm to (172.7, 121.5)
- moved C2 85.0 mm to (172.7, 111.5)
- moved C5 84.8 mm to (174.0, 92.3), turned to 180 degrees
- moved C8 84.7 mm to (171.9, 88.4), turned to 90 degrees
- moved C1 84.5 mm to (174.0, 85.6), turned to 180 degrees
- moved R8 83.6 mm to (188.5, 104.3), turned to 180 degrees
- moved C24 83.3 mm to (174.1, 89.0), turned to 90 degrees
- moved R9 83.1 mm to (188.5, 102.6), turned to 180 degrees
- moved C6 81.6 mm to (170.2, 89.8), turned to -90 degrees
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Routing:
- net +3.3V: track 0.00 -> 166.4 mm
- net GND: track 0.00 -> 75.0 mm, vias 0 -> 72
- net Net-(J2-CC1): track 0.00 -> 30.9 mm, vias 0 -> 2
- net Net-(IC1-FB): track 0.00 -> 30.2 mm, vias 0 -> 2
- net Net-(U1-EN): track 0.00 -> 30.0 mm
- net /BOOTMODE: track 0.00 -> 27.7 mm, vias 0 -> 2
- net Net-(J2-CC2): track 0.00 -> 24.7 mm, vias 0 -> 2
- net Net-(J1-Pin_1): track 0.00 -> 23.9 mm
- net /GPIO8: track 0.00 -> 23.0 mm, vias 0 -> 3
- net +5V: track 0.00 -> 21.2 mm, vias 0 -> 19
- net /GPIO9: track 0.00 -> 20.8 mm, vias 0 -> 2
- net Net-(U6-INL): track 0.00 -> 20.6 mm
- net VBUS: track 0.00 -> 19.0 mm
- net Net-(U6-INR): track 0.00 -> 18.0 mm
- net /RST: track 0.00 -> 17.8 mm, vias 0 -> 2
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- added copper zone on In2.Cu, net +5V
- added copper zone on In1.Cu, net GND
- removed copper zone on B.Cu, net GND
- removed copper zone on F.Cu, net GND
Other:
- copper layers 2 -> 4

Commit message: Production v2 radio
Routing:
- net Net-(J2-D--PadA7): track 13.7 -> 11.2 mm
- net Net-(J2-CC2): track 24.7 -> 23.5 mm
- net Net-(J2-CC1): track 30.9 -> 31.9 mm, vias 2 -> 0

Commit message: Shenanigooner
Parts:
- removed C13, C14, C9: 100nF, Capacitor_SMD:C_0603_1608Metric
- removed R2: 10k Ohm, Resistor_SMD:R_0603_1608Metric
- removed U2: SI4702-C19-GMR, footprints:SI470X_20_QFN
- added C29: 100nF, Capacitor_SMD:C_0603_1608Metric, F.Cu at (175.3, 101.5)
- added IC2: SI4732-A10-GSR, footprints:SOIC127P600X175-16N, F.Cu at (168.2, 97.7)
- added J4: Conn_01x10_Pin, Connector_PinHeader_2.54mm:PinHeader_1x10_P2.54mm_Vertical, F.Cu at (170.0, 137.8)
- added J7: AM-ANT, footprints:BAT_WIRELESS_BWSMA-KE-Z001, F.Cu at (162.2, 88.4)
- added L3: 500 uH, Inductor_SMD:L_Taiyo-Yuden_NR-40xx_HandSoldering, F.Cu at (160.6, 95.7)
- C27: value 10uF -> 470 nF
- C8: value 100nF -> 680 uF; footprint Capacitor_SMD:C_0603_1608Metric -> Capacitor_THT:CP_Radial_D12.5mm_P5.00mm
- J6: value BWSMA-KE-Z001 -> FM-ANT
- moved J9 40.4 mm to (192.9, 101.2), turned to 0 degrees
- moved S1 38.8 mm to (162.2, 135.4)
- moved R16 36.3 mm to (188.1, 94.6)
- moved R17 34.7 mm to (188.1, 98.1), turned to -90 degrees
- moved C26 34.0 mm to (158.3, 102.4)
- moved C1 33.9 mm to (187.3, 116.8), turned to -90 degrees
- moved U1 33.8 mm to (186.6, 126.5), turned to -90 degrees
- moved C19 33.6 mm to (150.8, 111.0)
- moved C8 33.1 mm to (161.8, 120.0), turned to 0 degrees
- moved J8 32.6 mm to (192.9, 96.6), turned to 0 degrees
- moved R1 30.2 mm to (173.2, 119.4), turned to 0 degrees
- moved L2 29.7 mm to (184.6, 95.2), turned to 90 degrees
- moved R6 29.6 mm to (179.9, 112.0), turned to 0 degrees
- moved C5 29.6 mm to (190.6, 116.8), turned to 90 degrees
- moved R7 29.4 mm to (179.2, 114.5)
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Connections:
- C25 pad 2: Net-(U2-FMIP) -> /FMI
- C27 pad 1: GND -> Net-(C27-Pad1)
- C27 pad 2: Net-(U2-VA) -> /AMI
- C8 pad 1: +3.3V -> +5V
- FB5 pad 1: +5V -> +3.3V
- FB5 pad 2: Net-(U2-VA) -> +3.3VA
- SW2 pad A: unconnected-(SW2-PadA) -> Net-(U1-EN)
- SW2 pad D: unconnected-(SW2-PadD) -> GND
- U1 pad 25: unconnected-(U1-IO21-Pad25) -> Net-(J4-Pin_1)
- U1 pad 26: unconnected-(U1-IO26-Pad26) -> Net-(J4-Pin_2)
- U1 pad 28: unconnected-(U1-IO33-Pad28) -> Net-(J4-Pin_3)
- U1 pad 29: unconnected-(U1-IO34-Pad29) -> Net-(J4-Pin_4)
- U1 pad 31: unconnected-(U1-IO35-Pad31) -> Net-(J4-Pin_5)
- U1 pad 32: unconnected-(U1-IO36-Pad32) -> Net-(J4-Pin_6)
- U1 pad 33: unconnected-(U1-IO37-Pad33) -> Net-(J4-Pin_7)
- U1 pad 34: unconnected-(U1-IO38-Pad34) -> Net-(J4-Pin_8)
- U1 pad 35: unconnected-(U1-IO39-Pad35) -> Net-(J4-Pin_9)
- U1 pad 36: unconnected-(U1-IO40-Pad36) -> Net-(J4-Pin_10)
Routing:
- net GND: track 75.0 -> 0.00 mm, vias 72 -> 71
- net +3.3V: track 166.3 -> 103.9 mm, vias 0 -> 1
- net +5V: track 21.2 -> 83.2 mm, vias 19 -> 3
- net Net-(J2-CC1): track 31.9 -> 10.5 mm, vias 0 -> 2
- net Net-(IC1-FB): track 30.2 -> 9.88 mm
- net /RST: track 17.8 -> 38.0 mm
- net /BOOTMODE: track 27.7 -> 44.4 mm, vias 2 -> 0
- net Net-(J2-D+-PadA6): track 12.8 -> 29.4 mm
- net Net-(U2-FMIP): track 16.1 -> 0.00 mm
- net Net-(U1-IO45): track 3.23 -> 19.3 mm
- net /GPIO8: track 23.0 -> 7.16 mm, vias 3 -> 2
- net Net-(J1-Pin_1): track 23.9 -> 8.01 mm
- net Net-(U6-INL): track 20.6 -> 4.81 mm
- net VBUS: track 18.6 -> 34.3 mm, vias 0 -> 2
- net /GPIO9: track 20.8 -> 5.28 mm, vias 2 -> 0
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- added copper zone on B.Cu, net GND
- added copper zone on F.Cu, net GND
- removed copper zone on In2.Cu, net +5V
- removed copper zone on In1.Cu, net GND
Other:
- board size 45.1 x 57 mm -> 49.4 x 57.1 mm
- copper layers 4 -> 2

Commit message: faj
Parts:
- R17: footprint Resistor_SMD:R_0805_2012Metric -> Resistor_SMD:R_0603_1608Metric
Routing:
- net Net-(IC1-PG): track 15.2 -> 4.86 mm, vias 0 -> 2
- net Net-(J2-D--PadA7): track 25.5 -> 29.0 mm, vias 2 -> 3
- net Net-(J2-D+-PadA6): track 29.4 -> 25.9 mm
- net /RST: track 38.0 -> 41.3 mm
- net Net-(U6-INR): track 15.1 -> 12.1 mm, vias 0 -> 2
- net Net-(J2-CC2): track 16.6 -> 19.2 mm
- net VBUS: track 34.3 -> 36.6 mm
- net Net-(IC1-FB): track 9.88 -> 7.89 mm
- net Net-(C18-Pad2): track 5.68 -> 7.19 mm
- net +5V: track 83.2 -> 81.8 mm, vias 3 -> 2
- net Net-(U6--OUT_R): track 12.0 -> 12.8 mm, vias 0 -> 2
- net +3.3V: track 103.9 -> 104.5 mm, vias 1 -> 0
- net Net-(C17-Pad2): track 8.33 -> 8.97 mm, vias 0 -> 2
- net Net-(J2-CC1): track 10.5 -> 9.94 mm
- net GND: vias 71 -> 72

Commit message: afh
Parts:
- R1: value 10k Ohm -> 4.7k
Connections:
- R10 pad 2: /GPIO9 -> /SCL
- R3 pad 2: /GPIO8 -> /SDA
- U1 pad 12: /GPIO8 -> /SDA
- U1 pad 13: /GPIO9 -> /SCL
Routing:
- net GND: track 0.00 -> 104.2 mm, vias 72 -> 130
- net /SDA: track 0.00 -> 42.7 mm, vias 0 -> 3
- net /SCL: track 0.00 -> 42.6 mm, vias 0 -> 2
- net Net-(U1-EN): track 41.0 -> 66.4 mm, vias 4 -> 2
- net Net-(IC2-ROUT/DOUT): track 6.89 -> 30.5 mm, vias 2 -> 0
- net Net-(C17-Pad2): track 8.97 -> 29.4 mm, vias 2 -> 0
- net Net-(U6--OUT_R): track 12.8 -> 30.9 mm, vias 2 -> 0
- net Net-(J3-Pin_2): track 9.32 -> 22.5 mm
- net Net-(IC2-LOUT/DFS): track 11.7 -> 21.7 mm, vias 2 -> 0
- net /GPIO8: track 7.13 -> 0.00 mm, vias 2 -> 0
- net Net-(J2-CC1): track 9.94 -> 15.5 mm
- net /GPIO9: track 5.28 -> 0.00 mm
- net Net-(U6-INR): track 12.1 -> 7.72 mm
- net Net-(J2-D+-PadA6): track 25.9 -> 22.0 mm
- net Net-(C18-Pad2): track 7.19 -> 10.8 mm
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- added copper zone on In1.Cu, net GND
- added copper zone on In2.Cu, net GND
- removed copper zone on B.Cu, net GND
- removed copper zone on F.Cu, net GND
Other:
- copper layers 2 -> 4
