File: FM-Radios/FM-Radio-v2/FM-Radio.kicad_sch (KiCad schematic)
At the start: 64 parts, among them IC2 SI4732-A10-GSR, J1 L_OUT, J10 3.3V, J11 SDA, J12 SCL, J2 USB_C_Receptacle_USB2.0, J3 R_OUT, J4 Conn_01x10_Pin, J5 GND, J6 FM-ANT, J7 AM-ANT, J9 VBUS, SW2 EN, U1 ESP32-S3-MINI-1U, U2 NCP1117-3.3_SOT223, U4 PRTR5V0U2X, U6 PAM8406D, Y1 32.768 kHz

Commit message: ajd
Parts:
- removed C1, C3: 10uF, Capacitor_SMD:C_0603_1608Metric, symbol Device:C
- removed C10, C11: 18pF, Capacitor_SMD:C_0603_1608Metric, symbol Device:C_Small
- removed C12, C2, C29, C30, C31, C4, C5, C6, C7: 100nF, Capacitor_SMD:C_0603_1608Metric, symbol Device:C
- removed C15, C24: 47uF, Capacitor_SMD:C_1206_3216Metric, symbol Device:C
- removed C16, C17, C18: 1 uF, Capacitor_SMD:C_0603_1608Metric, symbol Device:C
- removed C19, C20, C21, C26: 220pF, Capacitor_SMD:C_0603_1608Metric, symbol Device:C
- removed C23: 10uF, Capacitor_Tantalum_SMD:CP_EIA-3216-18_Kemet-A, symbol Device:C
- removed C25: 1 nF, Capacitor_SMD:C_0603_1608Metric, symbol Device:C_Small
- removed C27: 470 nF, Capacitor_SMD:C_0603_1608Metric, symbol Device:C_Small
- removed C28: 10 uF, Capacitor_Tantalum_SMD:CP_EIA-3216-18_Kemet-A, symbol Device:C_Small
- removed C8: 680 uF, Capacitor_THT:CP_Radial_D12.5mm_P5.00mm, symbol Device:C_Polarized
- removed FB1, FB2, FB3, FB4, FB5: 120Ohm 2A, Resistor_SMD:R_0805_2012Metric, symbol Device:FerriteBead
- removed IC2: SI4732-A10-GSR, SOIC127P600X175-16N, symbol Personal:SI4732-A10-GSR
- removed J1: L_OUT, footprints:WJ500V-5.08-2P, symbol Connector:Screw_Terminal_01x02
- removed J10: 3.3V, Connector_PinHeader_2.54mm:PinHeader_1x01_P2.54mm_Vertical, symbol Connector:Conn_01x01_Pin
- removed J11: SDA, Connector_PinHeader_2.54mm:PinHeader_1x01_P2.54mm_Vertical, symbol Connector:Conn_01x01_Pin
- removed J12: SCL, Connector_PinHeader_2.54mm:PinHeader_1x01_P2.54mm_Vertical, symbol Connector:Conn_01x01_Pin
- removed J2: USB_C_Receptacle_USB2.0, Connector_USB:USB_C_Receptacle_HRO_TYPE-C-31-M-12, symbol Connector:USB_C_Receptacle_USB2.0
- removed J3: R_OUT, footprints:WJ500V-5.08-2P, symbol Connector:Screw_Terminal_01x02
- removed J6: FM-ANT, footprints:BAT_WIRELESS_BWSMA-KE-Z001, symbol Personal:BWSMA-KE-Z001
- removed J7: AM-ANT, footprints:BAT_WIRELESS_BWSMA-KE-Z001, symbol Personal:BWSMA-KE-Z001
- removed J9: VBUS, Connector_PinHeader_2.54mm:PinHeader_1x01_P2.54mm_Vertical, symbol Connector:Conn_01x01_Pin
- removed L3: 500 uH, Inductor_SMD:L_Taiyo-Yuden_NR-40xx_HandSoldering, symbol Device:L
- removed R1: 4.7k, Resistor_SMD:R_0603_1608Metric, symbol Device:R_Small
- removed R11, R4: 10k Ohm, Resistor_SMD:R_0603_1608Metric, symbol Device:R_Small
- removed S1: SSSS811101, footprints:SSSS811101, symbol Personal:SSSS811101
- removed U2: NCP1117-3.3_SOT223, Package_TO_SOT_SMD:SOT-223-3_TabPin2, symbol Regulator_Linear:NCP1117-3.3_SOT223
- removed U6: PAM8406D, Package_SO:SOIC-16_3.9x9.9mm_P1.27mm, symbol Amplifier_Audio:PAM8406D
- removed Y1: 32.768 kHz, Crystal:Crystal_SMD_3215-2Pin_3.2x1.5mm, symbol Device:Crystal
- added C10: 100nF, Capacitor_SMD:C_0603_1608Metric, symbol Device:C
- added C38: 47uF, Capacitor_SMD:C_1206_3216Metric, symbol Device:C
- added C9: 10uF, Capacitor_SMD:C_0603_1608Metric, symbol Device:C
- added J2: USB_C_Receptacle_USB2.0_16P, Connector_USB:USB_C_Receptacle_HRO_TYPE-C-31-M-12, symbol Connector:USB_C_Receptacle_USB2.0_16P
- added J8: 5V, Connector_PinHeader_2.54mm:PinHeader_1x01_P2.54mm_Vertical, symbol Connector:Conn_01x01_Pin
- added R13, R14: 10k Ohm, Resistor_SMD:R_0603_1608Metric, symbol Device:R_Small
- added SW3: EN, footprints:KH-6X6X5H-STM_SKE, symbol 2026-02-17_13-05-37:KH-6X6X5H-STM
Connections:
- net +3.3V: now also C10.1, C38.1, C9.1, R13.1, R14.1
- net +5V: now also J8.1 (Pin_1)
- net BOOTMODE: now also SW3.B
- net GND: now also C10.2, C38.2, C9.2, J2.A1 (GND), J2.A12 (GND), J2.B1 (GND), J2.B12 (GND), J2.SH (SHIELD), SW3.C, SW3.D
- net VBUS: now also J2.A4 (VBUS), J2.A9 (VBUS), J2.B4 (VBUS), J2.B9 (VBUS)
- net at SW2.A, SW2.B, U1.45 (EN): now also R13.2
- net at R9.1: now also J2.A6 (D+), J2.B6 (D+)
- net at R8.1: now also J2.A7 (D-), J2.B7 (D-)
- net MODE: now reaches U1.15 (IO11)
- net MUTE: now reaches U1.16 (IO12)
- net at R7.1: now also J2.B5 (CC2)
- net at R6.2: now also J2.A5 (CC1)
- new net: R14.2, SW3.A
- no-connect marks 10 -> 3
Other:
- added sheet amp (amp.kicad_sch)
- added sheet power (power.kicad_sch)
- added sheet tuner (tuner.kicad_sch)
- moved on the sheet: C22, F1, J4, R10, R3, R5, SW2, U1, U4

Commit message: a
Parts:
- added C33, C34: 10uF, Capacitor_SMD:C_0603_1608Metric, symbol Device:C
- added J9: 3.3V, Connector_PinHeader_2.54mm:PinHeader_1x01_P2.54mm_Vertical, symbol Connector:Conn_01x01_Pin
- added U3: MIC5504-3.3YM5, Package_TO_SOT_SMD:SOT-23-5, symbol Regulator_Linear:MIC5504-3.3YM5
Connections:
- net +3.3V: now also C34.1, J9.1 (Pin_1), U3.5 (VOUT)
- net +5V: now also C33.1, U3.1 (VIN), U3.3 (EN)
- net GND: now also C33.2, C34.2, U3.2 (GND)
Other:
- removed sheet power

Commit message: faj
Parts:
- added C36, C37: 10uF, Capacitor_SMD:C_0603_1608Metric, symbol Device:C
- added J10: 1.8V, Connector_PinHeader_2.54mm:PinHeader_1x01_P2.54mm_Vertical, symbol Connector:Conn_01x01_Pin
- added U2: LD1117S18TR_SOT223, Package_TO_SOT_SMD:SOT-223-3_TabPin2, symbol Regulator_Linear:LD1117S18TR_SOT223
- C33, C34, C9: LCSC C1691 -> C19702
- J2: LCSC Part # (none) -> C165948
- R10, R3: LCSC Part # C99782 -> C23162
- R13, R14, R5: LCSC Part # C98220 -> C25804
- U1: LCSC Part # (none) -> C2980299
- U3: LCSC Part # (none) -> C88419
Connections:
- net +3.3V: now also C36.1, U2.3 (VI)
- net GND: now also C36.2, C37.2, U2.1 (GND)
- net MP0: now reaches U1.18 (IO14)
- net MP1: now reaches U1.19 (IO15)
- net MP2: now reaches U1.20 (IO16)
- new net +1V8: C37.1, J10.1 (Pin_1), U2.2 (VO)
Other:
- added sheet dsp (dsp.kicad_sch)
- moved on the sheet: C33, C34, J9, U3
