File: FM-Radios/FM-Radio-v2/FM-Radio.kicad_sch (KiCad schematic)
At the start: 30 parts, among them J10 1.8V, J2 USB_C_Receptacle_USB2.0_16P, J4 Conn_01x10_Pin, J5 GND, J8 5V, J9 3.3V, SW2 EN, SW3 EN, U1 ESP32-S3-MINI-1U, U2 LD1117S18TR_SOT223, U3 MIC5504-3.3YM5, U4 PRTR5V0U2X

Commit message: jfh
Parts:
- removed C22: 100nF, Capacitor_SMD:C_0603_1608Metric, symbol Device:C
- removed F1: 500 mA, Fuse:Fuse_1206_3216Metric, symbol Device:Polyfuse
- removed U4: PRTR5V0U2X, Package_TO_SOT_SMD:SOT-143, symbol Power_Protection:PRTR5V0U2X
Connections:
- net VBUS is gone; now on net +5V: J2.A4 (VBUS), J2.A9 (VBUS), J2.B4 (VBUS), J2.B9 (VBUS)
- net SHND: now also U1.17 (IO13)
- net MP0: no longer names the net of U1.18 (IO14)
- net MP1: no longer names the net of U1.19 (IO15)
- net MP2: no longer names the net of U1.20 (IO16)
- net RST: no longer names the net of U1.14 (IO10)
- no-connect marks 3 -> 21
Other:
- removed sheet dsp
- sheet tuner ports: added none; removed RST
- moved on the sheet: J8
