File: FM-Radios/FM-Radio-v2/dsp.kicad_sch (KiCad schematic)
At the start: 27 parts, among them SW1 BOOT, U7 ADAU1701, Y1 Crystal_GND24

Commit message: jfh
Parts:
- removed C12, C13: 12 pF, Capacitor_SMD:C_0805_2012Metric, symbol Device:C
- removed C17, C18: 1 uF, Capacitor_SMD:C_0603_1608Metric, symbol Device:C
- removed C39: 56 nF, Capacitor_SMD:C_0805_2012Metric, symbol Device:C
- removed C40: 3.3 nF, Capacitor_SMD:C_0805_2012Metric, symbol Device:C
- removed C41, C47, C49: 10 uF, Capacitor_SMD:C_0805_2012Metric, symbol Device:C
- removed C42, C43, C44, C45, C46, C48, C50: 100 nF, Capacitor_SMD:C_0805_2012Metric, symbol Device:C
- removed R11, R12, R4: 100 Ohm, Resistor_SMD:R_0603_1608Metric, symbol Device:R_Small
- removed R16, R17, R18, R19: 10k Ohm, Resistor_SMD:R_0603_1608Metric, symbol Device:R_Small
- removed R20: 475 Ω, Resistor_SMD:R_0805_2012Metric, symbol Device:R
- removed SW1: BOOT, footprints:KH-6X6X5H-STM_SKE, symbol 2026-02-17_13-05-37:KH-6X6X5H-STM
- removed U7: ADAU1701, Package_QFP:LQFP-48_7x7mm_P0.5mm, symbol DSP_AnalogDevices:ADAU1701
- removed Y1: Crystal_GND24, Crystal:Crystal_SMD_3225-4Pin_3.2x2.5mm, symbol Device:Crystal_GND24
Connections:
- no-connect marks 13 -> 0
