File: WalkieTalkies/WK-1/dac.kicad_sch (KiCad schematic)
At the start: 15 parts, among them U2 CS4344

Commit message: a
Parts:
- U2: LCSC Part # (none) -> C8952

Commit message: grrr
Parts:
- C10: LCSC C51412 -> (none); LCSC Part # (none) -> C51412
- C33: LCSC C96123 -> (none); LCSC Part # (none) -> C96123
- C34: LCSC C14663 -> (none); LCSC Part # (none) -> C14663
- C36, C37: LCSC C107050 -> (none); LCSC Part # (none) -> C107050
- C7, C9: LCSC C19702 -> (none); LCSC Part # (none) -> C19702
- R10, R11: LCSC Part # C98220 -> C25804
Changed lines of the file:
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@@
 			)
 		)
-		(property "LCSC" "C14663"
+		(property "LCSC Part #" "C14663"
 			(at 151.13 69.85 0)
 			(hide yes)
@@
 			)
 		)
-		(property "LCSC" "C107050"
+		(property "LCSC Part #" "C107050"
 			(at 180.34 86.36 0)
 			(hide yes)
@@
 			)
 		)
-		(property "LCSC" "C96123"
+		(property "LCSC Part #" "C96123"
 			(at 128.27 69.85 0)
 			(hide yes)
@@
 			)
 		)
-		(property "LCSC Part #" "C98220"
+		(property "LCSC Part #" "C25804"
 			(at 154.94 97.79 0)
 			(hide yes)
@@
 			)
 		)
-		(property "LCSC" "C19702"
+		(property "LCSC Part #" "C19702"
 			(at 140.97 69.85 0)
 			(hide yes)
@@
 			)
 		)
-		(property "LCSC" "C19702"
+		(property "LCSC Part #" "C19702"
 			(at 135.89 106.68 0)
 			(hide yes)
@@
 			)
 		)
-		(property "LCSC" "C51412"
+		(property "LCSC Part #" "C51412"
 			(at 97.79 106.68 0)
 			(hide yes)
@@
 			)
 		)
-		(property "LCSC" "C107050"
+		(property "LCSC Part #" "C107050"
 			(at 180.34 99.06 0)
 			(hide yes)
@@
 			)
 		)
-		(property "LCSC Part #" "C98220"
+		(property "LCSC Part #" "C25804"
 			(at 154.94 87.63 0)
 			(hide yes)
