File: WalkieTalkies/WK-1/WK-1.kicad_sch (KiCad schematic)
At the start: 20 parts, among them J6 FM-ANT, J7 FM-ANT, U2 Si4463, Y1 Crystal

Commit message: yarrr
Parts:
- removed C1: 150pF, symbol Device:C
- removed C2: 6.8 pF, symbol Device:C
- removed C4, C5: 8.2 pF, symbol Device:C
- removed C6: 3.9 pF, symbol Device:C
- removed C7: 2.2 pF, symbol Device:C
- removed C8: 150 pF, symbol Device:C
- removed J6, J7: FM-ANT, footprints:BAT_WIRELESS_BWSMA-KE-Z001, symbol Personal:BWSMA-KE-Z001
- removed L1: 220 nH, symbol Device:L
- removed L2: 24 nH, symbol Device:L
- removed L3, L5: 18 nH, symbol Device:L
- removed L4: 27 nH, symbol Device:L
- removed L6: 51 nH, symbol Device:L
- removed L7: 47 nH, symbol Device:L
- removed R1: 0 ohm, symbol Device:R
- removed U2: Si4463, Package_DFN_QFN:QFN-20-1EP_4x4mm_P0.5mm_EP2.6x2.6mm_ThermalVias, symbol RF:Si4463
- removed Y1: Crystal, symbol Device:Crystal
- added C22: 100nF, Capacitor_SMD:C_0603_1608Metric, symbol Device:C
- added C25: 47uF, Capacitor_SMD:C_1206_3216Metric, symbol Device:C
- added F1: 500 mA, Fuse:Fuse_1206_3216Metric, symbol Device:Polyfuse
- added J2: USB_C_Receptacle_USB2.0, Connector_USB:USB_C_Receptacle_HRO_TYPE-C-31-M-12, symbol Connector:USB_C_Receptacle_USB2.0
- added J5: GND, Connector_PinHeader_2.54mm:PinHeader_1x01_P2.54mm_Vertical, symbol Connector:Conn_01x01_Pin
- added R14, R2, R3: 4.7k, Resistor_SMD:R_0603_1608Metric, symbol Device:R_Small
- added R5: 10k Ohm, Resistor_SMD:R_0603_1608Metric, symbol Device:R_Small
- added R6, R7: 5.1k, Resistor_SMD:R_0603_1608Metric, symbol Device:R
- added R8, R9: 22, Resistor_SMD:R_0603_1608Metric, symbol Device:R
- added S1: SSSS811101, footprints:SSSS811101, symbol Personal:SSSS811101
- added SW100, SW99: EN, footprints:KH-6X6X5H-STM_SKE, symbol 2026-02-17_13-05-37:KH-6X6X5H-STM
- added U1: ESP32-S3-MINI-1U, RF_Module:ESP32-S2-MINI-1U, symbol RF_Module:ESP32-S3-MINI-1U
- added U10, U7, U8, U9: WS2812B-B, footprints:LED_WS2812B-B, symbol WS2812B-B:WS2812B-B
- added U4: PRTR5V0U2X, Package_TO_SOT_SMD:SOT-143, symbol Power_Protection:PRTR5V0U2X
- C3: value 6.8 pF -> 10uF; footprint (none) -> Capacitor_SMD:C_0603_1608Metric; LCSC (none) -> C1691
Connections:
- net +3.3V: now also C3.1, C25.1, R14.1, R2.1, R3.1, R5.2, S1.1, U1.3 (3V3)
- net GND: now also C3.2, C22.2, C25.2, J2.A1 (GND), J2.A12 (GND), J2.B1 (GND), J2.B12 (GND), J2.S1 (SHIELD), J5.1 (Pin_1), R6.1, R7.2, S1.3, SW99.C, SW99.D, U1.1 (GND), U1.2 (GND), U1.42 (GND), U1.43 (GND), U1.44 (IO46), U1.46 (GND), U1.47 (GND), U1.48 (GND), U1.49 (GND), U1.50 (GND), U1.51 (GND), U1.52 (GND), U1.53 (GND), U1.54 (GND), U1.55 (GND), U1.56 (GND), U1.57 (GND), U1.58 (GND), U1.59 (GND), U1.60 (GND), U1.61 (GND), U1.62 (GND), U1.63 (GND), U1.64 (GND), U1.65 (GND), U10.3 (VSS), U4.1 (GND), U7.3 (VSS), U8.3 (VSS), U9.3 (VSS); no longer C3.1
- net IRQ: now also U1.10 (IO6)
- net SCLK: now also U1.11 (IO7), U1.28 (IO33)
- net SDI: now also U1.12 (IO8)
- net SDN: now also U1.13 (IO9)
- net SDO: now also U1.14 (IO10)
- net SEL: now also U1.15 (IO11)
- new net: J2.A6 (D+), J2.B6 (D+), R9.1
- new net: U7.2 (DOUT), U8.4 (DIN)
- new net: U8.2 (DOUT), U9.4 (DIN)
- new net: J2.A7 (D-), J2.B7 (D-), R8.1
- new net: J2.A5 (CC1), R6.2
- new net: R2.2, SW99.A, SW99.B, U1.45 (EN)
- new net: U10.4 (DIN), U9.2 (DOUT)
- new net: J2.B5 (CC2), R7.1
- new net: R5.1, U1.41 (IO45)
- new net +5V: C22.1, F1.2, SW100.B, SW100.D, U10.1 (VDD), U4.4 (VCC), U7.1 (VDD), U8.1 (VDD), U9.1 (VDD)
- new net BOOTMODE: S1.2, U1.4 (IO0)
- new net D+: R9.2, U1.24 (USB_D+), U4.3 (I/O2)
- new net D-: R8.2, U1.23 (USB_D-), U4.2 (I/O1)
- new net K_OUT: U1.33 (IO37)
- new net LED_DIN: U1.35 (IO39), U7.4 (DIN)
- new net LRCK: U1.26 (IO26)
- new net MCLK: U1.29 (IO34)
- new net MODE: U1.20 (IO16)
- new net MUTE: U1.21 (IO17)
- new net SD-MIC: U1.31 (IO35)
- new net SDIN-DAC: U1.32 (IO36)
- new net SHND: U1.22 (IO18)
- new net SPEAK: SW100.A, SW100.C, U1.34 (IO38)
- new net VBUS: F1.1, J2.A4 (VBUS), J2.A9 (VBUS), J2.B4 (VBUS), J2.B9 (VBUS)
- new net keypad/SCL: R14.2, U1.18 (IO14)
- new net keypad/SDA: R3.2, U1.17 (IO13)
- no-connect marks 4 -> 12
Other:
- added sheet amp (amp.kicad_sch)
- added sheet dac (dac.kicad_sch)
- added sheet keypad (keypad.kicad_sch)
- added sheet microphone (microphone.kicad_sch)
- added sheet power (power.kicad_sch)
- added sheet transceiver (transceiver.kicad_sch)

Commit message: a
Parts:
- U1: LCSC Part # (none) -> C2980299

Commit message: grrr
Parts:
- removed J5: GND, Connector_PinHeader_2.54mm:PinHeader_1x01_P2.54mm_Vertical, symbol Connector:Conn_01x01_Pin
- added J8: Conn_01x04_Pin, Connector_PinSocket_2.54mm:PinSocket_1x04_P2.54mm_Vertical, symbol Connector:Conn_01x04_Pin
- added J9: DEBG, Connector_PinSocket_2.54mm:PinSocket_1x04_P2.54mm_Vertical, symbol Connector:Conn_01x04_Pin
- C3: LCSC C1691 -> (none); LCSC Part # (none) -> C19702
- F1: LCSC C135341 -> (none); LCSC Part # (none) -> C135341
- R14, R2, R3: LCSC Part # C99782 -> C23162
- R5: LCSC Part # C98220 -> C25804
- U10, U7, U8, U9: LCSC Part # C114586 -> C2761795
- U4: LCSC C2827688 -> (none); LCSC Part # (none) -> C2827688
Connections:
- net +3.3V: now also J8.3 (Pin_3), J9.3 (Pin_3)
- net GND: now also J8.4 (Pin_4), J9.4 (Pin_4)
- net keypad/SCL: now also J8.2 (Pin_2)
- net keypad/SDA: now also J8.1 (Pin_1)
- net TXD0: now reaches U1.39 (TXD0)
- net TXD0: now also J9.1 (Pin_1)
- net RDX0: now reaches U1.40 (RXD0)
- net RDX0: now also J9.2 (Pin_2)

Commit message: grr
Connections:
- net SPEAK: no longer SW100.A
- no-connect marks 12 -> 13
Changed lines of the file:
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@@
-	)
-	(junction
-		(at 218.44 140.97)
-		(diameter 0)
-		(color 0 0 0 0)
 	)
 	(junction
@@
 	)
 	(no_connect
+		(at 218.44 138.43)
+	)
+	(no_connect
 		(at 44.45 172.72)
 	)
@@
 	(wire
 		(pts
-			(xy 218.44 140.97) (xy 218.44 143.51)
-		)
-		(stroke
-			(width 0)
-			(type default)
-		)
-	)
-	(wire
-		(pts
 			(xy 91.44 166.37) (xy 105.41 166.37)
 		)
@@
 	(wire
 		(pts
-			(xy 218.44 138.43) (xy 218.44 140.97)
-		)
-		(stroke
-			(width 0)
-			(type default)
-		)
-	)
-	(wire
-		(pts
 			(xy 120.65 107.95) (xy 120.65 113.03)
 		)
@@
 	(wire
 		(pts
-			(xy 215.9 140.97) (xy 218.44 140.97)
+			(xy 215.9 143.51) (xy 218.44 143.51)
 		)
 		(stroke
@@
 	)
 	(label "SPEAK"
-		(at 215.9 140.97 180)
-		(effects
-			(font
+		(at 215.9 143.51 180)
+		(effects
+			(font

Commit message: afj
Other:
- sheet transceiver ports: added CS, SI, SO; removed IRQ, SDI, SDN, SDO, SEL
Changed lines of the file:
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@@
 	(wire
 		(pts
-			(xy 127 77.47) (xy 130.81 77.47)
-		)
-		(stroke
-			(width 0)
-			(type default)
-		)
-	)
-	(wire
-		(pts
 			(xy 50.8 57.15) (xy 62.23 57.15)
 		)
@@
 	(wire
 		(pts
-			(xy 127 85.09) (xy 130.81 85.09)
-		)
-		(stroke
-			(width 0)
-			(type default)
-		)
-	)
-	(wire
-		(pts
 			(xy 101.6 45.72) (xy 67.31 45.72)
 		)
@@
 		)
 	)
-	(label "SDN"
-		(at 127 85.09 180)
-		(effects
-			(font
-				(size 1.27 1.27)
-			)
-			(justify right bottom)
-		)
-	)
 	(label "LRCK"
 		(at 135.89 143.51 0)
@@
 		)
 	)
-	(label "IRQ"
-		(at 127 77.47 180)
-		(effects
-			(font
-				(size 1.27 1.27)
-			)
-			(justify right bottom)
-		)
-	)
 	(label "SD-MIC"
 		(at 157.48 58.42 180)
@@
 			)
 		)
-		(pin "IRQ" input
-			(at 130.81 77.47 180)
+		(pin "CS" input
+			(at 130.81 90.17 180)
 			(effects
 				(font
@@
 			)
 		)
-		(pin "SDI" input
+		(pin "SI" input
 			(at 130.81 82.55 180)
 			(effects
@@
 			)
 		)
-		(pin "SDN" input
-			(at 130.81 85.09 180)
-			(effects
-				(font
-					(size 1.27 1.27)
-				)
-				(justify left)
-			)
-		)
-		(pin "SDO" input
+		(pin "SO" input
 			(at 130.81 87.63 180)
 			(effects
 				(font
-					(size 1.27 1.27)
-				)
-				(justify left)
-			)
-		)
-		(pin "SEL" input
-			(at 130.81 90.17 180)
-			(effects
-				(font
