File: WalkieTalkies/WK-1/transceiver.kicad_sch (KiCad schematic)
At the start: 25 parts, among them J8 RX, J9 TX, U3 Si4463, Y2 30 Mhz

Commit message: a
Parts:
- removed J8: RX, footprints:BAT_WIRELESS_BWSMA-KE-Z001, symbol Personal:BWSMA-KE-Z001
- removed J9: TX, footprints:BAT_WIRELESS_BWSMA-KE-Z001, symbol Personal:BWSMA-KE-Z001
- added J6: TX, Connector_Coaxial:SMA_BAT_Wireless_BWSMA-KWE-Z001, symbol Connector:Conn_Coaxial
- added J7: RX, Connector_Coaxial:SMA_BAT_Wireless_BWSMA-KWE-Z001, symbol Connector:Conn_Coaxial
- added L15: 220 nH, Inductor_SMD:L_0805_2012Metric, symbol Device:L
- added R15: 33 ohm, Resistor_SMD:R_0805_2012Metric, symbol Device:R
- added U12: BGA616H6327XTSA1, PG-SOT343-4-2_INF, symbol symbols:BGA616H6327XTSA1
- C11, C12: LCSC Part # (none) -> C1648
- C13: LCSC Part # (none) -> C107038
- C14: LCSC Part # (none) -> C519107
- C15, C16: LCSC Part # (none) -> C1679
- C17, C18: LCSC Part # (none) -> C1651
- C19, C20: LCSC Part # (none) -> C1685
- L10: LCSC Part # (none) -> C1331755
- L11: LCSC Part # (none) -> C18221260
- L12: LCSC Part # (none) -> C317993
- L13: LCSC Part # (none) -> C98992
- L14: LCSC Part # (none) -> C964055
- L8: LCSC Part # (none) -> C2041935
- L9: LCSC Part # (none) -> C2042178
- R4: LCSC Part # (none) -> C100045
- U3: LCSC Part # (none) -> C476202
Connections:
- net GND: now also J6.2 (Ext), J7.2 (Ext), U12.2 (GND), U12.4 (GND)
- net at C18.1: now also J7.1 (In)
- net at L14.2: now also U12.1 (IN)
- new net: L15.1, R15.2
- new net: J6.1 (In), L15.2, U12.3 (OUT)
- new net +5V: R15.1

Commit message: grrr
Parts:
- C1: LCSC C1691 -> (none); LCSC Part # (none) -> C19702
- C11: LCSC Part # C1648 -> C1648
- C13: LCSC Part # C107038 -> C1594
- C2: LCSC C14663 -> (none)
- C24: LCSC C96123 -> (none); LCSC Part # (none) -> C96123
- R15: LCSC Part # C2907258 -> C17634
- R4: LCSC Part # C100045 -> C17477
- U12: footprint PG-SOT343-4-2_INF -> footprints:PG-SOT343-4-2_INF; LCSC Part # (none) -> C3191605
Changed lines of the file:
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@@
 			)
 		)
-		(property "LCSC" "C1691"
+		(property "LCSC Part #" "C19702"
 			(at 93.98 58.42 0)
 			(hide yes)
@@
 			)
 		)
-		(property "LCSC" "C14663"
-			(at 105.41 58.42 0)
-			(hide yes)
-			(show_name no)
-			(do_not_autoplace no)
-			(effects
-				(font
-					(size 1.27 1.27)
-				)
-			)
-		)
 		(property "JlcRotOffset" ""
 			(at 105.41 58.42 0)
@@
 			)
 		)
-		(property "LCSC" "C96123"
+		(property "LCSC Part #" "C96123"
 			(at 83.82 58.42 0)
 			(hide yes)
@@
 			)
 		)
-		(property "LCSC Part #" "C100045"
+		(property "LCSC Part #" "C17477 "
 			(at 127 66.04 0)
 			(hide yes)
@@
 			)
 		)
-		(property "LCSC Part #" "C107038"
+		(property "LCSC Part #" "C1594"
 			(at 137.16 69.85 90)
 			(hide yes)
@@
 			)
 		)
-		(property "LCSC Part #" "C1648"
+		(property "LCSC Part #" "C1648 "
 			(at 78.74 81.28 90)
 			(hide yes)
@@
 			)
 		)
-		(property "LCSC Part #" "C2907258"
+		(property "LCSC Part #" "C17634"
 			(at 237.49 52.07 0)
 			(hide yes)
@@
 			)
 		)
-		(property "Footprint" "PG-SOT343-4-2_INF"
+		(property "Footprint" "footprints:PG-SOT343-4-2_INF"
 			(at 204.47 68.58 0)
 			(hide yes)
@@
 			(at 204.47 68.58 0)
 			(hide yes)
+			(show_name no)
+			(do_not_autoplace no)
+			(effects
+				(font
+					(size 1.27 1.27)
+				)
+			)
+		)
+		(property "LCSC Part #" "C3191605"
+			(at 204.47 68.58 0)
+			(hide yes)

Commit message: afj
Parts:
- removed C1: 10uF, Capacitor_SMD:C_0603_1608Metric, symbol Device:C
- removed C13: 150pF, Capacitor_SMD:C_0603_1608Metric, symbol Device:C
- removed C14: 3.9 pF, Capacitor_SMD:C_0603_1608Metric, symbol Device:C
- removed C15, C16: 6.8 pF, Capacitor_SMD:C_0603_1608Metric, symbol Device:C
- removed C17, C18: 2.2 pF, Capacitor_SMD:C_0603_1608Metric, symbol Device:C
- removed C19, C20: 8.2 pF, Capacitor_SMD:C_0603_1608Metric, symbol Device:C
- removed C2: 100nF, Capacitor_SMD:C_0603_1608Metric, symbol Device:C
- removed C24: 47uF, Capacitor_SMD:C_1206_3216Metric, symbol Device:C
- removed J6: TX, Connector_Coaxial:SMA_BAT_Wireless_BWSMA-KWE-Z001, symbol Connector:Conn_Coaxial
- removed J7: RX, Connector_Coaxial:SMA_BAT_Wireless_BWSMA-KWE-Z001, symbol Connector:Conn_Coaxial
- removed L10: 24 nH, Inductor_SMD:L_0805_2012Metric, symbol Device:L
- removed L11: 3.3 nH, Inductor_SMD:L_0805_2012Metric, symbol Device:L
- removed L12: 4.7 nH, Inductor_SMD:L_0805_2012Metric, symbol Device:L
- removed L13: 27 nH, Inductor_SMD:L_0805_2012Metric, symbol Device:L
- removed L14: 2.2 nH, Inductor_SMD:L_0805_2012Metric, symbol Device:L
- removed L15, L8: 220 nH, Inductor_SMD:L_0805_2012Metric, symbol Device:L
- removed L9: 51 nH, Inductor_SMD:L_0805_2012Metric, symbol Device:L
- removed R15: 33 ohm, Resistor_SMD:R_0805_2012Metric, symbol Device:R
- removed R4: 0 ohm, Resistor_SMD:R_0805_2012Metric, symbol Device:R
- removed U12: BGA616H6327XTSA1, footprints:PG-SOT343-4-2_INF, symbol symbols:BGA616H6327XTSA1
- removed U3: Si4463, Package_DFN_QFN:QFN-20-1EP_4x4mm_P0.5mm_EP2.6x2.6mm_ThermalVias, symbol RF:Si4463
- removed Y2: 30 Mhz, Crystal:Crystal_SMD_3225-4Pin_3.2x2.5mm, symbol Device:Crystal
- added C32: 47uF, Capacitor_SMD:C_1206_3216Metric, symbol Device:C
- added C39: 10uF, Capacitor_SMD:C_0603_1608Metric, symbol Device:C
- added C41: 100nF, Capacitor_SMD:C_0603_1608Metric, symbol Device:C
- added C42: 1 uF, Capacitor_SMD:C_0603_1608Metric, symbol Device:C
- added C43, C45: 6.8 pF, Capacitor_SMD:C_0603_1608Metric, symbol Device:C
- added C44, C47: 220 pF, Capacitor_SMD:C_0603_1608Metric, symbol Device:C
- added C46: 12 pF, Capacitor_SMD:C_0603_1608Metric, symbol Device:C
- added IC1: CC110LRGPR, QFN50P400X400X100-21N-D, symbol symbols:CC110LRGPR
- added J10: ANT, Connector_Coaxial:SMA_BAT_Wireless_BWSMA-KWE-Z001, symbol Connector:Conn_Coaxial
- added L16, L19: 33 nH, Inductor_SMD:L_0805_2012Metric, symbol Device:L
- added L17, L18: 18 nH, Inductor_SMD:L_0805_2012Metric, symbol Device:L
- added Rbias1: 56k, Resistor_SMD:R_0603_1608Metric, symbol Device:R
- added Y1: 26MHz, Crystal:Crystal_SMD_3225-4Pin_3.2x2.5mm, symbol Device:Crystal_GND24
- C11, C12: value 20 pF -> 12 pF
Connections:
- net +3.3V: now also C32.1, C39.1, C41.1, IC1.11 (AVDD_2), IC1.14 (AVDD_3), IC1.15 (AVDD_4), IC1.18 (DGUARD), IC1.4 (DVDD), IC1.9 (AVDD_1)
- net GND: now also C32.2, C39.2, C41.2, C42.1, C43.1, C44.2, C46.2, IC1.16 (GND_1), IC1.19 (GND_2), IC1.21 (GND_3), J10.2 (Ext), Rbias1.1, Y1.2 (G), Y1.4 (G)
- net SCLK: now also IC1.1 (SCLK)
- net at C12.2: now also IC1.10 (XOSC_Q2), Y1.1
- net at C11.2: now also IC1.8 (XOSC_Q1), Y1.3
- new net: C45.2, L17.2, L18.1
- new net: C46.1, L18.2, L19.1
- new net: C44.1, L16.1
- new net: C45.1, IC1.12 (RF_P), L16.2
- new net: C47.1, L19.2
- new net: C47.2, J10.1 (In)
- new net: IC1.17 (RBIAS), Rbias1.2
- new net: C43.2, IC1.13 (RF_N), L17.1
- new net: C42.2, IC1.5 (DCOUPL)
- new net CS: IC1.7 (CSN)
- new net SI: IC1.20 (SI)
- new net SO: IC1.2 (SO_(GDO1))
- no-connect marks 5 -> 2
