File: Psu/HighEffNixiPSU/HighEffNixiPSU.kicad_sch (KiCad schematic)
At the start: 30 parts, among them J1 Jack-DC, Q1 FQD16N25CTM, U1 LM3478MM

Commit message: shenanigooner
Parts:
- added C2, C4: 100nF, Capacitor_SMD:C_1206_3216Metric, symbol Device:C
- renumbered C14 to C10, C4 to C5, C2 to C6, C12 to C8, C13 to C9, Ccomp3 to Ccomp1, Ccomp1 to Ccomp2, Ccomp2 to Ccomp3
Connections:
- net GND: now also C2.2, C4.2
- net VCC: now also C2.1, C4.1
Other:
- moved on the sheet: C10, C3, C5, C7, C8, C9

Commit message: Shenanigans
Parts:
- removed C10, C9: 100nF, Capacitor_SMD:C_0805_2012Metric, symbol Device:C
- removed J1: Jack-DC, Connector_BarrelJack:BarrelJack_CUI_PJ-063AH_Horizontal, symbol Connector:Jack-DC
- added C26: 47uF, Capacitor_SMD:C_1206_3216Metric, symbol Device:C
- added J3: Barrel_Jack_MountingPin, Connector_BarrelJack:BarrelJack_CUI_PJ-063AH_Horizontal, symbol Connector:Barrel_Jack_MountingPin
- C3: footprint Capacitor_SMD:C_0805_2012Metric -> Capacitor_SMD:C_0603_1608Metric; LCSC C15850 -> C1691
- C5, C7, C8: footprint Capacitor_SMD:C_0805_2012Metric -> Capacitor_SMD:C_0603_1608Metric; LCSC C28233 -> C14663
Connections:
- net +12V: now also C26.1, J3.1
- net GND: now also C26.2, J3.2, J3.MP (MountPin)
Other:
- sheet mcu ports: added CS, GPIO1, GPIO2, GPIO3, GPIO4, GPIO5, GPIO6, MOSI, SCLK; removed BL, CLK, DAT, LE, POL
- sheet nixi_driver ports: added CS, GPIO1, GPIO2, GPIO3, GPIO4, GPIO5, GPIO6, MOSI, SCLK; removed BL, CLK, DAT, LE, POL
- moved on the sheet: H1, H2, H3, H4

Commit message: FPGA time
Parts:
- added VIN2, VIN3: Conn_01x01, Connector_PinHeader_2.54mm:PinHeader_1x01_P2.54mm_Vertical, symbol Connector_Generic:Conn_01x01
- Cbyp1: LCSC Part # C784084 -> C28233
- Ccomp1: LCSC Part # C2168780 -> C1716
Connections:
- net VCC: now also VIN2.1 (Pin_1)
- new net +3V3: VIN3.1 (Pin_1)
