File: Psu/HighEffNixiPSU/HighEffNixiPSU.kicad_sch (KiCad schematic)
At the start: 33 parts, among them J3 Barrel_Jack_MountingPin, Q1 FQD16N25CTM, U1 LM3478MM

Commit message: jfahefh
Parts:
- removed J3: Barrel_Jack_MountingPin, Connector_BarrelJack:BarrelJack_CUI_PJ-063AH_Horizontal, symbol Connector:Barrel_Jack_MountingPin
- added J1: Screw_Terminal_01x02, footprints:WJ500V-5.08-2P, symbol Connector:Screw_Terminal_01x02
Connections:
- net +12V: now also J1.2 (Pin_2)
- net GND: now also J1.1 (Pin_1)
