File: Psu/HighEffNixiPSU/mcu.kicad_sch (KiCad schematic)
At the start: 57 parts, among them J2 USB_C_Receptacle_USB2.0, Q10 MMBTA06, Q12 MMBTA06, Q2 MMBTA06, Q3 MMBTA06, Q4 MMBTA06, Q5 MMBTA06, Q6 MMBTA06, Q7 MMBTA06, Q8 MMBTA06, Q9 MMBTA06, SW2 EN, U2 ESP32-S3-MINI-1, U3 TPS562202

Commit message: shenanigooner
Parts:
- removed U2: ESP32-S3-MINI-1, RF_Module:ESP32-S2-MINI-1, symbol RF_Module:ESP32-S3-MINI-1
- added C14: 100nF, Capacitor_SMD:C_0603_1608Metric, symbol Device:C
- added C15: 10uF, Capacitor_SMD:C_0603_1608Metric, symbol Device:C
- added C22: 22 uF, Capacitor_SMD:C_0603_1608Metric, symbol Device:C_Small
- added F1: 500 mA, Fuse:Fuse_1206_3216Metric, symbol Device:Polyfuse
- added J3: VBUS, Connector_PinHeader_2.54mm:PinHeader_1x01_P2.54mm_Vertical, symbol Connector:Conn_01x01_Pin
- added L3: 2.2 uH, footprints:IND_PA4332.222NLT, symbol Device:L
- added R27: 100k, Resistor_SMD:R_0603_1608Metric, symbol Device:R_Small
- added R28: 562kΩ, Resistor_SMD:R_0805_2012Metric, symbol Device:R_Small
- added R29: 180kΩ, Resistor_SMD:R_0805_2012Metric, symbol Device:R_Small
- added U2: PRTR5V0U2X, Package_TO_SOT_SMD:SOT-143, symbol Power_Protection:PRTR5V0U2X
- added U3: ESP32-S3-MINI-1U, RF_Module:ESP32-S2-MINI-1U, symbol RF_Module:ESP32-S3-MINI-1U
- added U5: TPS62160DSG, Package_SON:WSON-8-1EP_2x2mm_P0.5mm_EP0.9x1.6mm_ThermalVias, symbol Regulator_Switching:TPS62160DSG
- renumbered C18 to C11, C19 to C12, C17 to C13, C15 to C16, C5 to C17, C6 to C18, C16 to C19, C8 to C20, C9 to C21, C20 to C23, C10 to C24, C11 to C25, Q9 to Q10, Q10 to Q11, Q12 to Q2, Q5 to Q4, Q7 to Q5, Q2 to Q6, Q4 to Q7, Q6 to Q8, Q8 to Q9, R2 to R1, R7 to R10, R8 to R11, R9 to R12, R4 to R13, R13 to R14, R19 to R15, R21 to R16, R10 to R17, R14 to R18, R22 to R19, R11 to R2, R23 to R20, R24 to R21, R25 to R22, R26 to R23, R27 to R24, R1 to R25, R5 to R26, R15 to R3, R16 to R4, R3 to R5, R12 to R6, R17 to R7, R18 to R8, R6 to R9, SW2 to SW1, U3 to U4
Connections:
- net +3V3: now also U3.3 (3V3)
- net BL_OUT: now also U3.22 (IO18)
- net BOOTMODE: now also U3.4 (IO0)
- net CLK_OUT: now also U3.18 (IO14)
- net D+: now also U2.3 (I/O2), U3.24 (USB_D+)
- net D-: now also U2.2 (I/O1), U3.23 (USB_D-)
- net DAT_OUT: now also U3.19 (IO15)
- net GND: now also C14.2, C15.2, C22.2, R29.2, U2.1 (GND), U3.1 (GND), U3.2 (GND), U3.42 (GND), U3.43 (GND), U3.44 (IO46), U3.46 (GND), U3.47 (GND), U3.48 (GND), U3.49 (GND), U3.50 (GND), U3.51 (GND), U3.52 (GND), U3.53 (GND), U3.54 (GND), U3.55 (GND), U3.56 (GND), U3.57 (GND), U3.58 (GND), U3.59 (GND), U3.60 (GND), U3.61 (GND), U3.62 (GND), U3.63 (GND), U3.64 (GND), U3.65 (GND), U5.1 (PGND), U5.4 (AGND), U5.9 (PAD)
- net LE_OUT: now also U3.20 (IO16)
- net POL_OUT: now also U3.21 (IO17)
- net at R25.2, SW1.B: now also U3.45 (EN)
- net at R26.1: now also U3.41 (IO45)
- net at S2.2: now also U3.13 (IO9)
- net VBUS: now reaches J2.A4 (VBUS), J2.A9 (VBUS), J2.B4 (VBUS), J2.B9 (VBUS)
- net VBUS: now also F1.1
- new net: R27.2, U5.8 (PG)
- new net: R28.2, R29.1, U5.5 (FB)
- new net: L3.1, U5.7 (SW)
- new net +3.3V: C22.1, L3.2, R27.1, R28.1, U5.6 (VOS)
- new net +5V: C14.1, C15.1, F1.2, J3.1 (Pin_1), U2.4 (VCC), U5.2 (VIN), U5.3 (EN)
- no-connect marks 10 -> 9
Other:
- moved on the sheet: C11, C12, C13, C16, C19, C23, L2, Rfbb1, Rfbt1, U4

Commit message: Shenanigans
Parts:
- removed C17: 10uF, Capacitor_SMD:C_0805_2012Metric, symbol Device:C
- removed C18, C20, C21, C25: 100nF, Capacitor_SMD:C_0805_2012Metric, symbol Device:C
- removed C22: 22 uF, Capacitor_SMD:C_0603_1608Metric, symbol Device:C_Small
- removed F1: 500 mA, Fuse:Fuse_1206_3216Metric, symbol Device:Polyfuse
- removed J3: VBUS, Connector_PinHeader_2.54mm:PinHeader_1x01_P2.54mm_Vertical, symbol Connector:Conn_01x01_Pin
- removed L3: 2.2 uH, footprints:IND_PA4332.222NLT, symbol Device:L
- removed Q10, Q11, Q2, Q3, Q4, Q5, Q6, Q7, Q8, Q9: MMBTA06, Package_TO_SOT_SMD:SOT-23, symbol Transistor_BJT:MMBTA06
- removed R1, R13, R14, R15, R16, R2, R21, R22, R23, R3, R4, R5, R6, R7, R8: 10k, Resistor_SMD:R_0805_2012Metric, symbol Device:R_Small
- removed R17, R18, R19, R20, R24: 4.7k, Resistor_SMD:R_0805_2012Metric, symbol Device:R_Small
- removed R27: 100k, Resistor_SMD:R_0603_1608Metric, symbol Device:R_Small
- removed R28: 562kΩ, Resistor_SMD:R_0805_2012Metric, symbol Device:R_Small
- removed R29: 180kΩ, Resistor_SMD:R_0805_2012Metric, symbol Device:R_Small
- removed Rfbb1: 10 kOhm, Resistor_SMD:R_0603_1608Metric, symbol Device:R_Small
- removed S2: TL3340AF160QG, TL3340AF160QG:TL3340, symbol Personal:TL3340AF160QG
- removed U2: PRTR5V0U2X, Package_TO_SOT_SMD:SOT-143, symbol Power_Protection:PRTR5V0U2X
- removed U5: TPS62160DSG, Package_SON:WSON-8-1EP_2x2mm_P0.5mm_EP0.9x1.6mm_ThermalVias, symbol Regulator_Switching:TPS62160DSG
- added C10: 100nF, Capacitor_SMD:C_0603_1608Metric, symbol Device:C
- added C9: 10uF, Capacitor_SMD:C_0603_1608Metric, symbol Device:C
- added Rffb1: 10k Ohm, Resistor_SMD:R_0603_1608Metric, symbol Device:R_Small
- added SW2: EN, footprints:KH-6X6X5H-STM_SKE, symbol 2026-02-17_13-05-37:KH-6X6X5H-STM
- C11, C12: footprint Capacitor_SMD:C_0805_2012Metric -> Capacitor_SMD:C_0603_1608Metric; LCSC C6684487 -> C1691
- C13, C16: LCSC C22401913 -> C14663
- C15: value 10uF -> 100nF; LCSC C19702 -> C14663
- C19: footprint Capacitor_SMD:C_0402_1005Metric -> Resistor_SMD:R_0805_2012Metric; LCSC C22401913 -> C1804
- C24: value 100nF -> 47uF; footprint Capacitor_SMD:C_0805_2012Metric -> Capacitor_SMD:C_1206_3216Metric; LCSC C28233 -> C96123
- R10, R9: footprint Resistor_SMD:R_0805_2012Metric -> Resistor_SMD:R_0603_1608Metric; LCSC Part # C27834 -> C23186
- R11, R12: footprint Resistor_SMD:R_0805_2012Metric -> Resistor_SMD:R_0603_1608Metric; LCSC Part # C17561 -> C23345
- R25, R26: value 10k -> 10k Ohm; footprint Resistor_SMD:R_0805_2012Metric -> Resistor_SMD:R_0603_1608Metric; LCSC Part # C17414 -> C2930027
- Rfbt1: value 30 kOhm -> 30.9 kOhm; footprint Resistor_SMD:R_0805_2012Metric -> Resistor_SMD:R_0603_1608Metric; LCSC Part # C2907255 -> C2930090
- U3: LCSC Part # (none) -> C2980299
- U4: LCSC Part # (none) -> C2877547
Connections:
- net +5V is gone; now on net +3V3: C14.1, C15.1
- net +3V3: now also C10.1, C9.1
- net D+: now also R11.2; no longer R12.2
- net D-: now also R12.2; no longer R11.2
- net GND: now also SW1.D, C10.2, C9.2, Rffb1.2, SW2.A, SW2.B
- net at C19.2, Rfbt1.2, U4.6 (VFB): now also Rffb1.1
- net at SW1.A: now also SW1.B, U3.45 (EN)
- net at J2.A6 (D+), J2.B6 (D+): now also R11.1; no longer R12.1
- net at J2.A7 (D-), J2.B7 (D-): now also R12.1; no longer R11.1
- net at U3.13 (IO9): now also SW2.C, SW2.D
- net MOSI: now reaches U3.14 (IO10)
- net SCLK: now reaches U3.15 (IO11)
- net CS: now reaches U3.16 (IO12)
- net GPIO1: now reaches U3.25 (IO21)
- net GPIO2: now reaches U3.26 (IO26)
- net GPIO3: now reaches U3.28 (IO33)
- net GPIO4: now reaches U3.29 (IO34)
- net GPIO5: now reaches U3.31 (IO35)
- net GPIO6: now reaches U3.32 (IO36)
- net BL_OUT: no longer names the net of U3.22 (IO18)
- net CLK_OUT: no longer names the net of U3.18 (IO14)
- net DAT_OUT: no longer names the net of U3.19 (IO15)
- net LE_OUT: no longer names the net of U3.20 (IO16)
- net POL_OUT: no longer names the net of U3.21 (IO17)
- net VBUS: no longer names the net of J2.A4 (VBUS), J2.A9 (VBUS), J2.B4 (VBUS), J2.B9 (VBUS)
- now unconnected: R25.2
- no-connect marks 9 -> 8

Commit message: FPGA time
Parts:
- removed J2: USB_C_Receptacle_USB2.0, Connector_USB:USB_C_Receptacle_HRO_TYPE-C-31-M-12, symbol Connector:USB_C_Receptacle_USB2.0
- removed R10, R9: 5.1k, Resistor_SMD:R_0603_1608Metric, symbol Device:R
- removed R11, R12: 22, Resistor_SMD:R_0603_1608Metric, symbol Device:R
- removed R25, R26: 10k Ohm, Resistor_SMD:R_0603_1608Metric, symbol Device:R_Small
- removed S1: SSSS811101, footprints:SSSS811101, symbol Personal:SSSS811101
- removed SW1, SW2: EN, footprints:KH-6X6X5H-STM_SKE, symbol 2026-02-17_13-05-37:KH-6X6X5H-STM
- removed U3: ESP32-S3-MINI-1U, RF_Module:ESP32-S2-MINI-1U, symbol RF_Module:ESP32-S3-MINI-1U
- added C80: 100 nF, Capacitor_SMD:C_0805_2012Metric, symbol Device:C
- added J6: USB_C_Receptacle_USB2.0, Connector_USB:USB_C_Receptacle_HRO_TYPE-C-31-M-12, symbol Connector:USB_C_Receptacle_USB2.0
- added Q8: SS8050, Package_TO_SOT_SMD:SOT-23, symbol Simulation_SPICE:NPN
- added R39, R40: 5.1k, Resistor_SMD:R_0805_2012Metric, symbol Device:R
- added R41, R42: 22, Resistor_SMD:R_0805_2012Metric, symbol Device:R
- added R43, R44: 10k Ohm, Resistor_SMD:R_0805_2012Metric, symbol Device:R_Small
- added R45: 4.7k, Resistor_SMD:R_0603_1608Metric, symbol Device:R_Small
- added R46: 0 ohm, Resistor_SMD:R_0805_2012Metric, symbol Device:R
- added SS8050: NPN, Package_TO_SOT_SMD:SOT-23, symbol Simulation_SPICE:NPN
- added SW3, SW4: EN, footprints:KH-6X6X5H-STM_SKE, symbol 2026-02-17_13-05-37:KH-6X6X5H-STM
- added U7: ESP32-WROOM-32E-R2, RF_Module:ESP32-WROOM-32D, symbol RF_Module:ESP32-WROOM-32E-R2
- C11, C12: LCSC C1691 -> C92487
- C19: LCSC C1804 -> C107110
- C23: LCSC C441864 -> C45783
- Rffb1: LCSC Part # C2930027 -> C25804
Connections:
- net +3V3: now also C80.1, R45.1, R46.1, U7.2 (VDD)
- net CS: now also U7.23 (IO15)
- net D+: now also R42.2
- net D-: now also R41.2
- net GND: now also C80.2, J6.A1 (GND), J6.A12 (GND), J6.B1 (GND), J6.B12 (GND), J6.S1 (SHIELD), R39.1, R40.2, SW3.C, SW4.A, SW4.B, U7.1 (GND), U7.15 (GND), U7.24 (IO2), U7.38 (GND), U7.39 (GND)
- net GPIO1: now also U7.30 (IO18)
- net GPIO2: now also U7.31 (IO19)
- net GPIO3: now also U7.33 (IO21)
- net GPIO4: now also U7.36 (IO22)
- net GPIO5: now also U7.37 (IO23)
- net GPIO6: now also U7.10 (IO25)
- net MOSI: now also U7.16 (IO13)
- net SCLK: now also U7.13 (IO14)
- new net: SW4.C, SW4.D, U7.14 (IO12)
- new net: Q8.1 (C), R46.2, SW3.B, U7.3 (EN)
- new net: J6.B5 (CC2), R40.1
- new net: J6.A4 (VBUS), J6.A9 (VBUS), J6.B4 (VBUS), J6.B9 (VBUS)
- new net: J6.A5 (CC1), R39.2
- new net: J6.A6 (D+), J6.B6 (D+), R42.1
- new net: J6.A7 (D-), J6.B7 (D-), R41.1
- new net: Q8.2 (B), R43.2
- new net: R44.2, SS8050.2 (B)
- new net GPIO0: R45.2, SS8050.1 (C), U7.25 (IO0)
- new net RX_IN: U7.35 (TXD0/IO1)
- new net TX_OUT: U7.34 (RXD0/IO3)
- new net UART/DTR: R43.1, SS8050.3 (E)
- new net UART/RTS: Q8.3 (E), R44.1
- no-connect marks 8 -> 9
Other:
- added sheet UART (ch430G.kicad_sch)
