File: Psu/HighEffNixiPSU/mcu.kicad_sch (KiCad schematic)
At the start: 30 parts, among them J6 USB_C_Receptacle_USB2.0, Q8 SS8050, SW3 EN, SW4 EN, U4 TPS562202, U7 ESP32-WROOM-32E-R2

Commit message: jfahefh
Parts:
- removed R45: 4.7k, Resistor_SMD:R_0603_1608Metric, symbol Device:R_Small
- removed R46: 0 ohm, Resistor_SMD:R_0805_2012Metric, symbol Device:R
- added SW5: BOOT0, footprints:KH-6X6X5H-STM_SKE, symbol 2026-02-17_13-05-37:KH-6X6X5H-STM
- SW4: value EN -> CAL
Connections:
- net GND: now also SW3.D, SW5.C, SW5.D
- net GPIO0: now also SW5.A, SW5.B
- net at Q8.1 (C), SW3.B, U7.3 (EN): now also SW3.A
- no-connect marks 9 -> 14
