File: XC6SLX16-FTG256/XC6SLX16-FTG256.kicad_sch (KiCad schematic)
At the start: 41 parts, among them J1 DE15_Pins_HighDensity, J2 Bank 0, J3 Bank 1, J4 Bank 2, J5 Bank 3, Q2 SS8050, U1 ICE40HX1K-TQ144, U2 W25Q32JVSS

Commit message: FPGA time
Parts:
- removed C16, C18: 100 nF, Capacitor_SMD:C_0603_1608Metric, symbol Device:C_Small
- removed C17, C19: 10 uF, Capacitor_SMD:C_0603_1608Metric, symbol Device:C_Small
- removed J3: Bank 1, Connector_PinHeader_2.54mm:PinHeader_1x25_P2.54mm_Vertical, symbol Connector:Conn_01x25_Pin
- removed J4: Bank 2, Connector_PinHeader_2.54mm:PinHeader_1x20_P2.54mm_Vertical, symbol Connector:Conn_01x20_Pin
- removed unit 2 of U1
- removed unit 3 of U1
- added C22: 100 nF, Capacitor_SMD:C_0603_1608Metric, symbol Device:C_Small
- added Y1: 12MHZ, Crystal:Crystal_SMD_3225-4Pin_3.2x2.5mm, symbol Oscillator:ASCO
Connections:
- net +3V3: now also C22.2, Y1.1 (Tri-State), Y1.4 (VDD)
- net GND: now also C22.1, Y1.2 (GND)
- net at J5.13 (Pin_13): no longer U1.21 (IOL_7A_GBIN6)
- new net CLK: U1.21 (IOL_7A_GBIN6), Y1.3 (OUT)
- no-connect marks 10 -> 11
Other:
- added sheet sdram (sdram.kicad_sch)
- moved on the sheet: C13, C14, J5, U1D
