File: XC6SLX16-FTG256/XC6SLX16-FTG256.kicad_pcb (KiCad board)
At the start: 2 copper layers, 84.8 x 100.3 mm, 67 parts, among them J1 DE15_Pins_HighDensity, J2 Bank 0, J3 Bank 1, J4 Bank 2, J5 Bank 3, J6 USB_C_Receptacle_USB2.0, J7 ESP-BANK-1, Q1 SS8050, Q2 SS8050, SW2 EN, U1 ICE40HX1K-TQ144, U2 W25Q32JVSS, U3 LD1117S33TR_SOT223, U4 AP2112K-1.2, U5 ESP32-WROOM-32E-R2, U6 CH340G, Y3 12 MHz

Commit message: FPGA time
Parts:
- removed J4: Bank 2, Connector_PinHeader_2.54mm:PinHeader_1x20_P2.54mm_Vertical
- added C22: 100 nF, Capacitor_SMD:C_0603_1608Metric, F.Cu at (72.9, 68.3)
- added C23: 100 nF, Capacitor_SMD:C_0603_1608Metric, F.Cu at (63.2, 81.3)
- added C24: 10 uF, Capacitor_SMD:C_0603_1608Metric, F.Cu at (63.2, 74.6)
- added C25: 100 nF, Capacitor_SMD:C_0603_1608Metric, F.Cu at (70.2, 67.2)
- added C26: 100 nF, Capacitor_SMD:C_0603_1608Metric, F.Cu at (63.2, 94.0)
- added U7: IS42S16400J-xC, Package_SO:TSOP-II-54_22.2x10.16mm_P0.8mm, F.Cu at (71.6, 83.6)
- added Y1: 12MHZ, Crystal:Crystal_SMD_3225-4Pin_3.2x2.5mm, F.Cu at (76.3, 67.3)
- J3: value Bank 1 -> Bank 2; footprint Connector_PinHeader_2.54mm:PinHeader_1x25_P2.54mm_Vertical -> Connector_PinHeader_2.54mm:PinHeader_1x09_P2.54mm_Vertical
- moved J7 188.1 mm to (52.4, 117.4)
- moved R17 177.9 mm to (82.0, 137.8), turned to -90 degrees
- moved R18 172.7 mm to (86.5, 137.8), turned to 90 degrees
- moved R19 169.6 mm to (90.5, 142.6)
- moved R20 167.7 mm to (90.6, 140.6)
- moved C18 167.4 mm to (65.9, 70.3), turned to -90 degrees
- moved C16 167.0 mm to (63.2, 72.6)
- moved C19 163.4 mm to (70.2, 70.3), turned to -90 degrees
- moved C17 163.1 mm to (67.9, 70.3), turned to -90 degrees
- moved C2 160.6 mm to (60.9, 139.0), turned to -90 degrees
- moved C3 154.2 mm to (63.4, 130.8), turned to 90 degrees
- moved C1 150.3 mm to (72.2, 136.5)
- moved R21 148.7 mm to (105.6, 128.9), turned to 90 degrees
- moved C4 147.6 mm to (68.3, 127.5), turned to 90 degrees
- moved C6 145.8 mm to (80.4, 66.8), turned to -90 degrees
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Connections:
- J5 pad 13: Net-(J5-Pin_13) -> unconnected-(J5-Pin_13-Pad13)
- U1 pad 101: Net-(J3-Pin_20) -> Net-(U1B-IOR_67)
- U1 pad 102: Net-(J3-Pin_21) -> Net-(U1B-IOR_68)
- U1 pad 104: Net-(J3-Pin_22) -> Net-(U1B-IOR_69)
- U1 pad 105: Net-(J3-Pin_23) -> Net-(U1B-IOR_70)
- U1 pad 106: Net-(J3-Pin_24) -> Net-(U1B-IOR_71)
- U1 pad 107: Net-(J3-Pin_25) -> Net-(U1B-IOR_72)
- U1 pad 21: Net-(J5-Pin_13) -> /CLK
- U1 pad 50: Net-(J4-Pin_12) -> Net-(J3-Pin_1)
- U1 pad 52: Net-(J4-Pin_13) -> Net-(J3-Pin_2)
- U1 pad 56: Net-(J4-Pin_14) -> Net-(J3-Pin_3)
- U1 pad 58: Net-(J4-Pin_15) -> Net-(J3-Pin_4)
- U1 pad 60: Net-(J4-Pin_16) -> Net-(J3-Pin_5)
- U1 pad 61: Net-(J4-Pin_17) -> Net-(J3-Pin_6)
- U1 pad 62: Net-(J4-Pin_18) -> Net-(J3-Pin_7)
- U1 pad 63: Net-(J4-Pin_19) -> Net-(J3-Pin_8)
- U1 pad 64: Net-(J4-Pin_20) -> Net-(J3-Pin_9)
- U1 pad 73: Net-(J3-Pin_1) -> Net-(U1B-IOR_48)
- U1 pad 74: Net-(J3-Pin_2) -> Net-(U1B-IOR_49)
- U1 pad 75: Net-(J3-Pin_3) -> Net-(U1B-IOR_50)
- U1 pad 76: Net-(J3-Pin_4) -> Net-(U1B-IOR_51)
- U1 pad 78: Net-(J3-Pin_5) -> Net-(U1B-IOR_52)
- U1 pad 79: Net-(J3-Pin_6) -> Net-(U1B-IOR_53)
- U1 pad 80: Net-(J3-Pin_7) -> Net-(U1B-IOR_54)
- U1 pad 81: Net-(J3-Pin_8) -> Net-(U1B-IOR_55)
- U1 pad 87: Net-(J3-Pin_9) -> Net-(U1B-IOR_56)
- U1 pad 88: Net-(J3-Pin_10) -> Net-(U1B-IOR_57)
- U1 pad 90: Net-(J3-Pin_11) -> Net-(U1B-IOR_58)
- U1 pad 91: Net-(J3-Pin_12) -> Net-(U1B-IOR_59)
- U1 pad 93: Net-(J3-Pin_13) -> Net-(U1B-IOR_60_GBIN3)
- U1 pad 94: Net-(J3-Pin_14) -> Net-(U1B-IOR_61_GBIN2)
- U1 pad 95: Net-(J3-Pin_15) -> Net-(U1B-IOR_62)
- U1 pad 96: Net-(J3-Pin_16) -> Net-(U1B-IOR_63)
- U1 pad 97: Net-(J3-Pin_17) -> Net-(U1B-IOR_64)
- U1 pad 98: Net-(J3-Pin_18) -> Net-(U1B-IOR_65)
- U1 pad 99: Net-(J3-Pin_19) -> Net-(U1B-IOR_66)
Routing:
- net +3V3: track 0.00 -> 581.5 mm, vias 0 -> 5
- net +1V2: track 0.00 -> 101.3 mm, vias 0 -> 6
- net /mcu/SDO: track 0.00 -> 89.1 mm, vias 0 -> 8
- net Net-(J7-Pin_5): track 0.00 -> 86.3 mm, vias 0 -> 1
- net /mcu/SDI: track 0.00 -> 83.0 mm, vias 0 -> 8
- net Net-(J7-Pin_4): track 0.00 -> 82.7 mm, vias 0 -> 1
- net Net-(J7-Pin_10): track 0.00 -> 80.6 mm, vias 0 -> 2
- net Net-(J7-Pin_3): track 0.00 -> 79.5 mm, vias 0 -> 1
- net /mcu/SS: track 0.00 -> 79.5 mm, vias 0 -> 8
- net /mcu/SCK: track 0.00 -> 78.6 mm, vias 0 -> 8
- net Net-(J7-Pin_11): track 0.00 -> 78.4 mm, vias 0 -> 5
- net Net-(J7-Pin_2): track 0.00 -> 78.3 mm, vias 0 -> 2
- net Net-(J7-Pin_12): track 0.00 -> 74.6 mm, vias 0 -> 4
- net Net-(J7-Pin_1): track 0.00 -> 74.5 mm, vias 0 -> 1
- net Net-(J7-Pin_9): track 0.00 -> 72.1 mm, vias 0 -> 6
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- added copper zone on B.Cu, net GND
- added copper zone on F.Cu, net GND
