File: Psu/USB-PD-CH224K/USB-PD-CH224K.kicad_sch (KiCad schematic)
At the start: 15 parts, among them J1 USB_C_Receptacle_USB2.0_16P, SW1 CFG, U1 CH224K, U2 MCP1799x-500xxTT

Commit message: Rev 2 of ch224k)
Parts:
- removed C2, C3: 1 uF, Capacitor_SMD:C_0603_1608Metric, symbol Device:C_Small
- removed U2: MCP1799x-500xxTT, Package_TO_SOT_SMD:SOT-23, symbol Regulator_Linear:MCP1799x-500xxTT
- added D1: BZT52B3V3, Diode_SMD:D_SOD-123, symbol Diode:BZT52Bxx
- added R10: 100k, Resistor_SMD:R_0603_1608Metric, symbol Device:R_Small
- added R8, R9: 22, Resistor_SMD:R_0603_1608Metric, symbol Device:R_Small
Connections:
- net +3V3: now also D1.1 (K), R10.2
- net GND: now also D1.2 (A)
- net VBUS: now also R10.1
- net at J1.A6 (D+): now also J1.B6 (D+), R9.2
- net at J1.A7 (D-): now also J1.B7 (D-), R8.1
- net at U1.4 (DP): now also R9.1
- net at U1.5 (DM): now also R8.2
- no-connect marks 9 -> 3

Commit message: fdcj
Parts:
- added C2: 1 uF, Capacitor_SMD:C_0603_1608Metric, symbol Device:C_Small
- added D2: LED, LED_SMD:LED_0603_1608Metric, symbol Device:LED
- added D3: SD24C-01F, Diode_SMD:D_SOD-323, symbol Diode:SD24C-01F
- added D4: PESD5V0L4UG, Package_TO_SOT_SMD:SOT-353_SC-70-5, symbol Power_Protection:PESD5V0L4UG
- added F2: 3A, Fuse:Fuse_0603_1608Metric, symbol Device:Polyfuse
- added R3: 1k, Resistor_SMD:R_0603_1608Metric, symbol Device:R_Small
- R10: value 100k -> 10k
Connections:
- net +3V3: now also R3.2
- net GND: now also C2.2, D3.2 (A2), D4.2 (A)
- net VBUS: now also C2.1, D3.1 (A1), F2.2; no longer J1.A4 (VBUS), J1.A9 (VBUS), J1.B4 (VBUS), J1.B9 (VBUS)
- net at R9.1, U1.4 (DP): now also D4.3 (K2)
- net at R8.2, U1.5 (DM): now also D4.1 (K1)
- net at J1.A5 (CC1), U1.7 (CC1): now also D4.4 (K3)
- net at J1.B5 (CC2), U1.6 (CC2): now also D4.5 (K4)
- net PG: now reaches U1.10 (PG)
- net PG: now also D2.1 (K)
- new net: D2.2 (A), R3.1
- new net: F2.1, J1.A4 (VBUS), J1.A9 (VBUS), J1.B4 (VBUS), J1.B9 (VBUS)
- no-connect marks 3 -> 2
Other:
- moved on the sheet: C1, R1, R2, R5, R6, R7, SW1, TP1, U1
