File: Misc/ADS1293CISQ/ADS1293CISQ.kicad_sch (KiCad schematic)
At the start: 41 parts, among them IC1 ADS1293CISQ_NOPB, IC2 GD5F1GQ5REYIGR, J1 35RASMT4BHNTRX, J2 SPI, J3 SPI_FLASH, J6 VIn, J7 DESC, J8 35RASMT4BHNTRX, Q1 Q_PMOS_GSD, Y2 4.096 MHz

Commit message: dfjaj
Parts:
- removed J2: SPI, Connector_PinHeader_2.54mm:PinHeader_1x04_P2.54mm_Vertical, symbol Connector:Conn_01x04_Pin
- removed J3: SPI_FLASH, Connector_PinHeader_2.54mm:PinHeader_1x04_P2.54mm_Vertical, symbol Connector:Conn_01x04_Pin
- added J2: SPI, Connector_PinHeader_2.54mm:PinHeader_1x05_P2.54mm_Vertical, symbol Connector:Conn_01x05_Pin
- IC2: footprint SON127P800X600X80-9N-D -> footprints:SON127P800X600X80-9N-D
Connections:
- net CSB: now reaches IC2.1 (CS#)
- net CSB: now also J2.5 (Pin_5)
- net SDO: now reaches IC2.2 (SO/_SIO1)
- net SDO: now also IC1.19 (SDO), J2.1 (Pin_1)
- net SDI: now reaches IC2.5 (SI/_SIO0)
- net SDI: now also IC1.18 (SDI), J2.2 (Pin_2)
- net SCLK: now reaches IC2.6 (SCLK)
- net SCLK: now also IC1.17 (SCLK), J2.3 (Pin_3)
- net at IC1.16 (CSB): now also J2.4 (Pin_4)
Changed lines of the file:
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@@
 	(wire
 		(pts
-			(xy 269.24 149.86) (xy 210.82 149.86)
-		)
-		(stroke
-			(width 0)
-			(type default)
-		)
-	)
-	(wire
-		(pts
 			(xy 110.49 36.83) (xy 110.49 49.53)
 		)
@@
 	(wire
 		(pts
-			(xy 267.97 148.59) (xy 212.09 148.59)
-		)
-		(stroke
-			(width 0)
-			(type default)
-		)
-	)
-	(wire
-		(pts
 			(xy 109.22 138.43) (xy 109.22 147.32)
 		)
@@
 	(wire
 		(pts
-			(xy 212.09 123.19) (xy 223.52 123.19)
-		)
-		(stroke
-			(width 0)
-			(type default)
-		)
-	)
-	(wire
-		(pts
 			(xy 200.66 96.52) (xy 200.66 105.41)
 		)
@@
 	(wire
 		(pts
-			(xy 269.24 135.89) (xy 269.24 149.86)
-		)
-		(stroke
-			(width 0)
-			(type default)
-		)
-	)
-	(wire
-		(pts
 			(xy 115.57 59.69) (xy 115.57 68.58)
 		)
@@
 	(wire
 		(pts
-			(xy 212.09 148.59) (xy 212.09 123.19)
-		)
-		(stroke
-			(width 0)
-			(type default)
-		)
-	)
-	(wire
-		(pts
 			(xy 158.75 162.56) (xy 158.75 163.83)
 		)
@@
 	(wire
 		(pts
-			(xy 269.24 133.35) (xy 267.97 133.35)
-		)
-		(stroke
-			(width 0)
-			(type default)
-		)
-	)
-	(wire
-		(pts
 			(xy 110.49 49.53) (xy 110.49 57.15)
 		)
@@
 	(wire
 		(pts
-			(xy 210.82 149.86) (xy 210.82 125.73)
-		)
-		(stroke
-			(width 0)
-			(type default)
-		)
-	)
-	(wire
-		(pts
-			(xy 267.97 133.35) (xy 267.97 148.59)
-		)
-		(stroke
-			(width 0)
-			(type default)
-		)
-	)
-	(wire
-		(pts
 			(xy 95.25 147.32) (xy 104.14 147.32)
 		)
@@
 	(wire
 		(pts
-			(xy 210.82 125.73) (xy 223.52 125.73)
-		)
-		(stroke
-			(width 0)
-			(type default)
-		)
-	)
-	(wire
-		(pts
 			(xy 168.91 154.94) (xy 163.83 154.94)
 		)
@@
 		)
 	)
+	(label "SCLK"
+		(at 156.21 96.52 180)
+		(effects
+			(font
+				(size 1.27 1.27)
+			)
+			(justify right bottom)
+		)
+	)
 	(label "ALARMB"
 		(at 133.35 101.6 0)
@@
 		)
 	)
+	(label "SDI"
+		(at 156.21 93.98 180)
+		(effects
+			(font
+				(size 1.27 1.27)
+			)
+			(justify right bottom)
+		)
+	)
+	(label "SCLK"
+		(at 269.24 128.27 0)
+		(effects
+			(font
+				(size 1.27 1.27)
+			)
+			(justify left bottom)
+		)
+	)
+	(label "CSB"
+		(at 156.21 101.6 180)
+		(effects
+			(font
+				(size 1.27 1.27)
+			)
+			(justify right bottom)
+		)
+	)
 	(label "RLDOUT"
 		(at 95.25 147.32 180)
@@
 		)
 	)
+	(label "CSB"
+		(at 223.52 123.19 180)
+		(effects
+			(font
+				(size 1.27 1.27)
+			)
+			(justify right bottom)
+		)
+	)
 	(label "RLDOUT"
 		(at 110.49 119.38 270)
@@
 		)
 	)
+	(label "SDI"
+		(at 269.24 130.81 0)
+		(effects
+			(font
+				(size 1.27 1.27)
+			)
+			(justify left bottom)
+		)
+	)
+	(label "SDO"
+		(at 223.52 125.73 180)
+		(effects
+			(font
+				(size 1.27 1.27)
+			)
+			(justify right bottom)
+		)
+	)
 	(label "XTAL1"
 		(at 152.4 64.77 180)
@@
 		)
 	)
+	(label "SDO"
+		(at 156.21 91.44 180)
+		(effects
+			(font
+				(size 1.27 1.27)
+			)
+			(justify right bottom)
+		)
+	)
 	(label "LA"
 		(at 82.55 88.9 180)
@@
 			)
 		)
-		(property "Footprint" "SON127P800X600X80-9N-D"
+		(property "Footprint" "footprints:SON127P800X600X80-9N-D"
 			(at 265.43 218.11 0)
 			(hide yes)
@@
 	)
 	(symbol
-		(lib_id "Connector:Conn_01x04_Pin")
-		(at 274.32 130.81 0)
-		(mirror y)
-		(unit 1)
-		(body_style 1)
-		(exclude_from_sim no)
-		(in_bom yes)
-		(on_board yes)
-		(in_pos_files yes)
-		(dnp no)
-		(fields_autoplaced yes)
-		(property "Reference" "J3"
-			(at 275.59 133.3501 0)
-			(show_name no)
-			(do_not_autoplace no)
-			(effects
-				(font
-					(size 1.27 1.27)
-				)
-				(justify right)
-			)
-		)
-		(property "Value" "SPI_FLASH"
-			(at 275.59 130.8101 0)
-			(show_name no)
-			(do_not_autoplace no)
-			(effects
-				(font
-					(size 1.27 1.27)
-				)
-				(justify right)
-			)
-		)
-		(property "Footprint" "Connector_PinHeader_2.54mm:PinHeader_1x04_P2.54mm_Vertical"
-			(at 274.32 130.81 0)
-			(hide yes)
-			(show_name no)
-			(do_not_autoplace no)
-			(effects
-				(font
-					(size 1.27 1.27)
-				)
-			)
-		)
-		(property "Datasheet" ""
-			(at 274.32 130.81 0)
-			(hide yes)
-			(show_name no)
-			(do_not_autoplace no)
-			(effects
-				(font
-					(size 1.27 1.27)
-				)
-			)
-		)
-		(property "Description" "Generic connector, single row, 01x04, script generated"
-			(at 274.32 130.81 0)
-			(hide yes)
-			(show_name no)
-			(do_not_autoplace no)
-			(effects
-				(font
-					(size 1.27 1.27)
-				)
-			)
-		)
-		(pin "4"
-		)
-		(pin "2"
-		)
-		(pin "1"
-		)
-		(pin "3"
-		)
-		(instances
-			(project "ADS1293CISQ"
-				(path "/72e0f053-d8ab-4173-a900-56046048e6d8"
-					(reference "J3")
-					(unit 1)
-				)
-			)
-		)
-	)
-	(symbol
 		(lib_id "symbols:ADS1293CISQ_NOPB")
 		(at 100.33 86.36 0)
@@
 	)
 	(symbol
-		(lib_id "Connector:Conn_01x04_Pin")
-		(at 161.29 93.98 0)
+		(lib_id "Connector:Conn_01x05_Pin")
+		(at 161.29 96.52 0)
 		(mirror y)
 		(unit 1)
@@
 		(fields_autoplaced yes)
 		(property "Reference" "J2"
-			(at 162.56 96.5201 0)
+			(at 162.56 97.7901 0)
 			(show_name no)
 			(do_not_autoplace no)
@@
 		)
 		(property "Value" "SPI"
-			(at 162.56 93.9801 0)
+			(at 162.56 95.2501 0)
 			(show_name no)
 			(do_not_autoplace no)
@@
 			)
 		)
-		(property "Footprint" "Connector_PinHeader_2.54mm:PinHeader_1x04_P2.54mm_Vertical"
-			(at 161.29 93.98 0)
+		(property "Footprint" "Connector_PinHeader_2.54mm:PinHeader_1x05_P2.54mm_Vertical"
+			(at 161.29 96.52 0)
 			(hide yes)
 			(show_name no)
@@
 		)
 		(property "Datasheet" ""
-			(at 161.29 93.98 0)
+			(at 161.29 96.52 0)
 			(hide yes)
 			(show_name no)
@@
 			)
 		)
-		(property "Description" "Generic connector, single row, 01x04, script generated"
-			(at 161.29 93.98 0)
+		(property "Description" "Generic connector, single row, 01x05, script generated"
+			(at 161.29 96.52 0)
 			(hide yes)
 			(show_name no)
@@
 			)
 		)
-		(pin "4"
-		)
-		(pin "2"
-		)
 		(pin "1"
 		)
 		(pin "3"
 		)
+		(pin "4"
+		)
+		(pin "5"
+		)
+		(pin "2"
+		)
 		(instances
