File: Misc/ADS1293CISQ/ADS1293CISQ.kicad_sch (KiCad schematic)
At the start: 40 parts, among them IC1 ADS1293CISQ_NOPB, IC2 GD5F1GQ5REYIGR, J1 35RASMT4BHNTRX, J2 SPI, J6 VIn, J7 DESC, J8 35RASMT4BHNTRX, Q1 Q_PMOS_GSD, Y2 4.096 MHz

Commit message: AMP V2
Parts:
- C6: value 47 pF -> 1.5 nF
Changed lines of the file:
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@@
 			)
 		)
-		(property "Value" "47 pF"
+		(property "Value" "1.5 nF"
 			(at 106.6863 134.62 90)
 			(show_name no)
