File: Misc/ADS1293CISQ/ADS1293CISQ.kicad_pcb (KiCad board)
At the start: 4 copper layers, 48.3 x 24.6 mm, 40 parts, among them IC1 ADS1293CISQ_NOPB, IC2 GD5F1GQ5REYIGR, J1 35RASMT4BHNTRX, J2 SPI, J6 VIn, J7 DESC, J8 35RASMT4BHNTRX, Q1 Q_PMOS_GSD, Y2 4.096 MHz

Commit message: dkakw
Routing:
- net /SDI: track 30.6 -> 28.8 mm, vias 1 -> 0
- net /SDO: track 25.4 -> 26.0 mm

Commit message: AMP V2
Parts:
- C6: value 47 pF -> 1.5 nF
Changed lines of the file:
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@@
 				(font
 					(size 1.27 1.27)
+					(thickness 0.15)
 				)
 			)
@@
 			)
 		)
-		(property "Value" "47 pF"
+		(property "Value" "1.5 nF"
 			(at 0 1.16 90)
 			(layer "F.Fab")
@@
 			)
 		)
-		(property "LCSC" "C1567"
+		(property "LCSC" "C107022"
 			(at 0 0 0)
 			(layer "F.SilkS")
@@
 				(font
 					(size 1.27 1.27)
+					(thickness 0.15)
 				)
 			)
