File: Misc/adau1701-breakout/adau1701-breakout.kicad_sch (KiCad schematic)
At the start: 46 parts, among them J1 I2C, J2 MPx, J3 ADCx, J4 VOUTx, J5 MCLKx, J6 CTRL, SW2 RST, U1 ADAU1701, U2 24LC64, U3 5PB1108PGxx, U4 LD1117S18TR_SOT223, U7 MCP100-315D, Y1 ASV-24.576MHz

Commit message: dfjaj
Parts:
- removed J6: CTRL, Connector_PinHeader_2.54mm:PinHeader_1x03_P2.54mm_Vertical, symbol Connector:Conn_01x03_Pin
- removed U7: MCP100-315D, Package_TO_SOT_SMD:SOT-23-3, symbol Power_Supervisor:MCP100-315D
- added C48: 47 uF, Capacitor_SMD:CP_Elec_6.3x5.4, symbol Device:C_Polarized
- added J6: Ctrl, Connector_PinHeader_2.54mm:PinHeader_1x02_P2.54mm_Vertical, symbol Connector:Conn_01x02_Pin
- added R10, R5: 18k, Resistor_SMD:R_0603_1608Metric, symbol Device:R_Small
- Y1: value ASV-24.576MHz -> SX3M22.5792M20F30TNN; footprint Oscillator:Oscillator_SMD_Abracon_ASV-4Pin_7.0x5.1mm -> Crystal:Crystal_SMD_3225-4Pin_3.2x2.5mm
Connections:
- net GND: now also C48.2
- net RST: now also J6.1 (Pin_1)
- net WP: now also J6.2 (Pin_2)
- net at C23.1: now also R5.1; no longer U1.4 (ADC1)
- net at U1.2 (ADC0): now also R10.2; no longer C22.1
- net at C16.1, C17.1, U1.40 (CM): now also C48.1
- new net: R5.2, U1.4 (ADC1)
- new net: C22.1, R10.1
Other:
- moved on the sheet: C22, C23, J3, R8

Commit message: fdjf
Parts:
- removed C7: 1 uF, Capacitor_SMD:C_0603_1608Metric, symbol Device:C_Small
- removed C8: 100 nF, Capacitor_SMD:C_0603_1608Metric, symbol Device:C_Small
- removed U4: LD1117S18TR_SOT223, Package_TO_SOT_SMD:SOT-223-3_TabPin2, symbol Regulator_Linear:LD1117S18TR_SOT223
- added Q1: MMBT3906, Package_TO_SOT_SMD:SOT-23, symbol Transistor_BJT:MMBT3906
- added R11: 1k, Resistor_SMD:R_0603_1608Metric, symbol Device:R_Small
- C26: value 1 uF -> 10 uF
- C27: value 1 uF -> 100 nF
Connections:
- net +3V3: now also Q1.2 (E), R11.1; no longer C26.1
- net GND: now also C26.1, C27.1; no longer C26.2, C27.2, U1.17 (VDRIVE)
- net +1V8: no longer names the net of U1.13 (DVDD), U1.24 (DVDD)
- net +1V8: now also C26.2, C27.2, Q1.3 (C); no longer C27.1
- new net: Q1.1 (B), R11.2, U1.17 (VDRIVE)
