File: AMP/TPA3116D2DADR/TPA3116D2DADR.kicad_pcb (KiCad board)
At the start: 2 copper layers, 90 x 33.2 mm, 58 parts, among them IC1 TPA3116D2DADR, J1 Rin, J2 Lin, J3 Rout, J4 Lout, J7 PWR, Q1 BSC028N06LS3, U1 AMS1117-3.3, U2 LTC4359-DCB

Commit message: jahfd
Parts:
- removed Q1: BSC028N06LS3, Package_TO_SOT_SMD:TDSON-8-1
- added Q2: BSC028N06NSATMA1, footprints:TRANS_BSC028N06NSATMA1, F.Cu at (147.3, 117.9)
Routing:
- net Net-(D1-K): track 35.9 -> 34.2 mm
- net VCC: track 102.7 -> 103.4 mm
- net GND: vias 1 -> 2

Commit message: dfjaj
Routing:
- net GND: track 0.00 -> 24.1 mm, vias 2 -> 11
Changed lines of the file:
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@@
+	)
+	(segment
+		(start 144.48 119.74)
+		(end 144.48 120.98)
+		(width 0.3)
+		(layer "F.Cu")
+		(net "Net-(U2-GATE)")
+	)
+	(segment
+		(start 145.85 122.35)
+		(end 146.5025 122.35)
+		(width 0.3)
+		(layer "F.Cu")
+		(net "Net-(U2-GATE)")
+	)
+	(segment
+		(start 144.48 120.98)
+		(end 145.85 122.35)
+		(width 0.3)
+		(layer "F.Cu")
+		(net "Net-(U2-GATE)")
 	)
 	(segment
@@
 		(net "Net-(J3-Pin_1)")
 	)
+	(segment
+		(start 175.025 115.645)
+		(end 176.48 114.19)
+		(width 0.2)
+		(layer "F.Cu")
+		(net "GND")
+	)
+	(segment
+		(start 175.025 116.605)
+		(end 175.025 117.075)
+		(width 0.2)
+		(layer "F.Cu")
+		(net "GND")
+	)
+	(segment
+		(start 175.025 116.605)
+		(end 175.025 116.145)
+		(width 0.2)
+		(layer "F.Cu")
+		(net "GND")
+	)
+	(segment
+		(start 175.025 116.605)
+		(end 173.045 116.605)
+		(width 0.2)
+		(layer "F.Cu")
+		(net "GND")
+	)
+	(segment
+		(start 175.025 117.075)
+		(end 173.17 118.93)
+		(width 0.2)
+		(layer "F.Cu")
+		(net "GND")
+	)
+	(segment
+		(start 175.025 118.885)
+		(end 175.02 118.89)
+		(width 0.2)
+		(layer "F.Cu")
+		(net "GND")
+	)
+	(segment
+		(start 175.025 116.605)
+		(end 175.025 115.645)
+		(width 0.2)
+		(layer "F.Cu")
+		(net "GND")
+	)
+	(segment
+		(start 175.025 116.605)
+		(end 174.025 116.605)
+		(width 0.2)
+		(layer "F.Cu")
+		(net "GND")
+	)
+	(segment
+		(start 175.025 116.605)
+		(end 175.025 114.135)
+		(width 0.2)
+		(layer "F.Cu")
+		(net "GND")
+	)
+	(segment
+		(start 174.125 116.605)
+		(end 172.98 117.75)
+		(width 0.2)
+		(layer "F.Cu")
+		(net "GND")
+	)
+	(segment
+		(start 175.025 116.605)
+		(end 175.025 118.885)
+		(width 0.2)
+		(layer "F.Cu")
+		(net "GND")
+	)
+	(segment
+		(start 175.025 117.625)
+		(end 176.38 118.98)
+		(width 0.2)
+		(layer "F.Cu")
+		(net "GND")
+	)
+	(segment
+		(start 175.025 116.605)
+		(end 175.025 117.625)
+		(width 0.2)
+		(layer "F.Cu")
+		(net "GND")
+	)
+	(segment
+		(start 173.045 116.605)
+		(end 172.98 116.67)
+		(width 0.2)
+		(layer "F.Cu")
+		(net "GND")
+	)
+	(segment
+		(start 175.025 116.145)
+		(end 173.15 114.27)
+		(width 0.2)
+		(layer "F.Cu")
+		(net "GND")
+	)
+	(segment
+		(start 174.025 116.605)
+		(end 172.91 115.49)
+		(width 0.2)
+		(layer "F.Cu")
+		(net "GND")
+	)
+	(segment
+		(start 175.025 114.135)
+		(end 175.02 114.13)
+		(width 0.2)
+		(layer "F.Cu")
+		(net "GND")
+	)
+	(segment
+		(start 175.025 116.605)
+		(end 174.125 116.605)
+		(width 0.2)
+		(layer "F.Cu")
+		(net "GND")
+	)
+	(via
+		(at 175.02 118.89)
+		(size 0.6)
+		(drill 0.3)
+		(layers "F.Cu" "B.Cu")
+		(net "GND")
+	)
+	(via
+		(at 176.48 114.19)
+		(size 0.6)
+		(drill 0.3)
+		(layers "F.Cu" "B.Cu")
+		(net "GND")
+	)
+	(via
+		(at 176.38 118.98)
+		(size 0.6)
+		(drill 0.3)
+		(layers "F.Cu" "B.Cu")
+		(net "GND")
+	)
 	(via
 		(at 151.17 120.6)
@@
 	)
 	(via
+		(at 172.91 115.49)
+		(size 0.6)
+		(drill 0.3)
+		(layers "F.Cu" "B.Cu")
+		(net "GND")
+	)
+	(via
 		(at 145.63 117.31)
 		(size 0.6)
@@
 		(layers "F.Cu" "B.Cu")
 		(free yes)
+		(net "GND")
+	)
+	(via
+		(at 172.98 117.75)
+		(size 0.6)
+		(drill 0.3)
+		(layers "F.Cu" "B.Cu")
+		(net "GND")
+	)
+	(via
+		(at 173.17 118.93)
+		(size 0.6)
+		(drill 0.3)
+		(layers "F.Cu" "B.Cu")
+		(net "GND")
+	)
+	(via
+		(at 175.02 114.13)
+		(size 0.6)
+		(drill 0.3)
+		(layers "F.Cu" "B.Cu")
+		(net "GND")
+	)
+	(via
+		(at 172.98 116.67)
+		(size 0.6)
+		(drill 0.3)
+		(layers "F.Cu" "B.Cu")
+		(net "GND")
+	)
+	(via
+		(at 173.15 114.27)
+		(size 0.6)
+		(drill 0.3)
+		(layers "F.Cu" "B.Cu")
 		(net "GND")
 	)
@@
 		(net "Net-(IC1-AM2)")
 	)
-	(segment
-		(start 144.48 119.74)
-		(end 144.48 120.98)
-		(width 0.3)
-		(layer "F.Cu")
-		(net "Net-(U2-GATE)")
-	)
-	(segment
-		(start 145.85 122.35)
-		(end 146.5025 122.35)
-		(width 0.3)
-		(layer "F.Cu")
-		(net "Net-(U2-GATE)")
-	)
-	(segment
-		(start 144.48 120.98)
-		(end 145.85 122.35)
-		(width 0.3)
-		(layer "F.Cu")
-		(net "Net-(U2-GATE)")
-	)
 	(zone

Commit message: kdawjf
Parts:
- Q2: value BSC028N06NSATMA1 -> AO3400A; footprint footprints:TRANS_BSC028N06NSATMA1 -> Package_TO_SOT_SMD:SOT-23
- moved Q2 1.57 mm to (148.9, 117.8)
Connections:
- Q2 pad 1: VCC -> Net-(Q2-G)
- Q2 pad 3: VCC -> Net-(D1-K)
- U2 pad 2: Net-(U2-GATE) -> Net-(Q2-G)
Routing:
- net Net-(Q2-G): track 0.00 -> 10.8 mm, vias 0 -> 2
- net Net-(U2-GATE): track 3.83 -> 0.00 mm
- net VCC: track 103.4 -> 105.8 mm
