File: USB-Stick/AT1846S-breakout/AT1846S-breakout.kicad_pcb (KiCad board)
At the start: 2 copper layers, 41 parts, among them IC1 AT1846S, IC2 ASWD-S2-0005-T, J1 GPIOx, J2 CTRL, J3 MODE, J4 SPEAK, J5 PDN, J6 MIC, J8 SW, J9 FM-ANT, U1 YG401530VB, Y1 26 MHz

Commit message: 2kfjah
Parts:
- added C20: 100 nF, Capacitor_SMD:C_0603_1608Metric, F.Cu at (196.5, 84.5)
- added C21: 100 nF, Capacitor_SMD:C_0603_1608Metric, F.Cu at (196.5, 87.0)
- added J7: 5V, Connector_PinHeader_2.54mm:PinHeader_1x01_P2.54mm_Vertical, F.Cu at (204.8, 98.6)
- added U2: AMS1117-3.3, Package_TO_SOT_SMD:SOT-223-3_TabPin2, F.Cu at (216.6, 94.4)
- moved IC1 77.0 mm to (218.2, 74.3)
- moved J1 66.0 mm to (209.4, 84.8)
- moved J4 60.8 mm to (208.6, 76.6)
- moved C8 60.3 mm to (192.5, 72.0)
- moved Y1 59.0 mm to (217.2, 80.3)
- moved JP1 59.0 mm to (222.0, 79.8)
- moved C15 58.6 mm to (196.5, 72.0)
- moved C16 58.6 mm to (196.5, 74.5)
- moved R1 53.8 mm to (200.5, 72.0)
- moved R3 53.8 mm to (200.5, 77.0)
- moved R4 53.8 mm to (200.5, 79.5)
- moved R2 53.8 mm to (200.5, 74.5)
- moved J2 51.6 mm to (222.8, 100.9)
- moved S1 51.1 mm to (217.4, 87.2)
- moved L1 47.8 mm to (194.9, 102.4)
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Routing:
- added copper zone on In1.Cu, net GND
- added copper zone on In2.Cu, net GND
Other:
- board outline added: 99.8 x 39.8 mm
- copper layers 2 -> 4

Commit message: kfjaj
Parts:
- Y1: value 26 MHz -> 12.8 MHz
- moved J2 114.8 mm to (109.4, 82.7)
- moved JP1 110.8 mm to (111.3, 76.3)
- moved S1 107.9 mm to (111.7, 65.5), turned to 90 degrees
- moved Y1 100.2 mm to (117.5, 71.3), turned to 90 degrees
- moved J1 94.9 mm to (117.2, 62.6), turned to 90 degrees
- moved J3 93.6 mm to (112.0, 73.0)
- moved IC1 93.3 mm to (125.1, 69.9)
- moved J4 92.0 mm to (116.9, 84.1)
- moved R3 86.0 mm to (114.5, 76.4), turned to -90 degrees
- moved R4 83.3 mm to (117.3, 76.4), turned to -90 degrees
- moved J6 81.9 mm to (124.4, 78.9)
- moved U2 77.4 mm to (145.0, 65.1), turned to 180 degrees
- moved C14 74.7 mm to (120.2, 68.2), turned to 180 degrees
- moved R1 74.6 mm to (126.0, 75.3), turned to -90 degrees
- moved C1 72.8 mm to (115.8, 68.3)
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Routing:
- net +3V3: track 0.00 -> 103.6 mm, vias 0 -> 8
- net GND: track 0.00 -> 58.8 mm, vias 0 -> 30
- net /RFIN: track 0.00 -> 40.3 mm
- net Net-(IC1-SCLK): track 0.00 -> 27.7 mm, vias 0 -> 2
- net Net-(IC1-SDIO): track 0.00 -> 24.1 mm, vias 0 -> 2
- net Net-(IC1-SENB): track 0.00 -> 21.5 mm
- net Net-(IC1-MODE): track 0.00 -> 16.8 mm
- net +5V: track 0.00 -> 16.2 mm
- net Net-(JP1-A): track 0.00 -> 13.8 mm
- net Net-(IC1-PDN): track 0.00 -> 13.8 mm
- net Net-(C8-Pad2): track 0.00 -> 13.0 mm
- net Net-(J6-Pin_1): track 0.00 -> 12.3 mm
- net Net-(J4-Pin_1): track 0.00 -> 10.8 mm
- net Net-(IC1-GPIO7): track 0.00 -> 10.2 mm
- net /XTAL1: track 0.00 -> 8.65 mm
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Other:
- board size 99.8 x 39.8 mm -> 67.8 x 29.8 mm
