File: MCU/STM32F407VET6/STM32F407VET6.kicad_pcb (KiCad board)
At the start: 2 copper layers, 36 parts, among them J1 PROG, J2 USB_C_Receptacle_USB2.0_16P, J3 PAx, J4 PBx, J5 PCx, J6 PDx, J7 PEx, U1 STM32F407VETx, U2 AMS1117-3.3, Y1 8 MHz

Commit message: dkajhw
Parts:
- removed FB2: 120 Ohm, Resistor_SMD:R_0603_1608Metric
- added C17: 100 nF, Capacitor_SMD:C_0603_1608Metric, F.Cu at (174.5, 139.6)
- added C18: 100 nF, Capacitor_SMD:C_0603_1608Metric, F.Cu at (174.5, 142.1)
- added C19: 10 uF, Capacitor_SMD:C_0603_1608Metric, F.Cu at (174.5, 144.6)
- added C20: 10 uF, Capacitor_SMD:C_0603_1608Metric, F.Cu at (178.5, 134.6)
- added C21: 1 uF, Capacitor_SMD:C_0603_1608Metric, F.Cu at (178.5, 137.1)
- added C22: 100 nF, Capacitor_SMD:C_0603_1608Metric, F.Cu at (190.5, 112.4)
- added C23: 100 nF, Capacitor_SMD:C_0603_1608Metric, F.Cu at (190.5, 114.9)
- added C24: 100 nF, Capacitor_SMD:C_0603_1608Metric, F.Cu at (190.5, 117.4)
- added FB3: 120 Ohm, Resistor_SMD:R_0603_1608Metric, F.Cu at (178.5, 142.1)
- added J8: PCx, Connector_PinHeader_2.54mm:PinHeader_1x13_P2.54mm_Vertical, F.Cu at (107.5, 76.9)
- added R7: 12.1k 0.1%, Resistor_SMD:R_0603_1608Metric, F.Cu at (190.5, 120.0)
- added U3: AMS1117-3.3, Package_TO_SOT_SMD:SOT-223-3_TabPin2, F.Cu at (79.0, 58.6)
- added Y2: ECS-2520MV-500-BN-TR, Oscillator:Oscillator_SMD_ECS_2520MV-xxx-xx-4Pin_2.5x2.0mm, F.Cu at (170.4, 129.1)
- C10, C8, C9: value 1 uF -> 100 nF
- J2: footprint Connector_USB:USB_C_Receptacle_HRO_TYPE-C-31-M-17 -> Connector_USB:USB_C_Receptacle_HRO_TYPE-C-31-M-12
- J3: value PAx -> RJ45_Hanrun_HR911105A_Horizontal; footprint Connector_PinHeader_2.54mm:PinHeader_1x12_P2.54mm_Vertical -> Connector_RJ:RJ45_Hanrun_HR911105A_Horizontal
- J4: value PBx -> PAx; footprint Connector_PinHeader_2.54mm:PinHeader_1x15_P2.54mm_Vertical -> Connector_PinHeader_2.54mm:PinHeader_1x07_P2.54mm_Vertical
- J5: value PCx -> PBx; footprint Connector_PinHeader_2.54mm:PinHeader_1x16_P2.54mm_Vertical -> Connector_PinHeader_2.54mm:PinHeader_1x12_P2.54mm_Vertical
- U2: value AMS1117-3.3 -> LAN8742A; footprint Package_TO_SOT_SMD:SOT-223-3_TabPin2 -> Package_DFN_QFN:VQFN-24-1EP_4x4mm_P0.5mm_EP2.5x2.5mm_ThermalVias
- moved J1 111.5 mm to (64.6, 37.5)
- moved J2 108.6 mm to (65.4, 58.5), turned to -90 degrees
- moved Y1 82.3 mm to (117.0, 59.6), turned to -90 degrees
- moved NRST1 81.2 mm to (142.8, 32.2), turned to 180 degrees
- moved U2 76.2 mm to (144.9, 47.8), turned to 90 degrees
- moved BOOT1 75.1 mm to (132.1, 32.2), turned to 180 degrees
- moved J6 64.8 mm to (64.6, 76.9), turned to 90 degrees
- moved J7 61.7 mm to (102.7, 30.6), turned to -90 degrees
- moved U1 60.9 mm to (102.8, 58.5), turned to 180 degrees
- moved J4 55.6 mm to (122.8, 30.7), turned to -90 degrees
- moved C10 42.4 mm to (190.5, 109.9)
- moved C8 42.4 mm to (190.5, 104.9)
- moved C9 42.4 mm to (190.5, 107.4)
- moved R1 39.6 mm to (144.1, 154.6)
- moved R2 39.6 mm to (144.1, 157.1)
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Connections:
- net Net-(U1-VREF+) renamed VREF
- C10 pad 1: GND -> +3V3
- C10 pad 2: +3V3 -> GND
- C8 pad 1: VBUS -> +3V3
- J3 pad 1: Net-(J3-Pin_1) -> Net-(J3-TD+)
- J3 pad 10: Net-(J3-Pin_10) -> GND
- J3 pad 11: Net-(J3-Pin_11) -> GND
- J3 pad 12: Net-(J3-Pin_12) -> Net-(U2-LED2/~{INTSEL})
- J3 pad 2: Net-(J3-Pin_2) -> Net-(J3-TD-)
- J3 pad 3: Net-(J3-Pin_3) -> Net-(J3-RD+)
- J3 pad 4: Net-(J3-Pin_4) -> unconnected-(J3-TCT-Pad4)
- J3 pad 5: Net-(J3-Pin_5) -> unconnected-(J3-RCT-Pad5)
- J3 pad 6: Net-(J3-Pin_6) -> Net-(J3-RD-)
- J3 pad 7: Net-(J3-Pin_7) -> unconnected-(J3-NC-Pad7)
- J3 pad 8: Net-(J3-Pin_8) -> GND
- J3 pad 9: Net-(J3-Pin_9) -> Net-(U2-LED1/REGOFF)
- U1 pad 15: Net-(J5-Pin_1) -> Net-(J8-Pin_1)
- U1 pad 16: Net-(J5-Pin_2) -> /PC1
- U1 pad 17: Net-(J5-Pin_3) -> Net-(J8-Pin_2)
- U1 pad 18: Net-(J5-Pin_4) -> Net-(J8-Pin_3)
- U1 pad 22: Net-(U1-VDDA) -> VDDA
- U1 pad 23: Net-(J3-Pin_1) -> /PA0
- U1 pad 24: Net-(J3-Pin_2) -> /PA1
- U1 pad 25: Net-(J3-Pin_3) -> /PA2
- U1 pad 26: Net-(J3-Pin_4) -> Net-(J4-Pin_1)
- U1 pad 29: Net-(J3-Pin_5) -> Net-(J4-Pin_2)
- U1 pad 30: Net-(J3-Pin_6) -> Net-(J4-Pin_3)
- U1 pad 31: Net-(J3-Pin_7) -> Net-(J4-Pin_4)
- U1 pad 32: Net-(J3-Pin_8) -> /PA7
- U1 pad 33: Net-(J5-Pin_5) -> /PC4
- U1 pad 34: Net-(J5-Pin_6) -> /PC5
- U1 pad 35: Net-(J4-Pin_1) -> Net-(J5-Pin_1)
- U1 pad 36: Net-(J4-Pin_2) -> Net-(J5-Pin_2)
- U1 pad 37: Net-(J4-Pin_3) -> Net-(J5-Pin_3)
- U1 pad 47: Net-(J4-Pin_10) -> Net-(J5-Pin_10)
- U1 pad 48: Net-(J4-Pin_11) -> /PB11
- U1 pad 51: Net-(J4-Pin_12) -> /PB12
- U1 pad 52: Net-(J4-Pin_13) -> /PB13
- U1 pad 53: Net-(J4-Pin_14) -> Net-(J5-Pin_11)
- U1 pad 54: Net-(J4-Pin_15) -> Net-(J5-Pin_12)
- U1 pad 63: Net-(J5-Pin_7) -> Net-(J8-Pin_4)
- U1 pad 64: Net-(J5-Pin_8) -> Net-(J8-Pin_5)
- U1 pad 65: Net-(J5-Pin_9) -> Net-(J8-Pin_6)
- U1 pad 66: Net-(J5-Pin_10) -> Net-(J8-Pin_7)
- U1 pad 67: Net-(J3-Pin_9) -> Net-(J4-Pin_5)
- U1 pad 68: Net-(J3-Pin_10) -> Net-(J4-Pin_6)
- U1 pad 69: Net-(J3-Pin_11) -> Net-(J4-Pin_7)
- U1 pad 7: Net-(J5-Pin_14) -> Net-(J8-Pin_11)
- U1 pad 77: Net-(J3-Pin_12) -> /PA15
- U1 pad 78: Net-(J5-Pin_11) -> Net-(J8-Pin_8)
- U1 pad 79: Net-(J5-Pin_12) -> Net-(J8-Pin_9)
- U1 pad 8: Net-(J5-Pin_15) -> Net-(J8-Pin_12)
- U1 pad 80: Net-(J5-Pin_13) -> Net-(J8-Pin_10)
- U1 pad 9: Net-(J5-Pin_16) -> Net-(J8-Pin_13)
- U1 pad 90: Net-(J4-Pin_4) -> Net-(J5-Pin_4)
- U1 pad 91: Net-(J4-Pin_5) -> Net-(J5-Pin_5)
- U1 pad 92: Net-(J4-Pin_6) -> Net-(J5-Pin_6)
- U1 pad 93: Net-(J4-Pin_7) -> Net-(J5-Pin_7)
- U1 pad 95: Net-(J4-Pin_8) -> Net-(J5-Pin_8)
- U1 pad 96: Net-(J4-Pin_9) -> Net-(J5-Pin_9)
- U2 pad 1: GND -> Net-(U2-VDD2A)
- U2 pad 2: +3V3 -> Net-(U2-LED2/~{INTSEL})
- U2 pad 3: VBUS -> Net-(U2-LED1/REGOFF)
Routing:
- added copper zone on B.Cu, net GND
- added copper zone on F.Cu, net GND
- added copper zone on In1.Cu, net GND
- added copper zone on In2.Cu, net GND
Other:
- board outline added: 109.7 x 49.8 mm
- copper layers 2 -> 4
