File: MCU/STM32F407VET6/STM32F407VET6.kicad_sch (KiCad schematic)
At the start: 36 parts, among them J1 PROG, J2 USB_C_Receptacle_USB2.0_16P, J3 PAx, J4 PBx, J5 PCx, J6 PDx, J7 PEx, U1 STM32F407VETx, U2 AMS1117-3.3, Y1 8 MHz

Commit message: dkajhw
Parts:
- removed BOOT1, NRST1: KH-6X6X5H-STM, footprints:KH-6X6X5H-STM_SKE, symbol Personal:KH-6X6X5H-STM
- removed C10, C11, C12, C13, C14, C15, C16, C8, C9: 1 uF, Capacitor_SMD:C_0603_1608Metric, symbol Device:C_Small
- removed C3, C4, C5: 100nF, Capacitor_SMD:C_0603_1608Metric, symbol Device:C_Small
- removed FB1, FB2: 120 Ohm, Resistor_SMD:R_0603_1608Metric, symbol Device:FerriteBead_Small
- removed J2: USB_C_Receptacle_USB2.0_16P, Connector_USB:USB_C_Receptacle_HRO_TYPE-C-31-M-17, symbol Connector:USB_C_Receptacle_USB2.0_16P
- removed J3: PAx, Connector_PinHeader_2.54mm:PinHeader_1x12_P2.54mm_Vertical, symbol Connector:Conn_01x12_Pin
- removed J4: PBx, Connector_PinHeader_2.54mm:PinHeader_1x15_P2.54mm_Vertical, symbol Connector:Conn_01x15_Pin
- removed J5: PCx, Connector_PinHeader_2.54mm:PinHeader_1x16_P2.54mm_Vertical, symbol Connector:Conn_01x16_Pin
- removed R1, R2: 10k, Resistor_SMD:R_0603_1608Metric, symbol Device:R_Small
- removed R3, R4: 22, Resistor_SMD:R_0603_1608Metric, symbol Device:R_Small
- removed R5, R6: 5.1k, Resistor_SMD:R_0603_1608Metric, symbol Device:R_Small
- removed U2: AMS1117-3.3, Package_TO_SOT_SMD:SOT-223-3_TabPin2, symbol Regulator_Linear:AMS1117-3.3
- added J4: PAx, Connector_PinHeader_2.54mm:PinHeader_1x07_P2.54mm_Vertical, symbol Connector:Conn_01x07_Pin
- added J5: PBx, Connector_PinHeader_2.54mm:PinHeader_1x12_P2.54mm_Vertical, symbol Connector:Conn_01x12_Pin
- added J8: PCx, Connector_PinHeader_2.54mm:PinHeader_1x13_P2.54mm_Vertical, symbol Connector:Conn_01x13_Pin
Connections:
- net at U1.35 (PB0): now also J5.1 (Pin_1)
- net at U1.47 (PB10): now also J5.10 (Pin_10)
- net PB11: now reaches U1.48 (PB11)
- net PB12: now reaches U1.51 (PB12)
- net PB13: now reaches U1.52 (PB13)
- net at U1.53 (PB14): now also J5.11 (Pin_11)
- net at U1.54 (PB15): now also J5.12 (Pin_12)
- net at U1.36 (PB1): now also J5.2 (Pin_2)
- net at U1.37 (PB2): now also J5.3 (Pin_3)
- net at U1.90 (PB4): now also J5.4 (Pin_4)
- net at U1.91 (PB5): now also J5.5 (Pin_5)
- net at U1.92 (PB6): now also J5.6 (Pin_6)
- net at U1.93 (PB7): now also J5.7 (Pin_7)
- net at U1.95 (PB8): now also J5.8 (Pin_8)
- net at U1.96 (PB9): now also J5.9 (Pin_9)
- net at U1.15 (PC0): now also J8.1 (Pin_1)
- net at U1.66 (PC9): now also J8.7 (Pin_7)
- net at U1.78 (PC10): now also J8.8 (Pin_8)
- net at U1.79 (PC11): now also J8.9 (Pin_9)
- net at U1.80 (PC12): now also J8.10 (Pin_10)
- net at U1.7 (PC13): now also J8.11 (Pin_11)
- net at U1.8 (PC14): now also J8.12 (Pin_12)
- net at U1.9 (PC15): now also J8.13 (Pin_13)
- net PC1: now reaches U1.16 (PC1)
- net at U1.17 (PC2): now also J8.2 (Pin_2)
- net at U1.18 (PC3): now also J8.3 (Pin_3)
- net PC4: now reaches U1.33 (PC4)
- net PC5: now reaches U1.34 (PC5)
- net at U1.63 (PC6): now also J8.4 (Pin_4)
- net at U1.64 (PC7): now also J8.5 (Pin_5)
- net at U1.65 (PC8): now also J8.6 (Pin_6)
- net VREF: now reaches U1.21 (VREF+)
- net VDDA: now reaches U1.22 (VDDA)
- net PA0: now reaches U1.23 (PA0)
- net PA1: now reaches U1.24 (PA1)
- net PA2: now reaches U1.25 (PA2)
- net at U1.26 (PA3): now also J4.1 (Pin_1)
- net at U1.29 (PA4): now also J4.2 (Pin_2)
- net at U1.30 (PA5): now also J4.3 (Pin_3)
- net at U1.31 (PA6): now also J4.4 (Pin_4)
- net PA7: now reaches U1.32 (PA7)
- net at U1.67 (PA8): now also J4.5 (Pin_5)
- net at U1.68 (PA9): now also J4.6 (Pin_6)
- net at U1.69 (PA10): now also J4.7 (Pin_7)
- net PA15: now reaches U1.77 (PA15)
- no-connect marks 3 -> 1
Other:
- added sheet ctrl (ctrl.kicad_sch)
- added sheet ethernet (ethernet.kicad_sch)
- added sheet power (power.kicad_sch)
- added sheet usb (usb.kicad_sch)
- moved on the sheet: J1
