File: WalkieTalkies/si4463/si4463.kicad_pcb (KiCad board)
At the start: 2 copper layers, 60 x 22.2 mm, 33 parts, among them J1 CTRL, J2 GPIOx, J3 TX, J4 RX, J5 TXRAMP, J6 PWR3, J7 PWR5, U1 Si4463, U2 YG401530VB, Y1 Crystal_GND24

Commit message: KfjawJ
Parts:
- Y1: value Crystal_GND24 -> 30MHz
- moved C1 91.4 mm to (223.8, 87.9)
- moved LR2 89.2 mm to (210.5, 80.5), turned to 90 degrees
- moved C2 87.1 mm to (217.6, 84.8), turned to -90 degrees
- moved LC1 87.0 mm to (212.4, 91.7), turned to -90 degrees
- moved L0 82.8 mm to (209.0, 92.9)
- moved L2 82.5 mm to (208.8, 97.5), turned to 180 degrees
- moved L1 82.5 mm to (208.8, 95.0)
- moved C9 82.0 mm to (212.5, 88.0), turned to -90 degrees
- moved CM5 81.7 mm to (207.9, 86.6), turned to -90 degrees
- moved CM1 81.5 mm to (212.5, 94.9), turned to 180 degrees
- moved CM3 80.9 mm to (218.3, 93.9), turned to -90 degrees
- moved LR1 80.5 mm to (202.7, 81.9), turned to 90 degrees
- moved L3 79.9 mm to (205.8, 94.3), turned to -90 degrees
- moved CM4 79.7 mm to (216.5, 93.4), turned to 90 degrees
- moved CR2 76.9 mm to (206.8, 81.3), turned to -90 degrees
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Routing:
- net +5V: track 0.00 -> 52.6 mm
- net +3V3: track 0.00 -> 40.4 mm
- net Net-(J2-Pin_4): track 0.00 -> 23.0 mm, vias 0 -> 1
- net /IRQ: track 0.00 -> 22.0 mm, vias 0 -> 3
- net /RXp: track 0.00 -> 21.3 mm, vias 0 -> 2
- net Net-(J2-Pin_3): track 0.00 -> 19.8 mm, vias 0 -> 1
- net /RXn: track 0.00 -> 18.1 mm, vias 0 -> 2
- net /SEL: track 0.00 -> 17.3 mm, vias 0 -> 3
- net Net-(J2-Pin_2): track 0.00 -> 15.6 mm, vias 0 -> 1
- net /SDN: track 0.00 -> 15.0 mm, vias 0 -> 1
- net Net-(J2-Pin_1): track 0.00 -> 14.0 mm, vias 0 -> 1
- net /SDO: track 0.00 -> 13.9 mm, vias 0 -> 3
- net /SCLK: track 0.00 -> 12.6 mm, vias 0 -> 1
- net /SDI: track 0.00 -> 12.5 mm, vias 0 -> 3
- net /TX: track 0.00 -> 11.9 mm, vias 0 -> 2
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- added copper zone on B.Cu, net GND
- added copper zone on F.Cu, net GND

Commit message: kfjjfhawh
Parts:
- added J8: TX_PA, Connector_Coaxial:SMA_BAT_Wireless_BWSMA-KWE-Z001, F.Cu at (194.0, 86.0)
- J3: value TX -> TX_A
- moved J4 5.20 mm to (194.0, 76.7)
- moved CM8 5.12 mm to (201.2, 87.1), turned to -90 degrees
Routing:
- net Net-(J8-In): track 3.17 -> 17.5 mm
- net Net-(J4-In): track 9.74 -> 14.0 mm
- net /IRQ: track 22.0 -> 18.8 mm
Other:
- board size 60 x 22.2 mm -> 60 x 27.4 mm
