File: KakiDev/LFE5UM5G-85F-8BG381C/io.kicad_sch (KiCad schematic)
At the start: 5 parts, among them J4 PLX, J7 PRx, J8 PBx, J9 PTx, U1 ECP5-CABGA256

Commit message: 2kgjJ
Parts:
- removed J7: PRx, Connector_PinHeader_2.54mm:PinHeader_1x27_P2.54mm_Vertical, symbol Connector:Conn_01x27_Pin
- removed J9: PTx, Connector_PinHeader_2.54mm:PinHeader_1x19_P2.54mm_Vertical, symbol Connector:Conn_01x19_Pin
- added J10: PRx, Connector_PinHeader_2.54mm:PinHeader_2x14_P2.54mm_Vertical, symbol Connector:Conn_01x28_Pin
- added J7: PTx, Connector_PinHeader_2.54mm:PinHeader_2x10_P2.54mm_Vertical, symbol Connector:Conn_01x20_Pin
- J4: footprint Connector_PinHeader_2.54mm:PinHeader_1x26_P2.54mm_Vertical -> Connector_PinHeader_2.54mm:PinHeader_2x13_P2.54mm_Vertical
- J8: footprint Connector_PinHeader_2.54mm:PinHeader_1x08_P2.54mm_Vertical -> Connector_PinHeader_2.54mm:PinHeader_2x04_P2.54mm_Vertical
Connections:
- net at U1.D12 (PT58A/+): now also J7.1 (Pin_1)
- net at U1.C9 (PT38B/-/GR_PCLK1_1): now also J7.10 (Pin_10)
- net at U1.E8 (PT33A/+/PCLKT1_1): now also J7.11 (Pin_11)
- net at U1.D8 (PT33B/-/PCLKC1_1): now also J7.12 (Pin_12)
- net at U1.E7 (PT24A/+/GR_PCLK0_1): now also J7.13 (Pin_13)
- net at U1.D7 (PT24B/-/GR_PCLK0_0): now also J7.14 (Pin_14)
- net at U1.C6 (PT22A/+): now also J7.15 (Pin_15)
- net at U1.E6 (PT20A/+): now also J7.16 (Pin_16)
- net at U1.D6 (PT20B/-): now also J7.17 (Pin_17)
- net at U1.E5 (PT13A/+): now also J7.18 (Pin_18)
- net at U1.D5 (PT13B/-): now also J7.19 (Pin_19)
- net at U1.C12 (PT56B/-): now also J7.2 (Pin_2)
- net at U1.D11 (PT51A/+): now also J7.3 (Pin_3)
- net at U1.C11 (PT49B/-): now also J7.4 (Pin_4)
- net at U1.D10 (PT47A/+): now also J7.5 (Pin_5)
- net at U1.E10 (PT47B/-): now also J7.6 (Pin_6)
- net at U1.C10 (PT44B/-): now also J7.7 (Pin_7)
- net at U1.D9 (PT40A/+): now also J7.8 (Pin_8)
- net at U1.E9 (PT40B/-): now also J7.9 (Pin_9)
- net at U1.N11 (PR47B/0/HS/RDQ44): now also J10.1 (Pin_1)
- net at U1.L13 (PR29C/+/RDQ32/GR_PCLK3_1): now also J10.10 (Pin_10)
- net at U1.L12 (PR29D/-/RDQ32): now also J10.11 (Pin_11)
- net at U1.G16 (PR20A/+/HS/RDQS20/GR_PCLK2_1): now also J10.12 (Pin_12)
- net at U1.H15 (PR20B/-/HS/RDQSN20): now also J10.13 (Pin_13)
- net at U1.J14 (PR20C/+/RDQ20/GR_PCLK2_0): now also J10.14 (Pin_14)
- net at U1.K14 (PR20D/-/RDQ20): now also J10.15 (Pin_15)
- net at U1.H12 (PR17A/+/HS/RDQ20): now also J10.16 (Pin_16)
- net at U1.H13 (PR17B/-/HS/RDQ20): now also J10.17 (Pin_17)
- net at U1.J13 (PR17C/+/RDQ20): now also J10.18 (Pin_18)
- net at U1.J12 (PR17D/-/RDQ20): now also J10.19 (Pin_19)
- net at U1.M12 (PR44C/+/RDQ44): now also J10.2 (Pin_2)
- net at U1.F16 (PR14A/+/HS/RDQ20): now also J10.20 (Pin_20)
- net at U1.G14 (PR14C/+/RDQ20/VREF1_2): now also J10.21 (Pin_21)
- net at U1.G12 (PR11A/+/HS/RDQ8): now also J10.22 (Pin_22)
- net at U1.G13 (PR11B/-/HS/RDQ8): now also J10.23 (Pin_23)
- net at U1.E15 (PR8B/-/HS/RDQSN8): now also J10.24 (Pin_24)
- net at U1.F13 (PR8C/+/RDQ8): now also J10.25 (Pin_25)
- net at U1.F12 (PR8D/-/RDQ8): now also J10.26 (Pin_26)
- net at U1.F14 (PR5D/-/RDQ8): now also J10.27 (Pin_27)
- net at U1.P12 (PR47D/-/RDQ44/LRC_GPLL0C_IN): now also J10.3 (Pin_3)
- net at U1.P13 (PR41A/+/HS/RDQ44): now also J10.4 (Pin_4)
- net at U1.N13 (PR38A/+/HS/RDQ44): now also J10.5 (Pin_5)
- net at U1.M13 (PR35C/+/RDQ32): now also J10.6 (Pin_6)
- net at U1.N14 (PR35D/-/RDQ32): now also J10.7 (Pin_7)
- net at U1.K13 (PR29A/+/HS/RDQ32/GR_PCLK3_0): now also J10.8 (Pin_8)
- net at U1.K12 (PR29B/-/HS/RDQ32): now also J10.9 (Pin_9)
- new net GND: J10.28 (Pin_28), J7.20 (Pin_20)
