File: KakiDev/LFE5UM5G-85F-8BG381C/icepi-zero.kicad_pcb (KiCad board)
At the start: 4 copper layers, 109 x 79 mm, 132 parts, among them J1 Conn_02x20_Counter_Clockwise, J2 GPDI_C_1.3, J3 USB_C_Receptacle_USB2.0_16P, J4 PLX, J5 USB_C_Receptacle_USB2.0_16P, J6 Micro_SD_Card_Det2, J7 PRx, J8 PBx, J9 PTx, SW3 KH-6X6X5H-STM, SW4 KH-6X6X5H-STM, U1 ECP5-CABGA256, U11 W9825G6KH, U12 W25Q128JVS, U2 TLV62569DBV, U3 TLV62569DBV, U4 TLV62569DBV, U6 PCA9306DC1, U9 FT231XQ, Y1 SG-8018CG 50.000000MHz

Commit message: 2kgjJ
Parts:
- removed J9: PTx, Connector_PinHeader_2.54mm:PinHeader_1x19_P2.54mm_Vertical
- added J10: PRx, Connector_PinHeader_2.54mm:PinHeader_2x14_P2.54mm_Vertical, F.Cu at (180.9, 52.2)
- J4: footprint Connector_PinHeader_2.54mm:PinHeader_1x26_P2.54mm_Vertical -> Connector_PinHeader_2.54mm:PinHeader_2x13_P2.54mm_Vertical
- J7: value PRx -> PTx; footprint Connector_PinHeader_2.54mm:PinHeader_1x27_P2.54mm_Vertical -> Connector_PinHeader_2.54mm:PinHeader_2x10_P2.54mm_Vertical
- J8: footprint Connector_PinHeader_2.54mm:PinHeader_1x08_P2.54mm_Vertical -> Connector_PinHeader_2.54mm:PinHeader_2x04_P2.54mm_Vertical
- moved TP7 231.8 mm to (259.4, 80.2)
- moved TP8 231.8 mm to (259.4, 83.3)
- moved R43 229.7 mm to (245.9, 80.0)
- moved R44 229.7 mm to (245.9, 82.5)
- moved R45 229.7 mm to (245.9, 85.0)
- moved R46 229.7 mm to (245.9, 87.5)
- moved R47 229.7 mm to (245.9, 90.0)
- moved R48 229.7 mm to (245.9, 92.5)
- moved R49 229.7 mm to (245.9, 95.0)
- moved R50 229.7 mm to (245.9, 97.5)
- moved D1 222.6 mm to (255.9, 80.0)
- moved D2 222.6 mm to (255.9, 82.6)
- moved D3 222.6 mm to (255.9, 85.2)
- moved D4 222.6 mm to (255.9, 87.8)
- moved D5 222.6 mm to (255.9, 90.4)
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Connections:
- J7 pad 20: Net-(J7-Pin_20) -> GND
- U1 pad C10: Net-(J9-Pin_7) -> Net-(J7-Pin_7)
- U1 pad C11: Net-(J9-Pin_4) -> Net-(J7-Pin_4)
- U1 pad C12: Net-(J9-Pin_2) -> Net-(J7-Pin_2)
- U1 pad C6: Net-(J9-Pin_15) -> Net-(J7-Pin_15)
- U1 pad C9: Net-(J9-Pin_10) -> Net-(J7-Pin_10)
- U1 pad D10: Net-(J9-Pin_5) -> Net-(J7-Pin_5)
- U1 pad D11: Net-(J9-Pin_3) -> Net-(J7-Pin_3)
- U1 pad D12: Net-(J9-Pin_1) -> Net-(J7-Pin_1)
- U1 pad D5: Net-(J9-Pin_19) -> Net-(J7-Pin_19)
- U1 pad D6: Net-(J9-Pin_17) -> Net-(J7-Pin_17)
- U1 pad D7: Net-(J9-Pin_14) -> Net-(J7-Pin_14)
- U1 pad D8: Net-(J9-Pin_12) -> Net-(J7-Pin_12)
- U1 pad D9: Net-(J9-Pin_8) -> Net-(J7-Pin_8)
- U1 pad E10: Net-(J9-Pin_6) -> Net-(J7-Pin_6)
- U1 pad E15: Net-(J7-Pin_24) -> Net-(J10-Pin_24)
- U1 pad E5: Net-(J9-Pin_18) -> Net-(J7-Pin_18)
- U1 pad E6: Net-(J9-Pin_16) -> Net-(J7-Pin_16)
- U1 pad E7: Net-(J9-Pin_13) -> Net-(J7-Pin_13)
- U1 pad E8: Net-(J9-Pin_11) -> Net-(J7-Pin_11)
- U1 pad E9: Net-(J9-Pin_9) -> Net-(J7-Pin_9)
- U1 pad F12: Net-(J7-Pin_26) -> Net-(J10-Pin_26)
- U1 pad F13: Net-(J7-Pin_25) -> Net-(J10-Pin_25)
- U1 pad F14: Net-(J7-Pin_27) -> Net-(J10-Pin_27)
- U1 pad F16: Net-(J7-Pin_20) -> Net-(J10-Pin_20)
- U1 pad G12: Net-(J7-Pin_22) -> Net-(J10-Pin_22)
- U1 pad G13: Net-(J7-Pin_23) -> Net-(J10-Pin_23)
- U1 pad G14: Net-(J7-Pin_21) -> Net-(J10-Pin_21)
- U1 pad G16: Net-(J7-Pin_12) -> Net-(J10-Pin_12)
- U1 pad H12: Net-(J7-Pin_16) -> Net-(J10-Pin_16)
- U1 pad H13: Net-(J7-Pin_17) -> Net-(J10-Pin_17)
- U1 pad H15: Net-(J7-Pin_13) -> Net-(J10-Pin_13)
- U1 pad J12: Net-(J7-Pin_19) -> Net-(J10-Pin_19)
- U1 pad J13: Net-(J7-Pin_18) -> Net-(J10-Pin_18)
- U1 pad J14: Net-(J7-Pin_14) -> Net-(J10-Pin_14)
- U1 pad K12: Net-(J7-Pin_9) -> Net-(J10-Pin_9)
- U1 pad K13: Net-(J7-Pin_8) -> Net-(J10-Pin_8)
- U1 pad K14: Net-(J7-Pin_15) -> Net-(J10-Pin_15)
- U1 pad L12: Net-(J7-Pin_11) -> Net-(J10-Pin_11)
- U1 pad L13: Net-(J7-Pin_10) -> Net-(J10-Pin_10)
- U1 pad M12: Net-(J7-Pin_2) -> Net-(J10-Pin_2)
- U1 pad M13: Net-(J7-Pin_6) -> Net-(J10-Pin_6)
- U1 pad N11: Net-(J7-Pin_1) -> Net-(J10-Pin_1)
- U1 pad N13: Net-(J7-Pin_5) -> Net-(J10-Pin_5)
- U1 pad N14: Net-(J7-Pin_7) -> Net-(J10-Pin_7)
- U1 pad P12: Net-(J7-Pin_3) -> Net-(J10-Pin_3)
- U1 pad P13: Net-(J7-Pin_4) -> Net-(J10-Pin_4)
Other:
- board size 109 x 79 mm -> 89.8 x 73.5 mm

Commit message: jkfjhaqju
Parts:
- removed C54: 10uF, Capacitor_SMD:C_0603_1608Metric
- removed J6: Micro_SD_Card_Det2, icepi-lib:microSD_HC_SOFNG_TF-008
- added C55: 10uF, Capacitor_SMD:C_0603_1608Metric, F.Cu at (202.1, 61.8)
- added J9: Conn_02x05_Top_Bottom, Connector_PinHeader_2.54mm:PinHeader_2x05_P2.54mm_Vertical, F.Cu at (184.7, 63.7)
- added R28: 22, Resistor_SMD:R_0603_1608Metric, F.Cu at (169.9, 115.5)
- added R31: 22, Resistor_SMD:R_0603_1608Metric, F.Cu at (166.8, 115.5)
- C51, C52: value 22nF -> 100nF
- moved U2 127.2 mm to (108.3, 57.3), turned to 180 degrees
- moved U3 126.5 mm to (108.3, 66.0), turned to 180 degrees
- moved U4 126.1 mm to (108.3, 73.5), turned to 180 degrees
- moved L1 125.9 mm to (113.7, 56.4)
- moved L2 124.1 mm to (113.7, 65.1)
- moved L3 122.9 mm to (113.7, 72.6)
- moved U11 122.9 mm to (125.9, 85.5), turned to -90 degrees
- moved R7 117.9 mm to (114.0, 59.6), turned to 180 degrees
- moved R6 117.6 mm to (114.0, 58.0), turned to 180 degrees
- moved C33 115.8 mm to (109.6, 76.8), turned to -90 degrees
- moved R9 115.6 mm to (114.0, 68.3), turned to 180 degrees
- moved R8 115.5 mm to (114.0, 66.8), turned to 180 degrees
- moved R11 115.3 mm to (113.9, 75.8)
- moved R10 115.2 mm to (113.9, 74.2), turned to 180 degrees
- moved C18 110.7 mm to (109.7, 69.3), turned to -90 degrees
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Connections:
- J5 pad A6: Net-(U9-USBDP) -> Net-(J5-D+-PadA6)
- J5 pad A7: Net-(U9-USBDM) -> Net-(J5-D--PadA7)
- J5 pad B6: Net-(U9-USBDP) -> Net-(J5-D+-PadA6)
- J5 pad B7: Net-(U9-USBDM) -> Net-(J5-D--PadA7)
- R20 pad 2: /USB/D0I- -> /USB/D0-
- R22 pad 2: /USB/D0I- -> /USB/D0-
