File: Psu/LM5176PWP/LM5176PWP.kicad_pcb (KiCad board)
At the start: 2 copper layers, 110.1 x 50.2 mm, 47 parts, among them J1 Vin, J2 Vout, Q1 CSD17577Q5A, Q2 CSD17577Q5A, Q3 CSD17577Q5A, Q4 CSD17577Q5A, U1 LM5176PWP

Commit message: layout fuck yourself
Parts:
- moved CCs1 93.9 mm to (226.1, 139.2)
- moved CSlope1 93.9 mm to (226.1, 142.2)
- moved Cbias1 93.9 mm to (226.1, 145.2)
- moved Cboot1 93.9 mm to (226.1, 148.2)
- moved Cboot2 93.9 mm to (226.1, 151.2)
- moved Cout1 93.9 mm to (223.7, 113.7)
- moved Cout2 93.9 mm to (223.7, 120.6)
- moved Cout3 93.9 mm to (223.7, 127.4)
- moved Cout4 93.9 mm to (218.6, 141.8)
- moved Cout5 93.9 mm to (218.6, 149.9)
- moved Dboot1 93.9 mm to (240.5, 112.6)
- moved Dboot2 93.9 mm to (240.5, 117.1)
- moved Df1 93.9 mm to (240.5, 121.7)
- moved Cin1 93.9 mm to (205.8, 113.7)
- moved Cin2 93.9 mm to (205.8, 120.6)
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Connections:
- Q2 pad 1: /RCS_1 -> /RCS
- Q2 pad 2: /RCS_1 -> /RCS
- Q2 pad 3: /RCS_1 -> /RCS
- Q4 pad 1: /RCS_1 -> /RCS
- Q4 pad 2: /RCS_1 -> /RCS
- Q4 pad 3: /RCS_1 -> /RCS
- R1 pad 2: /RCS2 -> /RCS
- R2 pad 2: /CSG2 -> GND
- Rsense1 pad 2: /RCS_1 -> /RCS
Other:
- board outline removed
- copper layers 2 -> 4

Commit message: Kfjawjhrj
Parts:
- removed L1: WE-XHMI_7030, footprints:WE-XHMI_7030
- added CDith1: 150pF, Capacitor_SMD:C_0805_2012Metric, F.Cu at (211.5, 103.9)
- added L2: XAL1010-222MED, footprints:XAL1010222MED, F.Cu at (215.8, 95.2)
- CSlope1: value 100pF -> 150pF
- Ccomp1: value 4.7nF -> 15nF
- Ccomp2: value 220pF -> 560pF
- Rcomp1: value 5.49k -> 3.48k
- Rt1: value 23.2k -> 37.4k
- Rvisns1: value 36.5k -> 2k
Connections:
- U1 pad 5: GND -> Net-(U1-DITH)
