File: Psu/LM5176PWP/LM5176PWP.kicad_sch (KiCad schematic)
At the start: 47 parts, among them J1 Vin, J2 Vout, Q1 CSD17577Q5A, Q2 CSD17577Q5A, Q3 CSD17577Q5A, Q4 CSD17577Q5A, U1 LM5176PWP

Commit message: layout fuck yourself
Connections:
- net CSG2 is gone; now on net GND: R2.2
- net RCS_1 is gone; now on net RCS: Q2.1 (S), Q2.2 (S), Q2.3 (S), Q4.1 (S), Q4.2 (S), Q4.3 (S), Rsense1.2
- net RCS2 renamed RCS
Changed lines of the file:
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@@
+	)
+	(junction
+		(at 346.71 55.88)
+		(diameter 0)
+		(color 0 0 0 0)
+	)
+	(junction
+		(at 185.42 115.57)
+		(diameter 0)
+		(color 0 0 0 0)
+	)
+	(junction
+		(at 185.42 105.41)
+		(diameter 0)
+		(color 0 0 0 0)
+	)
+	(junction
+		(at 77.47 41.91)
+		(diameter 0)
+		(color 0 0 0 0)
+	)
+	(junction
+		(at 135.89 148.59)
+		(diameter 0)
+		(color 0 0 0 0)
+	)
+	(junction
+		(at 146.05 50.8)
+		(diameter 0)
+		(color 0 0 0 0)
+	)
+	(junction
+		(at 204.47 105.41)
+		(diameter 0)
+		(color 0 0 0 0)
+	)
+	(junction
+		(at 204.47 130.81)
+		(diameter 0)
+		(color 0 0 0 0)
+	)
+	(junction
+		(at 308.61 50.8)
+		(diameter 0)
+		(color 0 0 0 0)
+	)
+	(junction
+		(at 106.68 50.8)
+		(diameter 0)
+		(color 0 0 0 0)
+	)
+	(junction
+		(at 346.71 50.8)
+		(diameter 0)
+		(color 0 0 0 0)
+	)
+	(junction
+		(at 158.75 140.97)
+		(diameter 0)
+		(color 0 0 0 0)
 	)
 	(junction
@@
 	)
 	(junction
-		(at 346.71 55.88)
-		(diameter 0)
-		(color 0 0 0 0)
-	)
-	(junction
-		(at 185.42 115.57)
-		(diameter 0)
-		(color 0 0 0 0)
-	)
-	(junction
-		(at 185.42 105.41)
-		(diameter 0)
-		(color 0 0 0 0)
-	)
-	(junction
-		(at 77.47 41.91)
-		(diameter 0)
-		(color 0 0 0 0)
-	)
-	(junction
-		(at 135.89 148.59)
-		(diameter 0)
-		(color 0 0 0 0)
-	)
-	(junction
-		(at 146.05 50.8)
-		(diameter 0)
-		(color 0 0 0 0)
-	)
-	(junction
-		(at 204.47 105.41)
-		(diameter 0)
-		(color 0 0 0 0)
-	)
-	(junction
-		(at 204.47 130.81)
-		(diameter 0)
-		(color 0 0 0 0)
-	)
-	(junction
-		(at 308.61 50.8)
-		(diameter 0)
-		(color 0 0 0 0)
-	)
-	(junction
-		(at 106.68 50.8)
-		(diameter 0)
-		(color 0 0 0 0)
-	)
-	(junction
-		(at 346.71 50.8)
-		(diameter 0)
-		(color 0 0 0 0)
-	)
-	(junction
-		(at 158.75 140.97)
-		(diameter 0)
-		(color 0 0 0 0)
-	)
-	(junction
 		(at 86.36 57.15)
 		(diameter 0)
@@
 		)
 	)
-	(label "RCS2"
+	(label "RCS"
 		(at 102.87 144.78 270)
 		(effects
@@
 		)
 	)
-	(label "CSG_1"
-		(at 254 100.33 180)
+	(label "CSG"
+		(at 254 99.06 180)
 		(effects
 			(font
@@
 		)
 	)
-	(label "CSG2"
+	(label "CSG"
 		(at 116.84 144.78 270)
 		(effects
@@
 		)
 	)
-	(label "RCS_1"
+	(label "RCS"
 		(at 254 90.17 180)
 		(effects

Commit message: Kfjawjhrj
Parts:
- removed L1: WE-XHMI_7030, footprints:WE-XHMI_7030, symbol symbols:WE-XHMI_7030
- added CDith1: 150pF, Capacitor_SMD:C_0805_2012Metric, symbol Device:C_Small
- added L2: XAL1010-222MED, XAL1010222MED, symbol symbols:XAL1010-222MED
- CSlope1: value 100pF -> 150pF
- Ccomp1: value 4.7nF -> 15nF
- Ccomp2: value 220pF -> 560pF
- Rcomp1: value 5.49k -> 3.48k
- Rt1: value 23.2k -> 37.4k
- Rvisns1: value 36.5k -> 2k
Connections:
- net GND: now also CDith1.1; no longer U1.5 (DITH)
- net SW1: now also L2.1
- net SW2: now also L2.2
- new net: CDith1.2, U1.5 (DITH)
