File: MCU/CH569W/CH569W.kicad_sch (KiCad schematic)
At the start: 29 parts, among them J1 USB_C_Receptacle_USB2.0_16P, J2 SerDes, J3 Conn_02x09_Odd_Even, J4 Conn_01x07_Pin, U1 CH569W, U3 LT1117-3.3, U5 TLV75512PDBV, Y1 30MHz

Commit message: jfhah
Parts:
- removed U3: LT1117-3.3, Package_TO_SOT_SMD:TSOT-23-5, symbol Regulator_Linear:LT1117-3.3
- added U4: AP2112K-3.3, Package_TO_SOT_SMD:SOT-23-5, symbol Regulator_Linear:AP2112K-3.3
Connections:
- net +3V3: now also U4.5 (VOUT)
- net +5V: now also U4.1 (VIN), U4.3 (EN)
- net GND: now also U4.2 (GND)
Other:
- moved on the sheet: C24, C25
Changed lines of the file:
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@@
 	)
 	(junction
-		(at 20.32 119.38)
+		(at 26.67 116.84)
+		(diameter 0)
+		(color 0 0 0 0)
+	)
+	(junction
+		(at 20.32 116.84)
 		(diameter 0)
 		(color 0 0 0 0)
@@
 	)
 	(junction
-		(at 48.26 119.38)
+		(at 48.26 116.84)
 		(diameter 0)
 		(color 0 0 0 0)
@@
 	(wire
 		(pts
-			(xy 41.91 119.38) (xy 48.26 119.38)
+			(xy 41.91 116.84) (xy 48.26 116.84)
 		)
 		(stroke
@@
 	(wire
 		(pts
-			(xy 20.32 119.38) (xy 26.67 119.38)
+			(xy 20.32 116.84) (xy 26.67 116.84)
 		)
 		(stroke
@@
 	(wire
 		(pts
+			(xy 26.67 116.84) (xy 26.67 119.38)
+		)
+		(stroke
+			(width 0)
+			(type default)
+		)
+	)
+	(wire
+		(pts
 			(xy 45.72 57.15) (xy 54.61 57.15)
 		)
@@
 	(symbol
 		(lib_id "power:GND")
-		(at 48.26 124.46 0)
+		(at 48.26 121.92 0)
 		(unit 1)
 		(body_style 1)
@@
 		(fields_autoplaced yes)
 		(property "Reference" "#PWR059"
-			(at 48.26 130.81 0)
+			(at 48.26 128.27 0)
 			(hide yes)
 			(show_name no)
@@
 		)
 		(property "Value" "GND"
-			(at 48.26 129.54 0)
+			(at 48.26 127 0)
 			(show_name no)
 			(do_not_autoplace no)
@@
 		)
 		(property "Footprint" ""
-			(at 48.26 124.46 0)
+			(at 48.26 121.92 0)
 			(hide yes)
 			(show_name no)
@@
 		)
 		(property "Datasheet" ""
-			(at 48.26 124.46 0)
+			(at 48.26 121.92 0)
 			(hide yes)
 			(show_name no)
@@
 		)
 		(property "Description" "Power symbol creates a global label with name \"GND\" , ground"
-			(at 48.26 124.46 0)
+			(at 48.26 121.92 0)
 			(hide yes)
 			(show_name no)
@@
 	(symbol
 		(lib_id "power:+5V")
-		(at 20.32 119.38 0)
+		(at 20.32 116.84 0)
 		(unit 1)
 		(body_style 1)
@@
 		(fields_autoplaced yes)
 		(property "Reference" "#PWR055"
-			(at 20.32 123.19 0)
+			(at 20.32 120.65 0)
 			(hide yes)
 			(show_name no)
@@
 		)
 		(property "Value" "+5V"
-			(at 20.32 114.3 0)
+			(at 20.32 111.76 0)
 			(show_name no)
 			(do_not_autoplace no)
@@
 		)
 		(property "Footprint" ""
-			(at 20.32 119.38 0)
+			(at 20.32 116.84 0)
 			(hide yes)
 			(show_name no)
@@
 		)
 		(property "Datasheet" ""
-			(at 20.32 119.38 0)
+			(at 20.32 116.84 0)
 			(hide yes)
 			(show_name no)
@@
 		)
 		(property "Description" "Power symbol creates a global label with name \"+5V\""
-			(at 20.32 119.38 0)
+			(at 20.32 116.84 0)
 			(hide yes)
 			(show_name no)
@@
 	)
 	(symbol
+		(lib_id "Regulator_Linear:AP2112K-3.3")
+		(at 34.29 119.38 0)
+		(unit 1)
+		(body_style 1)
+		(exclude_from_sim no)
+		(in_bom yes)
+		(on_board yes)
+		(in_pos_files yes)
+		(dnp no)
+		(fields_autoplaced yes)
+		(property "Reference" "U4"
+			(at 34.29 110.49 0)
+			(show_name no)
+			(do_not_autoplace no)
+			(effects
+				(font
+					(size 1.27 1.27)
+				)
+			)
+		)
+		(property "Value" "AP2112K-3.3"
+			(at 34.29 113.03 0)
+			(show_name no)
+			(do_not_autoplace no)
+			(effects
+				(font
+					(size 1.27 1.27)
+				)
+			)
+		)
+		(property "Footprint" "Package_TO_SOT_SMD:SOT-23-5"
+			(at 34.29 111.125 0)
+			(hide yes)
+			(show_name no)
+			(do_not_autoplace no)
+			(effects
+				(font
+					(size 1.27 1.27)
+				)
+			)
+		)
+		(property "Datasheet" "https://www.diodes.com/assets/Datasheets/AP2112.pdf"
+			(at 34.29 116.84 0)
+			(hide yes)
+			(show_name no)
+			(do_not_autoplace no)
+			(effects
+				(font
+					(size 1.27 1.27)
+				)
+			)
+		)
+		(property "Description" "600mA low dropout linear regulator, with enable pin, 3.8V-6V input voltage range, 3.3V fixed positive output, SOT-23-5"
+			(at 34.29 119.38 0)
+			(hide yes)
+			(show_name no)
+			(do_not_autoplace no)
+			(effects
+				(font
+					(size 1.27 1.27)
+				)
+			)
+		)
+		(pin "3"
+		)
+		(pin "2"
+		)
+		(pin "5"
+		)
+		(pin "4"
+		)
+		(pin "1"
+		)
+		(instances
+			(project "CH569W"
+				(path "/5f355040-3c98-408f-a4c4-e9b21b64c196"
+					(reference "U4")
+					(unit 1)
+				)
+			)
+		)
+	)
+	(symbol
 		(lib_id "power:GND")
 		(at 264.16 44.45 0)
@@
 	(symbol
 		(lib_id "Device:C_Small")
-		(at 48.26 121.92 0)
+		(at 48.26 119.38 0)
 		(mirror y)
 		(unit 1)
@@
 		(fields_autoplaced yes)
 		(property "Reference" "C25"
-			(at 45.72 120.6499 0)
+			(at 45.72 118.1099 0)
 			(show_name no)
 			(do_not_autoplace no)
@@
 		)
 		(property "Value" "3.3uF"
-			(at 45.72 123.1899 0)
+			(at 45.72 120.6499 0)
 			(show_name no)
 			(do_not_autoplace no)
@@
 		)
 		(property "Footprint" "Capacitor_SMD:C_0603_1608Metric"
-			(at 48.26 121.92 0)
+			(at 48.26 119.38 0)
 			(hide yes)
 			(show_name no)
@@
 		)
 		(property "Datasheet" ""
-			(at 48.26 121.92 0)
+			(at 48.26 119.38 0)
 			(hide yes)
 			(show_name no)
@@
 		)
 		(property "Description" "Unpolarized capacitor, small symbol"
-			(at 48.26 132.08 0)
+			(at 48.26 129.54 0)
 			(hide yes)
 			(show_name no)
@@
 	)
 	(symbol
-		(lib_id "Regulator_Linear:LT1117-3.3")
-		(at 34.29 119.38 0)
-		(unit 1)
-		(body_style 1)
-		(exclude_from_sim no)
-		(in_bom yes)
-		(on_board yes)
-		(in_pos_files yes)
-		(dnp no)
-		(fields_autoplaced yes)
-		(property "Reference" "U3"
-			(at 34.29 113.03 0)
-			(show_name no)
-			(do_not_autoplace no)
-			(effects
-				(font
-					(size 1.27 1.27)
-				)
-			)
-		)
-		(property "Value" "LT1117-3.3"
-			(at 34.29 115.57 0)
-			(show_name no)
-			(do_not_autoplace no)
-			(effects
-				(font
-					(size 1.27 1.27)
-				)
-			)
-		)
-		(property "Footprint" "Package_TO_SOT_SMD:TSOT-23-5"
-			(at 34.29 119.38 0)
-			(hide yes)
-			(show_name no)
-			(do_not_autoplace no)
-			(effects
-				(font
-					(size 1.27 1.27)
-				)
-			)
-		)
-		(property "Datasheet" "https://www.analog.com/media/en/technical-documentation/data-sheets/1117fd.pdf"
-			(at 34.29 119.38 0)
-			(hide yes)
-			(show_name no)
-			(do_not_autoplace no)
-			(effects
-				(font
-					(size 1.27 1.27)
-				)
-			)
-		)
-		(property "Description" "800mA Low-Dropout Linear Regulator, 3.3V fixed output, SOT-223/TO-263"
-			(at 34.29 119.38 0)
-			(hide yes)
-			(show_name no)
-			(do_not_autoplace no)
-			(effects
-				(font
-					(size 1.27 1.27)
-				)
-			)
-		)
-		(pin "1"
-		)
-		(pin "3"
-		)
-		(pin "2"
-		)
-		(instances
-			(project "CH569W"
-				(path "/5f355040-3c98-408f-a4c4-e9b21b64c196"
-					(reference "U3")
-					(unit 1)
-				)
-			)
-		)
-	)
-	(symbol
 		(lib_id "power:GND")
 		(at 264.16 64.77 0)
@@
 	(symbol
 		(lib_id "power:GND")
-		(at 20.32 124.46 0)
+		(at 20.32 121.92 0)
 		(unit 1)
 		(body_style 1)
@@
 		(fields_autoplaced yes)
 		(property "Reference" "#PWR058"
-			(at 20.32 130.81 0)
+			(at 20.32 128.27 0)
 			(hide yes)
 			(show_name no)
@@
 		)
 		(property "Value" "GND"
-			(at 20.32 129.54 0)
+			(at 20.32 127 0)
 			(show_name no)
 			(do_not_autoplace no)
@@
 		)
 		(property "Footprint" ""
-			(at 20.32 124.46 0)
+			(at 20.32 121.92 0)
 			(hide yes)
 			(show_name no)
@@
 		)
 		(property "Datasheet" ""
-			(at 20.32 124.46 0)
+			(at 20.32 121.92 0)
 			(hide yes)
 			(show_name no)
@@
 		)
 		(property "Description" "Power symbol creates a global label with name \"GND\" , ground"
-			(at 20.32 124.46 0)
+			(at 20.32 121.92 0)
 			(hide yes)
 			(show_name no)
@@
 	(symbol
 		(lib_id "Device:C_Small")
-		(at 20.32 121.92 0)
+		(at 20.32 119.38 0)
 		(mirror y)
 		(unit 1)
@@
 		(fields_autoplaced yes)
 		(property "Reference" "C24"
-			(at 17.78 120.6499 0)
+			(at 17.78 118.1099 0)
 			(show_name no)
 			(do_not_autoplace no)
@@
 		)
 		(property "Value" "3.3uF"
-			(at 17.78 123.1899 0)
+			(at 17.78 120.6499 0)
 			(show_name no)
 			(do_not_autoplace no)
@@
 		)
 		(property "Footprint" "Capacitor_SMD:C_0603_1608Metric"
-			(at 20.32 121.92 0)
+			(at 20.32 119.38 0)
 			(hide yes)
 			(show_name no)
@@
 		)
 		(property "Datasheet" ""
-			(at 20.32 121.92 0)
+			(at 20.32 119.38 0)
 			(hide yes)
 			(show_name no)
@@
 		)
 		(property "Description" "Unpolarized capacitor, small symbol"
-			(at 20.32 132.08 0)
+			(at 20.32 129.54 0)
 			(hide yes)
 			(show_name no)
@@
 	(symbol
 		(lib_id "power:+3V3")
-		(at 48.26 119.38 0)
+		(at 48.26 116.84 0)
 		(unit 1)
 		(body_style 1)
@@
 		(fields_autoplaced yes)
 		(property "Reference" "#PWR057"
-			(at 48.26 123.19 0)
+			(at 48.26 120.65 0)
 			(hide yes)
 			(show_name no)
@@
 		)
 		(property "Value" "+3V3"
-			(at 48.26 114.3 0)
+			(at 48.26 111.76 0)
 			(show_name no)
 			(do_not_autoplace no)
@@
 		)
 		(property "Footprint" ""
-			(at 48.26 119.38 0)
+			(at 48.26 116.84 0)
 			(hide yes)
 			(show_name no)
@@
 		)
 		(property "Datasheet" ""
-			(at 48.26 119.38 0)
+			(at 48.26 116.84 0)
 			(hide yes)
 			(show_name no)
@@
 		)
 		(property "Description" "Power symbol creates a global label with name \"+3V3\""
-			(at 48.26 119.38 0)
+			(at 48.26 116.84 0)
 			(hide yes)
 			(show_name no)
