File: Misc/heart-blinky/heart-blinky.kicad_pcb (KiCad board)
At the start: 2 copper layers, 54.5 x 54.5 mm, 48 parts, among them J2 BAT+, J3 BAT-, Q1 AO3401A, SW1 e_manuel, U1 NCP1117-5.0_SOT223, U3 LMC555xM

Commit message: kcfjaj
Routing:
- net GND: vias 68 -> 72
