File: MCU/CH559-MASS/CH559-MASS.kicad_pcb (KiCad board)
At the start: 4 copper layers, 59.9 x 19.9 mm, 27 parts, among them J1 USB_C_Receptacle_USB2.0_16P, J2 GPIO1, J3 GPIO2, J4 GPIO3, J5 5V, J6 GPIO4, SW1 RST, U1 CH559L, U2 MKDN128GIL-ZC, U4 AZ1117-3.3, Y1 Crystal_GND24

Commit message: jafh
Parts:
- removed U2: MKDN128GIL-ZC, footprints:MKDN128GIL-ZC
- added U3: MKDN128GCL-AB, footprints:MKDN128GCL-AB, F.Cu at (164.4, 118.3)
- moved C3 0.30 mm to (164.4, 126.8)
Routing:
- net /CS: track 17.3 -> 19.7 mm
- net +3V3: track 15.9 -> 17.9 mm, vias 5 -> 7
- net Net-(J3-Pin_1): track 27.1 -> 28.2 mm
- net Net-(J6-Pin_7): track 19.8 -> 19.0 mm

Commit message: Resolve via size
Routing:
- net Net-(J4-Pin_3): track 21.3 -> 22.0 mm, vias 2 -> 1
- net Net-(J2-Pin_6): track 20.7 -> 21.2 mm
Changed lines of the file:
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@@
 	)
 	(segment
-		(start 169.0679 116.5229)
-		(end 159.6 116.5229)
-		(width 0.2)
+		(start 154.9 115.410001)
+		(end 154.9 115.02)
+		(width 0.1)
 		(layer "F.Cu")
 		(net "Net-(J1-D--PadA7)")
 	)
 	(segment
-		(start 154.82 115.429999)
-		(end 154.649999 115.6)
+		(start 169.0679 116.5229)
+		(end 159.6 116.5229)
 		(width 0.2)
 		(layer "F.Cu")
@@
 	)
 	(segment
-		(start 154.82 114.81)
-		(end 154.82 115.429999)
+		(start 154.9 115.349999)
+		(end 154.649999 115.6)
 		(width 0.2)
 		(layer "F.Cu")
@@
 	)
 	(segment
-		(start 154.61 114.6)
-		(end 154.82 114.81)
-		(width 0.2)
+		(start 154.850001 115.46)
+		(end 154.9 115.410001)
+		(width 0.1)
 		(layer "F.Cu")
 		(net "Net-(J1-D--PadA7)")
@@
 	)
 	(segment
-		(start 154.649999 115.6)
-		(end 153.925 115.6)
-		(width 0.1)
+		(start 154.9 114.89)
+		(end 154.61 114.6)
+		(width 0.2)
 		(layer "F.Cu")
 		(net "Net-(J1-D--PadA7)")
 	)
 	(segment
-		(start 154.850001 115.46)
-		(end 154.82 115.429999)
+		(start 154.649999 115.6)
+		(end 153.925 115.6)
 		(width 0.1)
 		(layer "F.Cu")
@@
 		(net "Net-(J1-D--PadA7)")
 	)
+	(segment
+		(start 154.9 115.02)
+		(end 154.9 115.349999)
+		(width 0.2)
+		(layer "F.Cu")
+		(net "Net-(J1-D--PadA7)")
+	)
+	(segment
+		(start 154.9 115.02)
+		(end 154.9 114.89)
+		(width 0.2)
+		(layer "F.Cu")
+		(net "Net-(J1-D--PadA7)")
+	)
 	(via
 		(at 155.3 115.46)
@@
 	)
 	(segment
-		(start 187.5 126.013994)
-		(end 189.222344 124.29165)
+		(start 189.222344 124.29165)
+		(end 193.180456 124.29165)
 		(width 0.0889)
 		(layer "F.Cu")
@@
 	)
 	(segment
-		(start 189.222344 124.29165)
-		(end 193.180456 124.29165)
+		(start 180.86 125.26)
+		(end 180.235766 125.884234)
 		(width 0.0889)
 		(layer "F.Cu")
@@
 	)
 	(segment
-		(start 180.86 125.26)
-		(end 180.235766 125.884234)
+		(start 187.306795 126.207199)
+		(end 189.222344 124.29165)
 		(width 0.0889)
 		(layer "F.Cu")
@@
 	)
 	(segment
+		(start 187.306795 126.341)
+		(end 187.306795 126.207199)
+		(width 0.0889)
+		(layer "F.Cu")
+		(net "Net-(J2-Pin_6)")
+	)
+	(segment
 		(start 180.235766 125.884234)
 		(end 175.795766 125.884234)
@@
 	)
 	(via
-		(at 187.5 126.013994)
-		(size 0.25)
-		(drill 0.15)
+		(at 187.306795 126.341)
+		(size 0.508)
+		(drill 0.2032)
 		(layers "F.Cu" "B.Cu")
 		(net "Net-(J2-Pin_6)")
@@
 	)
 	(segment
-		(start 183.063618 126.013994)
-		(end 187.5 126.013994)
+		(start 186.850029 125.884234)
+		(end 187.306795 126.341)
 		(width 0.0889)
 		(layer "B.Cu")
@@
 	)
 	(segment
-		(start 175.71 126.47)
-		(end 175.94165 126.23835)
+		(start 182.933858 125.884234)
+		(end 186.850029 125.884234)
 		(width 0.0889)
-		(layer "F.Cu")
-		(net "Net-(J2-Pin_8)")
+		(layer "B.Cu")
+		(net "Net-(J2-Pin_6)")
 	)
 	(segment
-		(start 188.98615 124.11385)
-		(end 195.542656 124.11385)
+		(start 175.71 126.47)
+		(end 175.94165 126.23835)
 		(width 0.0889)
 		(layer "F.Cu")
@@
 	)
 	(segment
-		(start 187.13 125.97)
-		(end 188.98615 124.11385)
+		(start 175.94165 126.23835)
+		(end 180.133098 126.23835)
 		(width 0.0889)
 		(layer "F.Cu")
@@
 	)
 	(segment
-		(start 175.94165 126.23835)
-		(end 180.133098 126.23835)
+		(start 186.759 126.341)
+		(end 188.98615 124.11385)
 		(width 0.0889)
 		(layer "F.Cu")
@@
 	)
 	(segment
-		(start 187.13 126.47)
-		(end 187.13 125.97)
+		(start 195.542656 124.11385)
+		(end 197.064108 125.635302)
 		(width 0.0889)
 		(layer "F.Cu")
@@
 	)
 	(segment
-		(start 195.542656 124.11385)
-		(end 197.064108 125.635302)
+		(start 188.98615 124.11385)
+		(end 195.542656 124.11385)
 		(width 0.0889)
 		(layer "F.Cu")
@@
 	)
 	(segment
+		(start 185.78 126.341)
+		(end 186.759 126.341)
+		(width 0.0889)
+		(layer "F.Cu")
+		(net "Net-(J2-Pin_8)")
+	)
+	(segment
 		(start 180.133098 126.23835)
 		(end 180.933648 125.4378)
@@
 	)
 	(via
-		(at 187.13 126.47)
-		(size 0.25)
-		(drill 0.15)
+		(at 185.78 126.341)
+		(size 0.508)
+		(drill 0.2032)
 		(layers "F.Cu" "B.Cu")
 		(net "Net-(J2-Pin_8)")
@@
 	)
 	(segment
-		(start 187.13 126.47)
-		(end 183.116086 126.47)
+		(start 185.664275 126.456725)
+		(end 185.78 126.341)
+		(width 0.0889)
+		(layer "B.Cu")
+		(net "Net-(J2-Pin_8)")
+	)
+	(segment
+		(start 183.102811 126.456725)
+		(end 185.664275 126.456725)
 		(width 0.0889)
 		(layer "B.Cu")
@@
 	)
 	(segment
-		(start 202.819189 121.789191)
-		(end 202.819189 121.005221)
-		(width 0.0889)
-		(layer "F.Cu")
-		(net "Net-(J4-Pin_3)")
-	)
-	(segment
 		(start 202.819189 121.005221)
 		(end 203.299108 120.525302)
@@
 	)
 	(via
-		(at 202.819189 121.789191)
-		(size 0.25)
-		(drill 0.15)
-		(layers "F.Cu" "B.Cu")
-		(net "Net-(J4-Pin_3)")
-	)
-	(via
 		(at 187.27 122.23)
 		(size 0.508)
@@
 		(width 0.0889)
 		(layer "B.Cu")
+		(net "Net-(J4-Pin_3)")
+	)
+	(segment
+		(start 202.819189 121.789191)
+		(end 202.819189 121.005221)
+		(width 0.0889)
+		(layer "B.Cu")
+		(net "Net-(J4-Pin_3)")
+	)
+	(segment
+		(start 202.819189 121.005221)
+		(end 203.299108 120.525302)
+		(width 0.0889)
+		(layer "B.Cu")

Commit message: fhahj
Parts:
- removed D2: SP0502BAHT, Package_TO_SOT_SMD:SOT-23
- removed Y1: Crystal_GND24, Crystal:Crystal_SMD_3225-4Pin_3.2x2.5mm
- added C10: 10uF, Capacitor_SMD:C_0805_2012Metric, F.Cu at (173.1, 124.3)
- added LED1: WS2812B-B/W, lcsc_footprints:C2761795_LED-SMD_4P-L5_0-W5_0-TL_WS2812B-B, F.Cu at (198.1, 119.8)
- added LED2: WS2812B-B/W, lcsc_footprints:C2761795_LED-SMD_4P-L5_0-W5_0-TL_WS2812B-B, F.Cu at (192.8, 119.8)
- added X1: OT252012MJBA4SL, lcsc_footprints:C669073_OSC-SMD_4P-L2_5-W2_0-BL, F.Cu at (173.3, 127.5)
- C2: value 3.3uF -> 10uF
- C5: value 18 pF -> 100nF
- C6: value 18 pF -> 10uF
- C7, C8, C9: value 3.3uF -> 10 uF
- D1: value PTVS7V5Z1USK -> PTVS5V0S1UR,115; footprint Diode_SMD:Nexperia_DSN1608-2_1.6x0.8mm -> lcsc_footprints:C478011_SOD-123_L2_8-W1_8-LS3_7-RD
- moved C6 21.2 mm to (189.2, 121.5), turned to 90 degrees
- moved D1 1.11 mm to (155.3, 121.7), turned to 180 degrees
- moved C5 0.86 mm to (169.8, 126.5), turned to 0 degrees
- moved C7 0.85 mm to (158.6, 121.5)
Connections:
- C5 pad 1: /XI -> GND
- C5 pad 2: GND -> +3V3
- C6 pad 1: /XO -> +5V
- J3 pad 9: Net-(J3-Pin_9) -> GND
- U1 pad 17: /XO -> unconnected-(U1-P4.7/XO/SCK_-Pad17)
- U1 pad 24: Net-(J3-Pin_9) -> Net-(LED1-DIN)
Routing:
- net Net-(J3-Pin_9): track 42.5 -> 0.00 mm, vias 2 -> 0
- net Net-(LED1-DIN): track 0.00 -> 40.6 mm, vias 0 -> 2
- net +5V: track 39.2 -> 65.1 mm, vias 3 -> 4
- net Net-(LED1-DOUT): track 0.00 -> 12.9 mm, vias 0 -> 2
- net /XO: track 11.7 -> 0.00 mm
- net +3V3: track 17.9 -> 24.9 mm, vias 7 -> 8
- net /XI: track 11.4 -> 6.12 mm
- net /D+: track 29.4 -> 24.4 mm
- net /D-: track 29.3 -> 24.4 mm
- net GND: track 28.7 -> 30.1 mm, vias 25 -> 26

Commit message: ifjqU
Parts:
- removed U3: MKDN128GCL-AB, footprints:MKDN128GCL-AB
- added U2: MKDN512GCL-ZC, lcsc_footprints:C52753986_LGA-16_L12_5-W9_0-P1_27-TL-EP, F.Cu at (164.4, 118.3)
