File: CursedAdapters/CH318/CH318.kicad_pcb (KiCad board)
At the start: 2 copper layers, 80.1 x 40 mm, 19 parts, among them U1 CH318T_C42387966, U2 NCP1117-3.3_SOT223, U3 G2415S, U4 RJ-064-1, Y1 20 MHz

Commit message: Jfhah
Parts:
- moved Y1 82.9 mm to (238.9, 127.1), turned to 180 degrees
- moved U2 74.2 mm to (250.8, 124.5), turned to -90 degrees
- moved C5 68.1 mm to (248.5, 117.2), turned to 90 degrees
- moved C7 67.1 mm to (242.8, 113.1), turned to 90 degrees
- moved C6 62.9 mm to (239.7, 113.1), turned to 90 degrees
- moved C9 61.5 mm to (245.4, 117.4), turned to -90 degrees
- moved C2 60.0 mm to (243.4, 127.2), turned to 90 degrees
- moved U3 57.4 mm to (226.7, 119.3), turned to 90 degrees
- moved C8 53.0 mm to (236.6, 113.3), turned to 90 degrees
- moved C1 51.4 mm to (234.7, 126.1), turned to 90 degrees
- moved R1 50.0 mm to (233.9, 129.7)
Routing:
- net +5V: track 0.00 -> 75.8 mm
- net /LED: track 0.00 -> 49.0 mm, vias 0 -> 3
- net Net-(U1-XO): track 0.00 -> 37.2 mm
- net /DMU: track 0.00 -> 33.5 mm
- net /DPU: track 0.00 -> 32.4 mm
- net /UD2_P: track 0.00 -> 30.0 mm
- net /UD2_N: track 0.00 -> 28.9 mm
- net GND: track 0.00 -> 20.5 mm, vias 0 -> 77
- net Net-(U1-XI): track 0.00 -> 8.52 mm
- net /DPX: track 0.00 -> 7.49 mm
- net /DMX: track 0.00 -> 6.91 mm
- net Net-(U3-MX1+): track 0.00 -> 6.13 mm
- net Net-(U3-MX1-): track 0.00 -> 6.10 mm
- net Net-(U1-AVDDK): track 0.00 -> 5.88 mm
- net Net-(R3-Pad2): track 0.00 -> 5.69 mm, vias 0 -> 2
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- added copper zone on B.Cu, net +3V3
- added copper zone on F.Cu, net +3V3
- added copper zone on In1.Cu, net GND
- added copper zone on In2.Cu, net GND
Other:
- copper layers 2 -> 4

Commit message: jfhah
Parts:
- moved C1 7.18 mm to (241.9, 126.9)
- moved R1 2.28 mm to (236.0, 128.7), turned to 90 degrees
- moved C2 0.69 mm to (243.8, 126.6)
Routing:
- net Net-(U1-XO): track 37.2 -> 8.19 mm
- net GND: track 20.5 -> 23.9 mm
- net Net-(U1-XI): track 8.52 -> 5.65 mm

Commit message: jru
Routing:
- net +5V: track 75.8 -> 49.9 mm, vias 0 -> 2
- net GND: track 23.9 -> 20.4 mm
- net +3V3: vias 3 -> 4
Changed lines of the file:
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@@
-	)
-	(segment
-		(start 239.687919 111.230241)
-		(end 239.687919 111.669401)
-		(width 0.152552)
-		(layer "F.Cu")
-		(net "GND")
 	)
 	(segment
@@
 	)
 	(segment
+		(start 239.687919 111)
+		(end 239.687919 112.170988)
+		(width 0.152552)
+		(layer "F.Cu")
+		(net "GND")
+	)
+	(segment
 		(start 249.17982 116.229425)
 		(end 249.561659 116.229425)
@@
 		(start 239.966286 129.047661)
 		(end 240.029637 128.98431)
-		(width 0.152552)
-		(layer "F.Cu")
-		(net "GND")
-	)
-	(segment
-		(start 240.575225 107.886935)
-		(end 239.687919 108.774241)
 		(width 0.152552)
 		(layer "F.Cu")
@@
 	)
 	(segment
-		(start 239.687919 108.774241)
-		(end 239.687919 111.230241)
-		(width 0.152552)
-		(layer "F.Cu")
-		(net "GND")
-	)
-	(segment
-		(start 239.687919 111.669401)
-		(end 239.687919 112.170988)
-		(width 0.152552)
-		(layer "F.Cu")
-		(net "GND")
-	)
-	(segment
 		(start 240.029637 128.98431)
 		(end 240.029637 128.799995)
@@
 	)
 	(via
-		(at 240.575225 107.886935)
+		(at 239.687919 111)
 		(size 0.61021)
 		(drill 0.305105)
@@
 	)
 	(via
+		(at 237.94 115.24)
+		(size 0.61021)
+		(drill 0.305105)
+		(layers "F.Cu" "B.Cu")
+		(net "+3V3")
+	)
+	(via
 		(at 245.039116 115.637301)
 		(size 0.61021)
@@
 	)
 	(segment
-		(start 267.960392 111.229608)
-		(end 267.960392 107.365211)
-		(width 0.16018)
-		(layer "F.Cu")
-		(net "+5V")
-	)
-	(segment
 		(start 248.460184 121.319425)
 		(end 248.460184 121.069422)
@@
 	)
 	(segment
-		(start 249.17982 118.129425)
+		(start 248.482656 118.1)
 		(end 248.453231 118.129425)
-		(width 0.16018)
-		(layer "F.Cu")
-		(net "+5V")
-	)
-	(segment
-		(start 251.012714 118.129425)
-		(end 249.633759 118.129425)
-		(width 0.16018)
-		(layer "F.Cu")
-		(net "+5V")
-	)
-	(segment
-		(start 249.633759 118.129425)
-		(end 249.17982 118.129425)
-		(width 0.16018)
+		(width 0.2)
 		(layer "F.Cu")
 		(net "+5V")
@@
 	)
 	(segment
-		(start 267.304407 106.709226)
-		(end 262.432913 106.709226)
-		(width 0.16018)
+		(start 249.89 118.1)
+		(end 248.482656 118.1)
+		(width 0.2)
 		(layer "F.Cu")
 		(net "+5V")
@@
 	)
 	(segment
-		(start 262.432913 106.709226)
-		(end 251.012714 118.129425)
-		(width 0.16018)
-		(layer "F.Cu")
-		(net "+5V")
-	)
-	(segment
 		(start 267.908148 134.081852)
 		(end 267.908148 126.281998)
@@
 	)
 	(segment
-		(start 267.200404 111.989596)
-		(end 267.79179 111.39821)
-		(width 0.16018)
-		(layer "F.Cu")
-		(net "+5V")
-	)
-	(segment
 		(start 266.93 113.478755)
 		(end 266.93 113.024817)
@@
 	)
 	(segment
-		(start 267.79179 111.39821)
-		(end 267.960392 111.229608)
-		(width 0.16018)
-		(layer "F.Cu")
-		(net "+5V")
-	)
-	(segment
 		(start 267.908148 126.281998)
 		(end 266.93 125.303851)
@@
 	)
 	(segment
-		(start 267.960392 107.365211)
-		(end 267.304407 106.709226)
-		(width 0.16018)
-		(layer "F.Cu")
-		(net "+5V")
-	)
-	(segment
 		(start 266.93 113.024817)
 		(end 266.93 112.26)
 		(width 0.16018)
 		(layer "F.Cu")
+		(net "+5V")
+	)
+	(via
+		(at 249.56 119.99)
+		(size 0.61021)
+		(drill 0.305105)
+		(layers "F.Cu" "B.Cu")
+		(net "+5V")
+	)
+	(via
+		(at 249.89 118.1)
+		(size 0.61021)
+		(drill 0.305105)
+		(layers "F.Cu" "B.Cu")
+		(net "+5V")
+	)
+	(segment
+		(start 249.56 119.99)
+		(end 249.56 118.44)
+		(width 0.2)
+		(layer "B.Cu")
+		(net "+5V")
+	)
+	(segment
+		(start 249.56 118.44)
+		(end 249.91 118.09)
+		(width 0.2)
+		(layer "B.Cu")
 		(net "+5V")
 	)
@@
 		(polygon
 			(pts
-				(xy 245.124997 127.35878) (xy 244.594993 127.3537) (xy 242.765297 120.601907) (xy 242.765297 114.293844)
+				(xy 245.124997 127.35878) (xy 244.594993 127.3537) (xy 243.69721 124.040777) (xy 234.63 113.14)
 				(xy 245.039874 112.019268) (xy 250.788761 115.549417) (xy 258.035214 122.795871) (xy 255.890158 131.233788)
 				(xy 245.646473 131.233788) (xy 245.124997 129.30948)
