File: IMU/V1/V1.kicad_pcb (KiCad board)
At the start: 2 copper layers, 41 parts, among them J1 USB_C_Receptacle_USB2.0_16P, J2 Conn_02x05_Odd_Even, J3 GND, SW1 NRST, U1 NCP1117-3.3_SOT223, U2 LIS2DW12TR-MS, U3 ICM-42688-P(TOKMAS), U4 MMC5983MA, U5 BMP581, U6 TMP117NAIDRVR, U7 SHT45-AD1F-R2, U8 STM32G431CBT6, Y1 8 MHz

Commit message: fhah
Parts:
- removed BOOT0, SW1: NRST, footprints:KH-6X6X5H-STM_SKE
- added SW2: NRST, lcsc_footprints:C2837531_SW-SMD_4P-L6_0-W6_0-P4_50-LS9_0_H5_0, F.Cu at (157.2, 100.4)
- added SW3: BOOT, lcsc_footprints:C2837531_SW-SMD_4P-L6_0-W6_0-P4_50-LS9_0_H5_0, F.Cu at (157.2, 114.0)
- moved J1 84.5 mm to (227.7, 99.9), turned to 90 degrees
- moved C10 84.1 mm to (217.1, 109.3), turned to 90 degrees
- moved C15 83.7 mm to (220.7, 107.8), turned to 90 degrees
- moved C1 79.5 mm to (208.5, 105.2), turned to 270 degrees
- moved C16 77.4 mm to (214.5, 109.3), turned to 90 degrees
- moved C14 75.2 mm to (211.8, 109.3), turned to 90 degrees
- moved C2 74.8 mm to (203.9, 99.4), turned to 180 degrees
- moved C13 70.4 mm to (203.3, 106.5), turned to 180 degrees
- moved R1 70.0 mm to (207.2, 111.3)
- moved J2 69.6 mm to (225.8, 108.1)
- moved C18 68.8 mm to (221.0, 113.0), turned to 270 degrees
- moved C17 67.9 mm to (204.2, 96.4)
- moved R6 67.2 mm to (208.3, 108.6)
- moved U8 67.1 mm to (215.7, 101.4), turned to -90 degrees
- moved R2 66.6 mm to (203.7, 109.9), turned to 90 degrees
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Connections:
- J2 pad 5: +3V3 -> +3.3V
Routing:
- net +3.3V: track 0.00 -> 196.4 mm
- net /I2C1_SCL: track 0.00 -> 88.7 mm, vias 0 -> 3
- net /I2C2_SCL: track 0.00 -> 79.3 mm, vias 0 -> 5
- net /I2C2_SDA: track 0.00 -> 78.3 mm, vias 0 -> 5
- net /BOOT0: track 0.00 -> 78.1 mm, vias 0 -> 2
- net /I2C1_SDA: track 0.00 -> 72.3 mm, vias 0 -> 5
- net Net-(U8-PG10-NRST): track 0.00 -> 68.4 mm
- net GND: track 0.00 -> 67.0 mm, vias 0 -> 103
- net /MAGNET_INT: track 0.00 -> 58.2 mm, vias 0 -> 2
- net /BARO-INT: track 0.00 -> 52.6 mm, vias 0 -> 2
- net /ACCEL-INT-1: track 0.00 -> 38.8 mm, vias 0 -> 2
- net /ACCEL-INT-2: track 0.00 -> 38.5 mm, vias 0 -> 2
- net Net-(J2-Pin_7): track 0.00 -> 36.3 mm, vias 0 -> 1
- net Net-(J2-Pin_9): track 0.00 -> 35.2 mm, vias 0 -> 1
- net +5V: track 0.00 -> 32.3 mm
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- added copper zone on In1.Cu, net GND
- added copper zone on In2.Cu, net GND
Other:
- board outline added: 76.3 x 25.6 mm
- copper layers 2 -> 4
