File: AMP/AB-V2/AB-V2.kicad_sch (KiCad schematic)
At the start: 56 parts, among them J1 AUX, J3 AUX, P1 WJ500V-5.08-3P, Q1 MJL3281AG, Q13 BD140, Q14 BD140, Q15 BD139, Q16 BD139, Q17 BD140, Q18 BD140, Q2 MJL3281AG, Q21 BD139, T1 36Vac, U1 CYA0630-4.7UH

Commit message: Jfhah
Parts:
- removed Q1, Q2: MJL3281AG, lcsc_footprints:C327498_TO-264-3_L20_0-W5_0-P5_45-L, symbol lcsc_imported:MJL3281AG
- added Q1, Q2: 2SC5200N-OSEN, lcsc_footprints:C49055716_TO-3P-3_L15_6-W4_8-P5_45-L, symbol lcsc_imported:2SC5200N-OSEN
Connections:
- net +VDC: now also Q1.2 (C)
- net at C8.1, Q18.1 (E), R23.1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: now also Q2.2 (C)
- net at C6.1, Q18.2 (C), R28.2: now also Q2.1 (B)
- net at R31.2: now also Q1.3 (E)
- net at Q21.1 (E), R30.2: now also Q1.1 (B)
- net at R29.2: now also Q2.3 (E)

Commit message: kfahh
Parts:
- removed C4: 10 pF, Capacitor_SMD:C_0805_2012Metric, symbol Device:C_Small
- removed C8: 100 nF, Capacitor_SMD:C_0805_2012Metric, symbol Device:C_Small
- removed D1: 1SMA4749A, lcsc_footprints:C173489_SMA_L4_4-W2_8-LS5_4-RD, symbol lcsc_imported:1SMA4749A
- removed D3, D4: 1N4007, Diode_THT:D_DO-41_SOD81_P10.16mm_Horizontal, symbol Diode:1N4007
- removed Q1, Q2: 2SC5200N-OSEN, lcsc_footprints:C49055716_TO-3P-3_L15_6-W4_8-P5_45-L, symbol lcsc_imported:2SC5200N-OSEN
- removed Q13, Q14, Q17, Q18: BD140, Package_TO_SOT_THT:TO-126-3_Vertical, symbol Transistor_BJT:BD140
- removed Q15, Q16, Q21: BD139, Package_TO_SOT_THT:TO-126-3_Vertical, symbol Transistor_BJT:BD139
- removed R27: 150, Resistor_SMD:R_0805_2012Metric, symbol Device:R_Small
- removed R28, R30: 100, Resistor_SMD:R_0805_2012Metric, symbol Device:R_Small
- removed R31: 0.47, Resistor_THT:R_Axial_DIN0617_L17.0mm_D6.0mm_P25.40mm_Horizontal, symbol Device:R_Small
- removed R32, R33: 10, Resistor_SMD:R_0805_2012Metric, symbol Device:R_Small
- removed R36: 10k, Resistor_SMD:R_0805_2012Metric, symbol Device:R_Small
- removed U1: CYA0630-4.7UH, lcsc_footprints:C5189748_IND-SMD_L7_2-W6_6_GPSR07X0, symbol lcsc_imported:CYA0630-4_7UH
- added C4: 100 uF, Capacitor_SMD:C_Elec_6.3x7.7, symbol Device:C_Polarized_Small
- added D1: 1N4007, Diode_THT:D_DO-41_SOD81_P10.16mm_Horizontal, symbol Diode:1N4007
- added Q1, Q2, Q7: BD140, Package_TO_SOT_THT:TO-126-3_Vertical, symbol Transistor_BJT:BD140
- added Q3, Q4: BD139, Package_TO_SOT_THT:TO-126-3_Vertical, symbol Transistor_BJT:BD139
- added Q5: 2SC5200N-OSEN, lcsc_footprints:C49055716_TO-3P-3_L15_6-W4_8-P5_45-L, symbol lcsc_imported:2SC5200N-OSEN
- added Q6: 2SA1943-O(Q, lcsc_footprints:C545244_TO-3PL_L20_0-W5_0-P5_45-L_1, symbol lcsc_imported:2SA1943-O(Q
- added R1, R2: CR-L5W-0.33ΩJ, lcsc_footprints:C334290_RES-TH_BD9_5-L22_0-P26_00-D0_7, symbol lcsc_imported:CR-L5W-0_33ΩJ
- added R21: 470, Resistor_SMD:R_0805_2012Metric, symbol Device:R_Small
- added R3: RK09K1130A70, lcsc_footprints:C351173_RES-TH_RK09K1130A70, symbol lcsc_imported:RK09K1130A70
- C1: value 2.2 uF -> 10 uF
- C2, C5: value 100 uF -> 100 pF; footprint Capacitor_THT:CP_Radial_D8.0mm_P3.50mm -> Capacitor_SMD:C_1206_3216Metric
- C3: value 10 pF -> 10 uF; footprint Capacitor_SMD:C_0805_2012Metric -> Capacitor_SMD:C_1206_3216Metric
- C6, C7: value 1 nF -> 470 pF; footprint Capacitor_SMD:C_0805_2012Metric -> Capacitor_SMD:C_1206_3216Metric
- R17: value 3.3k -> 22k
- R19: value 33k -> 3.3k
- R20: value 4.7k -> 22k
- R22: value 1k -> 1.5k
- R23: value 68k -> 33
- R24: value 150 -> 10
- R25: value 150 -> 100; footprint Resistor_SMD:R_0805_2012Metric -> Resistor_SMD:R_1206_3216Metric
- R26: value 33 -> 100; footprint Resistor_SMD:R_0805_2012Metric -> Resistor_SMD:R_1206_3216Metric
- R29: value 0.47 -> 10; footprint Resistor_THT:R_Axial_DIN0617_L17.0mm_D6.0mm_P25.40mm_Horizontal -> Resistor_SMD:R_0805_2012Metric
- Rload1: now not fitted
Connections:
- net +VDC: now also C6.2, R17.1, R18.1, Q4.2 (C), Q5.2 (C); no longer C7.1, R20.1, R24.1, R25.1
- net -VDC: now also C7.1, R22.1, R23.1, Q2.2 (C), Q6.2 (C), Q7.2 (C); no longer R17.2, R18.2, R29.1
- net GND: now also C2.1, C4.2; no longer C2.2, C5.1
- net IN: now also C2.2, R3.2; no longer J1.2 (Pin_2)
- net OUT: now also C3.1, R20.2, R25.1, R26.2, R1.1, R2.2
- net at D2.1 (K): now also C5.1, C7.2, Q3.2 (C), Q7.3 (B)
- net at C6.1: now also R19.2, D1.2 (A), Q4.3 (B)
- net at R22.2: now also C5.2, Q1.2 (C), Q3.3 (B); no longer R23.2
- net at R25.2: now also R24.1, Q4.1 (E)
- net at C3.2: now also R18.2, R19.1; no longer R17.1
- net at C1.2, R16.1: now also Q1.3 (B)
- net at R26.1: now also R29.1, Q7.1 (E)
- net at D2.2 (A): now also D1.1 (K); no longer R24.2
- net at R29.2: now also Q6.1 (B)
- new net: J1.2 (Pin_2), R3.3
- new net: Q2.3 (B), R20.1, R21.2
- new net: Q1.1 (E), Q2.1 (E), R17.2
- new net: C4.1, R21.1
- new net: Q5.1 (B), R24.2
- new net: Q5.3 (E), R1.2
- new net: Q6.3 (E), R2.1
- new net: Q3.1 (E), R23.2
- no-connect marks 0 -> 3
Other:
- moved on the sheet: J1, J3

Commit message: Jfhaz
Parts:
- added C8, C9: 100 uF, Capacitor_THT:CP_Radial_D8.0mm_P3.50mm, symbol Device:C_Polarized
Connections:
- net +VDC: now also C8.1
- net -VDC: now also C9.1
- net GND: now also C8.2, C9.2

Commit message: Kfhah
Connections:
- net GND: now also R3.4 (EH), R3.5 (EH)
- no-connect marks 3 -> 1
