File: Networking/Ch398/Ch398.kicad_pcb (KiCad board)
At the start: 4 copper layers, 92.7 x 29.7 mm, 38 parts, among them U1 HR682430E, U2 CH398X5, U3 HC-USB3.0-L168-WP, Y1 25 MHz

Commit message: Jfhah
Parts:
- moved C9 5.34 mm to (213.5, 121.6)
- moved C21 5.26 mm to (211.9, 121.6), turned to 90 degrees
- moved C8 1.88 mm to (210.4, 121.6)
Routing:
- net /AVDD33: track 155.8 -> 54.4 mm, vias 3 -> 5
- net /AVDDK: track 132.9 -> 106.2 mm, vias 2 -> 6
- net /SS_TXB: track 22.8 -> 3.63 mm
- net GND: track 34.4 -> 35.0 mm, vias 104 -> 103

Commit message: jghah
Routing:
- net /SS_TXA: track 4.36 -> 4.04 mm, vias 2 -> 0
