File: MCU/STM32F072xB/STM32F072xB.kicad_pcb (KiCad board)
At the start: 4 copper layers, 82.3 x 32.8 mm, 38 parts, among them J1 5V GPIOx, J2 5V GPIOx, J3 GPIOb, J4 GPIOa, J6 USB_C_Receptacle_USB2.0_16P, SW1 NRST, SW2 NRST, U1 STM32F072C8T6, U2 TXS0108EPW, U3 TXS0102DCT, U4 NCP1117-3.3_SOT223, Y1 8 MHz

Commit message: kafh
Parts:
- removed R8, R9: 22, Resistor_SMD:R_0603_1608Metric
- moved C11 0.06 mm to (187.5, 121.0)
Connections:
- J6 pad A6: Net-(J6-D+-PadA6) -> /D+
- J6 pad A7: Net-(J6-D--PadA7) -> /D-
- J6 pad B6: Net-(J6-D+-PadA6) -> /D+
- J6 pad B7: Net-(J6-D--PadA7) -> /D-
Routing:
- net +3V3: track 0.00 -> 165.6 mm
- net +5V: track 0.00 -> 125.9 mm
- net Net-(U1-PA7): track 0.00 -> 56.4 mm, vias 0 -> 2
- net Net-(J4-Pin_2): track 0.00 -> 55.7 mm, vias 0 -> 1
- net Net-(J3-Pin_12): track 0.00 -> 53.8 mm, vias 0 -> 1
- net Net-(J3-Pin_16): track 0.00 -> 52.7 mm, vias 0 -> 1
- net Net-(J3-Pin_14): track 0.00 -> 52.2 mm, vias 0 -> 1
- net GND: track 0.00 -> 51.8 mm, vias 0 -> 33
- net Net-(U1-PA6): track 0.00 -> 50.4 mm, vias 0 -> 2
- net Net-(J3-Pin_15): track 0.00 -> 50.1 mm, vias 0 -> 1
- net Net-(J3-Pin_13): track 0.00 -> 50.0 mm, vias 0 -> 1
- net Net-(J3-Pin_11): track 0.00 -> 48.9 mm, vias 0 -> 1
- net Net-(U1-PA0): track 0.00 -> 48.1 mm, vias 0 -> 2
- net Net-(J3-Pin_2): track 0.00 -> 47.8 mm
- net Net-(J4-Pin_1): track 0.00 -> 47.4 mm, vias 0 -> 2
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- added copper zone on In2.Cu, net GND

Commit message: buck
Parts:
- added C15: 4.7 uF, Capacitor_SMD:C_0805_2012Metric, F.Cu at (210.2, 102.3)
- added C16: 100 nF, Capacitor_SMD:C_0805_2012Metric, F.Cu at (212.2, 102.3)
- added C17: 47 uF, lcsc_footprints:C141425_CAP-SMD_BD6_3-L6_6-W6_6-FD, F.Cu at (234.0, 103.5)
- added Cboot1: 100 nF, Capacitor_SMD:C_0805_2012Metric, F.Cu at (221.9, 101.6)
- added Cff1: 1 pF, Capacitor_SMD:C_0805_2012Metric, F.Cu at (225.4, 101.6)
- added J5: Vin, footprints:WJ500V-5.08-2P, F.Cu at (203.6, 105.5)
- added Renb1: 200k, Resistor_SMD:R_0603_1608Metric, F.Cu at (211.8, 105.6)
- added Rent1: 715k, Resistor_SMD:R_0603_1608Metric, F.Cu at (210.3, 105.6)
- added Rfbb1: 19.1k, Resistor_SMD:R_0603_1608Metric, F.Cu at (214.0, 102.1)
- added Rfbt1: 100k, Resistor_SMD:R_0603_1608Metric, F.Cu at (215.6, 102.1)
- added U5: LMR51625XDDCR, lcsc_footprints:C44750835_SOT-23-6_L2_9-W1_6-P0_95-LS2_9-BL, F.Cu at (218.2, 103.0)
- added U6: CYA0630-10UH, lcsc_footprints:C5189958_IND-SMD_L7_2-W6_6_GPSR07X0, F.Cu at (225.3, 106.2)
- moved C7 1.38 mm to (211.8, 109.7)
Connections:
- R3 pad 2: +3V3 -> GND
- SW2 pad 1: GND -> +3V3
Routing:
- net +5V: track 125.9 -> 167.4 mm, vias 0 -> 3
- net Net-(J5-Pin_1): track 0.00 -> 13.9 mm
- net /FB: track 0.00 -> 12.9 mm, vias 0 -> 2
- net Net-(U5-EN): track 0.00 -> 10.7 mm
- net GND: track 51.8 -> 61.5 mm, vias 33 -> 36
- net Net-(U5-SW): track 0.00 -> 7.65 mm
- net /BOOT0: track 20.4 -> 12.8 mm
- net Net-(J3-Pin_2): track 47.8 -> 51.5 mm
- net Net-(U5-CB): track 0.00 -> 2.31 mm
- net +3V3: track 165.6 -> 166.0 mm, vias 0 -> 2

Commit message: forgor gnd
Routing:
- net GND: track 61.5 -> 64.4 mm, vias 36 -> 37

Commit message: kfdh
Parts:
- added C18: 47 uF, lcsc_footprints:C141425_CAP-SMD_BD6_3-L6_6-W6_6-FD, F.Cu at (235.5, 110.5)
Routing:
- net +5V: track 167.4 -> 173.7 mm, vias 3 -> 4
- net GND: track 64.4 -> 67.0 mm, vias 37 -> 38
