File: MCU/STM32F072xB/STM32F072xB.kicad_sch (KiCad schematic)
At the start: 38 parts, among them J1 5V GPIOx, J2 5V GPIOx, J3 GPIOb, J4 GPIOa, J6 USB_C_Receptacle_USB2.0_16P, SW1 NRST, SW2 NRST, U1 STM32F072C8T6, U2 TXS0108EPW, U3 TXS0102DCT, U4 NCP1117-3.3_SOT223, Y1 8 MHz

Commit message: kafh
Parts:
- removed R8, R9: 22, Resistor_SMD:R_0603_1608Metric, symbol Device:R_Small
Connections:
- net D+: now also J6.A6 (D+), J6.B6 (D+)
- net D-: now also J6.A7 (D-), J6.B7 (D-)
Changed lines of the file:
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@@
 	(paper "A4")
 	(junction
-		(at 233.68 59.69)
-		(diameter 0)
-		(color 0 0 0 0)
-	)
-	(junction
 		(at 53.34 137.16)
 		(diameter 0)
@@
 	)
 	(junction
-		(at 233.68 54.61)
-		(diameter 0)
-		(color 0 0 0 0)
-	)
-	(junction
 		(at 252.73 77.47)
 		(diameter 0)
@@
 	)
 	(label "D-"
-		(at 228.6 54.61 180)
+		(at 233.68 54.61 180)
 		(effects
 			(font
@@
 	)
 	(label "D+"
-		(at 228.6 59.69 180)
+		(at 233.68 59.69 180)
 		(effects
 			(font
@@
 	)
 	(symbol
-		(lib_id "Device:R_Small")
-		(at 231.14 59.69 90)
-		(mirror x)
-		(unit 1)
-		(body_style 1)
-		(exclude_from_sim no)
-		(in_bom yes)
-		(on_board yes)
-		(in_pos_files yes)
-		(dnp no)
-		(fields_autoplaced yes)
-		(property "Reference" "R9"
-			(at 231.14 64.77 90)
-			(show_name no)
-			(do_not_autoplace no)
-			(effects
-				(font
-					(size 1.016 1.016)
-				)
-			)
-		)
-		(property "Value" "22"
-			(at 231.14 62.23 90)
-			(show_name no)
-			(do_not_autoplace no)
-			(effects
-				(font
-					(size 1.27 1.27)
-				)
-			)
-		)
-		(property "Footprint" "Resistor_SMD:R_0603_1608Metric"
-			(at 231.14 59.69 0)
-			(hide yes)
-			(show_name no)
-			(do_not_autoplace no)
-			(effects
-				(font
-					(size 1.27 1.27)
-				)
-			)
-		)
-		(property "Datasheet" ""
-			(at 231.14 59.69 0)
-			(hide yes)
-			(show_name no)
-			(do_not_autoplace no)
-			(effects
-				(font
-					(size 1.27 1.27)
-				)
-			)
-		)
-		(property "Description" "Resistor, small symbol"
-			(at 231.14 59.69 0)
-			(hide yes)
-			(show_name no)
-			(do_not_autoplace no)
-			(effects
-				(font
-					(size 1.27 1.27)
-				)
-			)
-		)
-		(pin "2"
-		)
-		(pin "1"
-		)
-		(instances
-			(project "STM32F072xB"
-				(path "/89b92340-dd4a-422b-a554-a83312c57f0c"
-					(reference "R9")
-					(unit 1)
-				)
-			)
-		)
-	)
-	(symbol
 		(lib_id "power:GND")
 		(at 100.33 73.66 270)
@@
 					(unit 1)
 				)
-			)
-		)
-	)
-	(symbol
-		(lib_id "Device:R_Small")
-		(at 231.14 54.61 90)
-		(unit 1)
-		(body_style 1)
-		(exclude_from_sim no)
-		(in_bom yes)
-		(on_board yes)
-		(in_pos_files yes)
-		(dnp no)
-		(fields_autoplaced yes)
-		(property "Reference" "R8"
-			(at 231.14 49.53 90)
-			(show_name no)
-			(do_not_autoplace no)
-			(effects
-				(font
-					(size 1.016 1.016)
-				)
-			)
-		)
-		(property "Value" "22"
-			(at 231.14 52.07 90)
-			(show_name no)
-			(do_not_autoplace no)
-			(effects
-				(font
-					(size 1.27 1.27)
-				)
-			)
-		)
-		(property "Footprint" "Resistor_SMD:R_0603_1608Metric"
-			(at 231.14 54.61 0)
-			(hide yes)
-			(show_name no)
-			(do_not_autoplace no)
-			(effects
-				(font
-					(size 1.27 1.27)
-				)
-			)
-		)
-		(property "Datasheet" ""
-			(at 231.14 54.61 0)
-			(hide yes)
-			(show_name no)
-			(do_not_autoplace no)
-			(effects
-				(font
-					(size 1.27 1.27)
-				)
-			)
-		)
-		(property "Description" "Resistor, small symbol"
-			(at 231.14 54.61 0)
-			(hide yes)
-			(show_name no)
-			(do_not_autoplace no)
-			(effects
-				(font
-					(size 1.27 1.27)
-				)
-			)
-		)
-		(pin "2"
-		)
-		(pin "1"
-		)
-		(instances
-			(project "STM32F072xB"
-				(path "/89b92340-dd4a-422b-a554-a83312c57f0c"
-					(reference "R8")
-					(unit 1)
-				)

Commit message: buck
Parts:
- added C15: 4.7 uF, Capacitor_SMD:C_0805_2012Metric, symbol Device:C_Small
- added C16, Cboot1: 100 nF, Capacitor_SMD:C_0805_2012Metric, symbol Device:C_Small
- added C17: 47 uF, lcsc_footprints:C141425_CAP-SMD_BD6_3-L6_6-W6_6-FD, symbol lcsc_imported:VT1E470M0605
- added Cff1: 1 pF, Capacitor_SMD:C_0805_2012Metric, symbol Device:C_Small
- added J5: Vin, footprints:WJ500V-5.08-2P, symbol Connector:Screw_Terminal_01x02
- added Renb1: 200k, Resistor_SMD:R_0603_1608Metric, symbol Device:R_Small
- added Rent1: 715k, Resistor_SMD:R_0603_1608Metric, symbol Device:R_Small
- added Rfbb1: 19.1k, Resistor_SMD:R_0603_1608Metric, symbol Device:R_Small
- added Rfbt1: 100k, Resistor_SMD:R_0603_1608Metric, symbol Device:R_Small
- added U5: LMR51625XDDCR, lcsc_footprints:C44750835_SOT-23-6_L2_9-W1_6-P0_95-LS2_9-BL, symbol lcsc_imported:LMR51625XDDCR_C44750835
- added U6: CYA0630-10UH, lcsc_footprints:C5189958_IND-SMD_L7_2-W6_6_GPSR07X0, symbol lcsc_imported:CYA0630-10UH
Connections:
- net +3V3: now also SW2.1; no longer R3.2
- net +5V: now also C17.1, Cff1.1, Rfbt1.1, U6.2
- net GND: now also R3.2, C15.2, C16.2, C17.2, J5.2 (Pin_2), Renb1.1, Rfbb1.2, U5.4 (GND); no longer SW2.1
- new net: C15.1, C16.1, J5.1 (Pin_1), Rent1.2, U5.3 (VIN)
- new net: Cboot1.1, U5.6 (CB)
- new net: Cboot1.2, U5.5 (SW), U6.1
- new net: Renb1.2, Rent1.1, U5.2 (EN)
- new net FB: Cff1.2, Rfbb1.1, Rfbt1.2, U5.1 (FB)
Other:
- moved on the sheet: C1, C10, C11, C12, C13, C14, C2, C3, C4, C5, C6, C7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

Commit message: kfdh
Parts:
- added C18: 47 uF, lcsc_footprints:C141425_CAP-SMD_BD6_3-L6_6-W6_6-FD, symbol lcsc_imported:VT1E470M0605
Connections:
- net +5V: now also C18.1
- net GND: now also C18.2
Changed lines of the file:
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@@
 	)
 	(junction
+		(at 115.57 49.53)
+		(diameter 0)
+		(color 0 0 0 0)
+	)
+	(junction
 		(at 73.66 49.53)
 		(diameter 0)
@@
 	(wire
 		(pts
-			(xy 110.49 49.53) (xy 102.87 49.53)
+			(xy 120.65 49.53) (xy 115.57 49.53)
 		)
 		(stroke
@@
 	(wire
 		(pts
+			(xy 115.57 49.53) (xy 102.87 49.53)
+		)
+		(stroke
+			(width 0)
+			(type default)
+		)
+	)
+	(wire
+		(pts
 			(xy 129.54 111.76) (xy 154.94 111.76)
 		)
@@
 	(symbol
 		(lib_id "power:+5V")
-		(at 110.49 49.53 270)
+		(at 120.65 49.53 270)
 		(unit 1)
 		(body_style 1)
@@
 		(fields_autoplaced yes)
 		(property "Reference" "#PWR049"
-			(at 106.68 49.53 0)
+			(at 116.84 49.53 0)
 			(hide yes)
 			(show_name no)
@@
 		)
 		(property "Value" "+5V"
-			(at 114.3 49.5299 90)
+			(at 124.46 49.5299 90)
 			(show_name no)
 			(do_not_autoplace no)
@@
 		)
 		(property "Footprint" ""
-			(at 110.49 49.53 0)
+			(at 120.65 49.53 0)
 			(hide yes)
 			(show_name no)
@@
 		)
 		(property "Datasheet" ""
-			(at 110.49 49.53 0)
+			(at 120.65 49.53 0)
 			(hide yes)
 			(show_name no)
@@
 		)
 		(property "Description" "Power symbol creates a global label with name \"+5V\""
-			(at 110.49 49.53 0)
+			(at 120.65 49.53 0)
 			(hide yes)
 			(show_name no)
@@
 	)
 	(symbol
+		(lib_id "lcsc_imported:VT1E470M0605")
+		(at 115.57 45.72 90)
+		(unit 1)
+		(body_style 1)
+		(exclude_from_sim no)
+		(in_bom yes)
+		(on_board yes)
+		(in_pos_files yes)
+		(dnp no)
+		(fields_autoplaced yes)
+		(property "Reference" "C18"
+			(at 119.38 45.0567 90)
+			(show_name no)
+			(do_not_autoplace no)
+			(effects
+				(font
+					(size 1.27 1.27)
+				)
+				(justify right)
+			)
+		)
+		(property "Value" "47 uF"
+			(at 119.38 47.5967 90)
+			(show_name no)
+			(do_not_autoplace no)
+			(effects
+				(font
+					(size 1.27 1.27)
+				)
+				(justify right)
+			)
+		)
+		(property "Footprint" "lcsc_footprints:C141425_CAP-SMD_BD6_3-L6_6-W6_6-FD"
+			(at 125.73 45.72 0)
+			(hide yes)
+			(show_name no)
+			(do_not_autoplace no)
+			(effects
+				(font
+					(size 1.27 1.27)
+				)
+			)
+		)
+		(property "Datasheet" "https://www.lcsc.com/datasheet/lcsc_datasheet_2304140030_ROQANG-VT1E470M0605_C141425.pdf"
+			(at 115.443 48.006 0)
+			(hide yes)
+			(show_name no)
+			(do_not_autoplace no)
+			(effects
+				(font
+					(size 1.27 1.27)
+				)
+			)
+		)
+		(property "Description" "VT1E470M0605"
+			(at 115.57 45.72 0)
+			(hide yes)
+			(show_name no)
+			(do_not_autoplace no)
+			(effects
+				(font
+					(size 1.27 1.27)
+				)
+			)
+		)
+		(property "LCSC" "C141425"
+			(at 115.57 45.72 0)
+			(hide yes)
+			(show_name no)
+			(do_not_autoplace no)
+			(effects
+				(font
+					(size 1.27 1.27)
+				)
+			)
+		)
+		(property "Manufacturer" "ROQANG(容强)"
+			(at 115.57 45.72 0)
+			(hide yes)
+			(show_name no)
+			(do_not_autoplace no)
+			(effects
+				(font
+					(size 1.27 1.27)
+				)
+			)
+		)
+		(pin "1"
+		)
+		(pin "2"
+		)
+		(instances
+			(project "STM32F072xB"
+				(path "/89b92340-dd4a-422b-a554-a83312c57f0c"
+					(reference "C18")
+					(unit 1)
+				)
+			)
+		)
+	)
+	(symbol
 		(lib_id "power:GND")
 		(at 102.87 78.74 180)
@@
 					(unit 1)
 				)
+			)
+		)
+	)
+	(symbol
+		(lib_id "power:GND")
+		(at 115.57 41.91 180)
+		(unit 1)
+		(body_style 1)
+		(exclude_from_sim no)
+		(in_bom yes)
+		(on_board yes)
+		(in_pos_files yes)
+		(dnp no)
+		(fields_autoplaced yes)
+		(property "Reference" "#PWR050"
+			(at 115.57 35.56 0)
+			(hide yes)
+			(show_name no)
+			(do_not_autoplace no)
+			(effects
+				(font
+					(size 1.27 1.27)
+				)
+			)
+		)
+		(property "Value" "GND"
+			(at 115.57 36.83 0)
+			(show_name no)
+			(do_not_autoplace no)
+			(effects
+				(font
+					(size 1.27 1.27)
+				)
+			)
+		)
+		(property "Footprint" ""
+			(at 115.57 41.91 0)
+			(hide yes)
+			(show_name no)
+			(do_not_autoplace no)
+			(effects
+				(font
+					(size 1.27 1.27)
+				)
+			)
+		)
+		(property "Datasheet" ""
+			(at 115.57 41.91 0)
+			(hide yes)
+			(show_name no)
+			(do_not_autoplace no)
+			(effects
+				(font
+					(size 1.27 1.27)
+				)
+			)
+		)
+		(property "Description" "Power symbol creates a global label with name \"GND\" , ground"
+			(at 115.57 41.91 0)
+			(hide yes)
+			(show_name no)
+			(do_not_autoplace no)
+			(effects
+				(font
+					(size 1.27 1.27)
+				)
+			)
+		)
+		(pin "1"
+		)
+		(instances
+			(project "STM32F072xB"
+				(path "/89b92340-dd4a-422b-a554-a83312c57f0c"
+					(reference "#PWR050")
+					(unit 1)
+				)
