File: Psu/V1/MCU.kicad_sch (KiCad schematic)
At the start: 15 parts, among them J4 SWD, U5 STM32G474RET6

Commit message: Jfjja
Connections:
- net RELAY_EN: now reaches U5.33 (PB11)
- net DRV_IN2: now reaches U5.44 (PA10)
- no-connect marks 13 -> 11
Other:
- note added: "STM32G474RET6: HRTIM generates the 4-switch buck-boost PWM (CHA1 input leg, CHB1 output leg), 12-bit ADCs close the CV/CC loops, DACs set OVP/OCP thresholds, native USB FS device (CDC/SCPI). No crystal: HSI48 + CRS locks to USB SOF."
- note removed: "STM32G474RET6: HRTIM generates the buck PWM, 12-bit ADCs close the CV/CC loops, DACs set OVP/OCP thresholds, native USB FS device (CDC/SCPI). No crystal: HSI48 + CRS locks to USB SOF."
Changed lines of the file:
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@@
 		)
 	)
-	(text "STM32G474RET6: HRTIM generates the buck PWM, 12-bit ADCs close the CV/CC loops, DACs set OVP/OCP thresholds, native USB FS device (CDC/SCPI). No crystal: HSI48 + CRS locks to USB SOF."
+	(text "STM32G474RET6: HRTIM generates the 4-switch buck-boost PWM (CHA1 input leg, CHB1 output leg), 12-bit ADCs close the CV/CC loops, DACs set OVP/OCP thresholds, native USB FS device (CDC/SCPI). No crystal: HSI48 + CRS locks to USB SOF."
 		(exclude_from_sim no)
 		(at 12.954 14.478 0)
@@
 	)
 	(no_connect
-		(at 195.58 132.08)
-	)
-	(no_connect
 		(at 195.58 144.78)
 	)
@@
 		(at 287.02 149.86)
 	)
-	(no_connect
-		(at 195.58 177.8)
-	)
 	(wire
 		(pts
@@
 	(wire
 		(pts
+			(xy 195.58 132.08) (xy 241.3 132.08)
+		)
+		(stroke
+			(width 0)
+			(type default)
+		)
+	)
+	(wire
+		(pts
 			(xy 195.58 114.3) (xy 241.3 114.3)
 		)
@@
 		)
 	)
+	(wire
+		(pts
+			(xy 195.58 177.8) (xy 241.3 177.8)
+		)
+		(stroke
+			(width 0)
+			(type default)
+		)
+	)
 	(hierarchical_label "IOUT_ADC"
 		(shape bidirectional)
@@
 		)
 	)
+	(hierarchical_label "RELAY_EN"
+		(shape bidirectional)
+		(at 241.3 177.8 0)
+		(effects
+			(font
+				(size 1.27 1.27)
+			)
+			(justify left)
+		)
+	)
 	(hierarchical_label "BTN_PRESET"
 		(shape bidirectional)
@@
 			)
 			(justify right)
+		)
+	)
+	(hierarchical_label "DRV_IN2"
+		(shape bidirectional)
+		(at 241.3 132.08 0)
+		(effects
+			(font
+				(size 1.27 1.27)
+			)
+			(justify left)
 		)
 	)
@@
 			)
 		)
-		(property "Sim.Pins" "12=vout 13=iout 14=vin 15=vss 16=vdd 18=ovp_dac 19=ocp_dac 26=drv_en 30=fault_n 42=drv_in"
+		(property "Sim.Pins" "12=vout 13=iout 14=vin 15=vss 16=vdd 18=ovp_dac 19=ocp_dac 26=drv_en 30=fault_n 33=relay_en 42=drv_in 44=drv_in2"
 			(at 177.8 147.32 0)
 			(hide yes)
@@
 			)
 		)
-		(property "Sim.Params" "vset=50 iset=5 ovp=110 ocp=6 ki=5 kd=3.5u tss=3m fsw=200k"
+		(property "Sim.Params" "vset=50 iset=5 ovp=110 ocp=6 ki=5 kd=3.5u tss=3m fsw=200k tstab=2m"
 			(at 177.8 147.32 0)
 			(hide yes)
