File: Psu/V1/V1.kicad_sch (KiCad schematic)
At the start: 0 parts

Commit message: Jfjja
Other:
- sheet MCU renamed AnalogCtl
- sheet AnalogCtl: file MCU.kicad_sch -> AnalogCtl.kicad_sch
- sheet AnalogCtl ports: added DRV_IN2, RELAY_EN; removed BTN_LOCK, BTN_MODE, BTN_OUT, BTN_PRESET, ENCI_A, ENCI_B, ENCI_SW, ENCV_A, ENCV_B, ENCV_SW, FAN_PWM, FAN_TACH, LCD_BL, LCD_CS, LCD_DC, LCD_MOSI, LCD_RST, LCD_SCK, LED_CC, LED_CV, LED_FLT, LED_OUT, TEMP1_ADC, TEMP2_ADC, USB_DM, USB_DP, V12_ADC
- sheet PowerStage ports: added DRV_IN2, RELAY_EN; removed none

Commit message: Jfhah
Connections:
- no-connect marks 0 -> 4
Other:
- removed sheet UserInterface
- added sheet Buck3V3 (Buck3V3.kicad_sch)
- sheet AnalogCtl ports: added FAN_PWM, TEMP1_ADC, TEMP2_ADC; removed none
Changed lines of the file:
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@@
-	)
-	(sheet
-		(at 340.36 66.04)
-		(size 76.2 121.92)
-		(exclude_from_sim no)
-		(in_bom yes)
-		(on_board yes)
-		(dnp no)
-		(stroke
-			(width 0.1524)
-			(type solid)
-		)
-		(fill
-			(color 0 0 0 0)
-		)
-		(property "Sheetname" "UserInterface"
-			(at 340.36 65.34 0)
-			(show_name no)
-			(do_not_autoplace no)
-			(effects
-				(font
-					(size 1.27 1.27)
-				)
-				(justify left bottom)
-			)
-		)
-		(property "Sheetfile" "UserInterface.kicad_sch"
-			(at 340.36 188.66 0)
-			(show_name no)
-			(do_not_autoplace no)
-			(effects
-				(font
-					(size 1.27 1.27)
-				)
-				(justify left top)
-			)
-		)
-		(pin "ENCV_A" bidirectional
-			(at 340.36 76.2 180)
-			(effects
-				(font
-					(size 1.27 1.27)
-				)
-				(justify left)
-			)
-		)
-		(pin "ENCV_B" bidirectional
-			(at 340.36 81.28 180)
-			(effects
-				(font
-					(size 1.27 1.27)
-				)
-				(justify left)
-			)
-		)
-		(pin "ENCV_SW" bidirectional
-			(at 340.36 86.36 180)
-			(effects
-				(font
-					(size 1.27 1.27)
-				)
-				(justify left)
-			)
-		)
-		(pin "ENCI_A" bidirectional
-			(at 340.36 91.44 180)
-			(effects
-				(font
-					(size 1.27 1.27)
-				)
-				(justify left)
-			)
-		)
-		(pin "ENCI_B" bidirectional
-			(at 340.36 96.52 180)
-			(effects
-				(font
-					(size 1.27 1.27)
-				)
-				(justify left)
-			)
-		)
-		(pin "ENCI_SW" bidirectional
-			(at 340.36 101.6 180)
-			(effects
-				(font
-					(size 1.27 1.27)
-				)
-				(justify left)
-			)
-		)
-		(pin "BTN_OUT" bidirectional
-			(at 340.36 106.68 180)
-			(effects
-				(font
-					(size 1.27 1.27)
-				)
-				(justify left)
-			)
-		)
-		(pin "BTN_MODE" bidirectional
-			(at 340.36 111.76 180)
-			(effects
-				(font
-					(size 1.27 1.27)
-				)
-				(justify left)
-			)
-		)
-		(pin "BTN_PRESET" bidirectional
-			(at 340.36 116.84 180)
-			(effects
-				(font
-					(size 1.27 1.27)
-				)
-				(justify left)
-			)
-		)
-		(pin "BTN_LOCK" bidirectional
-			(at 340.36 121.92 180)
-			(effects
-				(font
-					(size 1.27 1.27)
-				)
-				(justify left)
-			)
-		)
-		(pin "LED_OUT" bidirectional
-			(at 340.36 127 180)
-			(effects
-				(font
-					(size 1.27 1.27)
-				)
-				(justify left)
-			)
-		)
-		(pin "LED_CV" bidirectional
-			(at 340.36 132.08 180)
-			(effects
-				(font
-					(size 1.27 1.27)
-				)
-				(justify left)
-			)
-		)
-		(pin "LED_CC" bidirectional
-			(at 340.36 137.16 180)
-			(effects
-				(font
-					(size 1.27 1.27)
-				)
-				(justify left)
-			)
-		)
-		(pin "LED_FLT" bidirectional
-			(at 340.36 142.24 180)
-			(effects
-				(font
-					(size 1.27 1.27)
-				)
-				(justify left)
-			)
-		)
-		(pin "LCD_CS" bidirectional
-			(at 340.36 147.32 180)
-			(effects
-				(font
-					(size 1.27 1.27)
-				)
-				(justify left)
-			)
-		)
-		(pin "LCD_SCK" bidirectional
-			(at 340.36 152.4 180)
-			(effects
-				(font
-					(size 1.27 1.27)
-				)
-				(justify left)
-			)
-		)
-		(pin "LCD_MOSI" bidirectional
-			(at 340.36 157.48 180)
-			(effects
-				(font
-					(size 1.27 1.27)
-				)
-				(justify left)
-			)
-		)
-		(pin "LCD_RST" bidirectional
-			(at 340.36 162.56 180)
-			(effects
-				(font
-					(size 1.27 1.27)
-				)
-				(justify left)
-			)
-		)
-		(pin "LCD_DC" bidirectional
-			(at 340.36 167.64 180)
-			(effects
-				(font
-					(size 1.27 1.27)
-				)
-				(justify left)
-			)
-		)
-		(pin "LCD_BL" bidirectional
-			(at 340.36 172.72 180)
-			(effects
-				(font
-					(size 1.27 1.27)
-				)
-				(justify left)
-			)
-		)
-		(instances
-			(project "V1"
-				(path "/ac43abac-3a45-4cc0-8cc7-86391d0cc456"
-					(page "6")
-				)
-			)
-		)
 	)
 	(sheet
@@
 			)
 		)
+		(pin "TEMP1_ADC" bidirectional
+			(at 177.8 147.32 180)
+			(effects
+				(font
+					(size 1.27 1.27)
+				)
+				(justify left)
+			)
+		)
+		(pin "TEMP2_ADC" bidirectional
+			(at 177.8 152.4 180)
+			(effects
+				(font
+					(size 1.27 1.27)
+				)
+				(justify left)
+			)
+		)
+		(pin "FAN_PWM" bidirectional
+			(at 254 35.56 0)
+			(effects
+				(font
+					(size 1.27 1.27)
+				)
+				(justify right)
+			)
+		)
 		(instances
 			(project "V1"
@@
 		)
 	)
+	(sheet
+		(at 340.36 66.04)
+		(size 76.2 20.32)
+		(exclude_from_sim no)
+		(in_bom yes)
+		(on_board yes)
+		(dnp no)
+		(stroke
+			(width 0.1524)
+			(type solid)
+		)
+		(fill
+			(color 0 0 0 0)
+		)
+		(property "Sheetname" "Buck3V3"
+			(at 340.36 65.34 0)
+			(show_name no)
+			(do_not_autoplace no)
+			(effects
+				(font
+					(size 1.27 1.27)
+				)
+				(justify left bottom)
+			)
+		)
+		(property "Sheetfile" "Buck3V3.kicad_sch"
+			(at 340.36 87.1 0)
+			(show_name no)
+			(do_not_autoplace no)
+			(effects
+				(font
+					(size 1.27 1.27)
+				)
+				(justify left top)
+			)
+		)
+		(instances
+			(project "V1"
+				(path "/ac43abac-3a45-4cc0-8cc7-86391d0cc456"
+					(page "6")
+				)
+			)
+		)
+	)
+	(wire
+		(pts
+			(xy 91.44 147.32) (xy 177.8 147.32)
+		)
+		(stroke
+			(width 0)
+			(type default)
+		)
+	)
+	(wire
+		(pts
+			(xy 91.44 152.4) (xy 177.8 152.4)
+		)
+		(stroke
+			(width 0)
+			(type default)
+		)
+	)
+	(wire
+		(pts
+			(xy 254 35.56) (xy 340.36 35.56)
+		)
+		(stroke
+			(width 0)
+			(type default)
+		)
+	)
+	(no_connect
+		(at 340.36 25.4)
+	)
+	(no_connect
+		(at 340.36 30.48)
+	)
+	(no_connect
+		(at 340.36 40.64)
+	)
+	(no_connect
+		(at 91.44 142.24)
+	)
 	(sheet_instances

Commit message: jfha
Other:
- note added: "CONTROL"
- note added: "I/O + SUPPLIES"
- note added: "POWER STAGE + SENSING"
