File: Psu/V1/AnalogCtl.kicad_sch (KiCad schematic)
At the start: 100 parts, among them Q101 2N7002, Q102 2N7002, Q103 2N7002, Q104 2N7002, Q105 2N7002, Q106 BC857, Q107 2N7002, Q108 2N7002, SW101 SW_SPST, U101 TL431, U102 LM358, U103 LM393, U104 LM393, U105 LM393, U106 LM358, U107 LM358, U109 LM311, U110 LM311, U111 LM311

Commit message: Jfhah
Parts:
- added D110, D111: D1N4148, Diode_SMD:D_SOD-123, symbol Device:D
- added R170: 6.2k, Resistor_SMD:R_0603_1608Metric, symbol Device:R
- added R171: 4.3k, Resistor_SMD:R_0603_1608Metric, symbol Device:R
- added R172, R173: 10k, Resistor_SMD:R_0603_1608Metric, symbol Device:R
- added R174: 100k, Resistor_SMD:R_0603_1608Metric, symbol Device:R
- added U112: LM393, Package_SO:SOIC-8_3.9x4.9mm_P1.27mm, symbol Comparator:LM393
Connections:
- net +12V: now also U112.8 (V+)
- net +3V3: now also R172.1, R173.1
- net GND: now also R171.2, R174.2, U112.4 (V-)
- net CCN: now reaches D108.1 (K), LED102.1 (K), R137.2, U105.1
- net N1: now reaches D108.2 (A), Q103.3 (D), Q104.1 (G), R129.2
- net EAI: now reaches C105.1, D102.1 (K), D104.2 (A), R124.1, U105.3 (+), U107.7
- net TM: now reaches C106.1, R130.2, R131.1, R159.1, U103.5 (+)
- net EAV: now reaches C103.1, D101.1 (K), D103.2 (A), D106.2 (A), R122.1, U107.1
- net COMP: now reaches D101.2 (A), D102.2 (A), R115.1, R125.2, R148.1
- net WIN: now reaches Q103.1 (G), R110.2, U104.1, U104.7
- net VSPB: now reaches R111.1, U102.6 (-), U102.7, U106.3 (+), U107.3 (+)
- net RAMP: now reaches C108.1, Q106.3 (C), R140.2, U109.3 (-), U110.2 (+), U111.2 (+)
- net VREF3: now reaches R102.1, R106.1, R119.1, R127.1, R156.1, RV101.1, U102.1
- net VREF3: now also R170.1
- new net: R170.2, R171.1, U112.3 (+), U112.5 (+)
- new net: D111.2 (A), R173.2, U112.7
- new net: D110.2 (A), R172.2, U112.1
- new net FAN_PWM: D110.1 (K), D111.1 (K), R174.1
- new net TEMP1_ADC: U112.2 (-)
- new net TEMP2_ADC: U112.6 (-)

Commit message: jfha
Parts:
- C106: value 27n -> 150n
Connections:
- net RAMP_RST: now reaches Q107.1 (G), Q108.1 (G), R160.2, U111.7
- net VREF_LOW: now reaches R156.2, R157.1, RV102.3, U103.6 (-), U105.5 (+)
- net SS_G: now reaches Q101.1 (G), Q102.3 (D), R105.2
Other:
- note added: "+12 V DECOUPLING"
- note added: "3.0 V REFERENCE"
- note added: "CURRENT ERROR AMP (CC) + LIMIT KNOB"
- note added: "ENABLE"
- note added: "ERROR SELECT (CV/CC) + MODE"
- note added: "FAN / TEMPERATURE"
- note added: "OUTPUT WINDOW MONITOR (+/-5 %)"
- note added: "OVP / OCP THRESHOLDS"
- note added: "PWM COMPARATOR 1 (DRV_IN)"
- note added: "PWM COMPARATOR 2 (DRV_IN2)"
- note added: "RAMP GENERATOR"
- note added: "STARTUP TIMER + RELAY ENABLE + FAULT"
- note added: "VOLTAGE ERROR AMP (CV)"
- note added: "VOLTAGE SETPOINT + SOFT-START"
- moved on the sheet: C101, C102, C103, C104, C105, C106, C108, C109, C110, C111, D101, D102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

Commit message: Jfhjh
Parts:
- added C112: 470n, Capacitor_SMD:C_0603_1608Metric, symbol Device:C
- added C113: 100n, Capacitor_SMD:C_0603_1608Metric, symbol Device:C
- added Q109: 2N7002, Package_TO_SOT_SMD:SOT-23, symbol Transistor_FET:2N7002
- added R175, R177: 100k, Resistor_SMD:R_0603_1608Metric, symbol Device:R
- added R176: 6Meg, Resistor_SMD:R_0603_1608Metric, symbol Device:R
- added R178: 10k, Resistor_SMD:R_0603_1608Metric, symbol Device:R
- added R179: 1k, Resistor_SMD:R_0603_1608Metric, symbol Device:R
- added U113: LM393, Package_SO:SOIC-8_3.9x4.9mm_P1.27mm, symbol Comparator:LM393
- C106: value 150n -> 27n
Connections:
- net +12V: now also R176.1, R178.1, U113.8 (V+)
- net GND: now also C112.2, C113.2, Q109.2 (S), U113.4 (V-), U113.5 (+)
- net TM: now also R179.1
- net VIN_ADC: now also R175.1, R177.1
- net VREF3: now also U113.6 (-)
- net RAMP_RST: no longer names the net of Q107.1 (G), Q108.1 (G), R160.2, U111.7
- net SS_G: no longer names the net of Q101.1 (G), Q102.3 (D), R105.2
- net VREF_LOW: no longer names the net of R156.2, R157.1, RV102.3, U103.6 (-), U105.5 (+)
- new net: C112.1, R175.2, R176.2, U113.2 (-)
- new net: C113.1, R177.2, U113.3 (+)
- new net: Q109.3 (D), R179.2
- new net: Q109.1 (G), R178.2, U113.1
- no-connect marks 6 -> 7
Other:
- note added: "8 MEG"
- note removed: "+12 V DECOUPLING"
- note removed: "3.0 V REFERENCE"
- note removed: "CURRENT ERROR AMP (CC) + LIMIT KNOB"
- note removed: "ENABLE"
- note removed: "ERROR SELECT (CV/CC) + MODE"
- note removed: "FAN / TEMPERATURE"
- note removed: "OUTPUT WINDOW MONITOR (+/-5 %)"
- note removed: "OVP / OCP THRESHOLDS"
- note removed: "PWM COMPARATOR 1 (DRV_IN)"
- note removed: "PWM COMPARATOR 2 (DRV_IN2)"
- note removed: "RAMP GENERATOR"
- note removed: "STARTUP TIMER + RELAY ENABLE + FAULT"
- note removed: "VOLTAGE ERROR AMP (CV)"
- note removed: "VOLTAGE SETPOINT + SOFT-START"

Commit message: Jfhh
Parts:
- removed unit 2 of U113
Connections:
- no-connect marks 7 -> 6
Changed lines of the file:
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@@
 	)
 	(no_connect
-		(at 452.12 158.75)
-	)
-	(no_connect
 		(at 182.88 48.26)
 	)
@@
 	(wire
 		(pts
-			(xy 436.88 156.21) (xy 434.34 156.21)
-		)
-		(stroke
-			(width 0)
-			(type default)
-		)
-	)
-	(wire
-		(pts
 			(xy 209.55 50.8) (xy 209.55 54.61)
 		)
@@
 		)
 	)
-	(label "VREF3"
-		(at 436.88 161.29 180)
-		(effects
-			(font
-				(size 1.27 1.27)
-			)
-			(justify right bottom)
-		)
-	)
 	(label "RAMP"
 		(at 473.71 130.81 180)
@@
 	(symbol
 		(lib_id "Comparator:LM393")
-		(at 444.5 158.75 0)
-		(unit 2)
-		(body_style 1)
-		(exclude_from_sim no)
-		(in_bom yes)
-		(on_board yes)
-		(in_pos_files yes)
-		(dnp no)
-		(property "Reference" "U113"
-			(at 451.49 156.84 0)
-			(show_name no)
-			(do_not_autoplace no)
-			(effects
-				(font
-					(size 1.27 1.27)
-				)
-				(justify left)
-			)
-		)
-		(property "Value" "LM393"
-			(at 451.49 158.75 0)
-			(show_name no)
-			(do_not_autoplace no)
-			(effects
-				(font
-					(size 1.27 1.27)
-				)
-				(justify left)
-			)
-		)
-		(property "Footprint" "Package_SO:SOIC-8_3.9x4.9mm_P1.27mm"
-			(at 444.5 158.75 0)
-			(hide yes)
-			(show_name no)
-			(do_not_autoplace no)
-			(effects
-				(font
-					(size 1.27 1.27)
-				)
-			)
-		)
-		(property "Datasheet" ""
-			(at 444.5 158.75 0)
-			(hide yes)
-			(show_name no)
-			(do_not_autoplace no)
-			(effects
-				(font
-					(size 1.27 1.27)
-				)
-			)
-		)
-		(property "Description" ""
-			(at 444.5 158.75 0)
-			(hide yes)
-			(show_name no)
-			(do_not_autoplace no)
-			(effects
-				(font
-					(size 1.27 1.27)
-				)
-			)
-		)
-		(property "Sim.Device" "SUBCKT"
-			(at 444.5 158.75 0)
-			(hide yes)
-			(show_name no)
-			(do_not_autoplace no)
-			(effects
-				(font
-					(size 1.27 1.27)
-				)
-			)
-		)
-		(property "Sim.Library" "${KIPRJMOD}/models/psu_models.lib"
-			(at 444.5 158.75 0)
-			(hide yes)
-			(show_name no)
-			(do_not_autoplace no)
-			(effects
-				(font
-					(size 1.27 1.27)
-				)
-			)
-		)
-		(property "Sim.Name" "LM393"
-			(at 444.5 158.75 0)
-			(hide yes)
-			(show_name no)
-			(do_not_autoplace no)
-			(effects
-				(font
-					(size 1.27 1.27)
-				)
-			)
-		)
-		(property "Sim.Pins" "1=out1 2=inm1 3=inp1 4=vee 5=inp2 6=inm2 7=out2 8=vcc"
-			(at 444.5 158.75 0)
-			(hide yes)
-			(show_name no)
-			(do_not_autoplace no)
-			(effects
-				(font
-					(size 1.27 1.27)
-				)
-			)
-		)
-		(pin "5"
-		)
-		(pin "6"
-		)
-		(pin "7"
-		)
-		(pin "1"
-		)
-		(pin "2"
-		)
-		(pin "3"
-		)
-		(pin "4"
-		)
-		(pin "8"
-		)
-		(instances
-			(project "V1"
-				(path "/ac43abac-3a45-4cc0-8cc7-86391d0cc456/6ff5dedc-2375-436c-82db-06b4588cec6b"
-					(reference "U113")
-					(unit 2)
-				)
-			)
-		)
-	)
-	(symbol
-		(lib_id "Comparator:LM393")
 		(at 264.16 247.65 0)
 		(unit 1)
@@
 					(unit 1)
 				)
-			)
-		)
-	)
-	(symbol
-		(lib_id "power:GND")
-		(at 434.34 156.21 270)
-		(unit 1)
-		(body_style 1)
-		(exclude_from_sim no)
-		(in_bom no)
-		(on_board no)
-		(in_pos_files no)
-		(dnp no)
-		(property "Reference" "#PWR465"
-			(at 434.34 156.21 0)
-			(hide yes)
-			(show_name no)
-			(do_not_autoplace no)
-			(effects
-				(font
-					(size 1.27 1.27)
-				)
-			)
-		)
-		(property "Value" "GND"
-			(at 436.88 156.21 0)
-			(show_name no)
-			(do_not_autoplace no)
-			(effects
-				(font
-					(size 1.27 1.27)
-				)
-			)
-		)
-		(property "Footprint" ""
-			(at 434.34 156.21 0)
-			(hide yes)
-			(show_name no)
-			(do_not_autoplace no)
-			(effects
-				(font
-					(size 1.27 1.27)
-				)
-			)
-		)
-		(property "Datasheet" ""
-			(at 434.34 156.21 0)
-			(hide yes)
-			(show_name no)
-			(do_not_autoplace no)
-			(effects
-				(font
-					(size 1.27 1.27)
-				)
-			)
-		)
-		(property "Description" ""
-			(at 434.34 156.21 0)
-			(hide yes)
-			(show_name no)
-			(do_not_autoplace no)
-			(effects
-				(font
-					(size 1.27 1.27)
-				)
-			)
-		)
-		(pin "1"
-		)
-		(instances
-			(project "V1"
-				(path "/ac43abac-3a45-4cc0-8cc7-86391d0cc456/6ff5dedc-2375-436c-82db-06b4588cec6b"
-					(reference "#PWR465")
-					(unit 1)
-				)

Commit message: Jfhaha
Parts:
- added D112, D113, D114: D1N4148, Diode_SMD:D_SOD-123, symbol Device:D
- C102: value 47n -> 470n
- C104: value 10n -> 470n
- C106: value 27n -> 150n
- R122: value 10k -> 330
- R124: value 47k -> 1k
- R131: value 1k -> 100k
Connections:
- net EAI: now also D112.2 (A)
- net IAMP_INV: now reaches C104.2, C105.2, R123.2, U107.6 (-)
- net IAMP_INV: now also D114.1 (K)
- new net: D113.1 (K), D114.2 (A)
- new net: D112.1 (K), D113.2 (A)
Other:
- note added: "WINDUP CLAMP: limits how far the current amp (EAI) can wind up above its inverting input; keeps constant-current engagement fast"
