File: Psu/V1/Mains.kicad_sch (KiCad schematic)
At the start: 23 parts, among them J10 PE lug, J12 Toroid primary 230V (AA,AB), J13 Toroid secondary SA,SB,SC,SD, J9 IEC C14 inlet, SW7 DPST 250V 6A, T1 SIM: toroid 230V:2x45V 500VA, U8 IRM-10-12 (12V 0.85A)

Commit message: Jfhjh
Parts:
- removed R45: SIM: N-GND ref 1R, symbol Device:R_Small
- added C67: 3300uF 160V, Capacitor_THT:CP_Radial_D35.0mm_P10.00mm_SnapIn, symbol Device:C_Polarized
Connections:
- net +HV: now also C67.1
- net GND: now also C67.2
Other:
- moved on the sheet: R50, R51
