File: Psu/V1/PowerStage.kicad_sch (KiCad schematic)
At the start: 44 parts, among them J2 OUTPUT 0-100V 5A, Q1 IRFS4127PBF, Q2 IRFS4127PBF, U1 IR2184S

Commit message: Jfjja
Parts:
- added C63: 10uF 25V, Capacitor_SMD:C_0805_2012Metric, symbol Device:C_Small
- added C64, C65: 1uF 25V, Capacitor_SMD:C_0603_1608Metric, symbol Device:C_Small
- added C66: 470pF 250V, Capacitor_SMD:C_0805_2012Metric, symbol Device:C_Small
- added D15, D17, D18: BAS21, Package_TO_SOT_SMD:SOT-23, symbol Device:D
- added D16: ES1D, Diode_SMD:D_SMA, symbol Device:D
- added K1: RELAY SPST-NO 12V coil, Relay_THT:Relay_1-Form-A_Schrack-RYII_RM5mm, symbol Relay:Relay_SPST-NO
- added Q4, Q5: IRFS4127PBF, Package_TO_SOT_SMD:TO-263-2, symbol Transistor_FET:IRFS4127
- added Q6: 2N7002, Package_TO_SOT_SMD:SOT-23, symbol Transistor_FET:2N7002
- added R52: 10R 1W, Resistor_SMD:R_1206_3216Metric, symbol Device:R_Small
- added R53, R54: 4.7R, Resistor_SMD:R_0603_1608Metric, symbol Device:R_Small
- added R55, R57, R58: 10k, Resistor_SMD:R_0603_1608Metric, symbol Device:R_Small
- added R56: 2.2R, Resistor_SMD:R_0603_1608Metric, symbol Device:R_Small
- added R59: 100k, Resistor_SMD:R_0603_1608Metric, symbol Device:R_Small
- added R60: 100R, Resistor_SMD:R_0603_1608Metric, symbol Device:R_Small
- added U9: IR2184S, Package_SO:SOIC-8_3.9x4.9mm_P1.27mm, symbol Driver_FET:IR2184
- F1: value 10A fast, 150VDC -> 20A fast, 150VDC
- L1: value 200uH 8A sat -> 200uH 20A sat
- V1: value 120V -> 60V
Connections:
- net +12V: now also C63.1, C65.1, D16.2 (A), D18.1 (K), K1.A1, U9.5 (VCC)
- net GND: now also C63.2, C65.2, C66.2, Q5.3 (S), Q6.2 (S), R55.2, R58.2, R59.2, U9.3 (COM)
- net OUT_POS: now also K1.14, Q4.2 (D); no longer J2.1 (Pin_1), L1.2, R14.1
- net at D2.2 (A), R1.2, R2.1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: now also U9.2 (~{SD})
- new net: D15.2 (A), Q5.1 (G), R54.2, R58.1
- new net: C64.2, L1.2, Q4.3 (S), Q5.2 (D), R52.1, R57.2, U9.6 (VS)
- new net: D15.1 (K), R54.1, U9.4 (LO)
- new net: D18.2 (A), K1.A2, Q6.3 (D)
- new net: C66.1, R52.2
- new net: D17.1 (K), R53.1, U9.7 (HO)
- new net: C64.1, R56.2, U9.8 (VB)
- new net: Q6.1 (G), R59.1, R60.2
- new net: D17.2 (A), Q4.1 (G), R53.2, R57.1
- new net: D16.1 (K), R56.1
- new net DRV_IN2: R55.1, U9.1 (IN)
- new net OUT: J2.1 (Pin_1), K1.13, R14.1
- new net RELAY_EN: R60.1
Other:
- note added: ".tran 100n 40m"
- note added: "INPUT: external isolated 40-130 VDC bus (>=600 W)"
- note removed: ".tran 100n 10m"
- note removed: "INPUT: external isolated 110-130 VDC bus (>=600 W)"
- title: Power stage - 120V bus to 0-100V / 5A synchronous buck -> Power stage - 40-130V bus to 0-100V / 5A 4-switch buck-boost
- moved on the sheet: J2, R14, R2, R3

Commit message: jfha
Other:
- note added: ".options reltol=1e-3 itl4=100 gmin=1e-10"
- note added: ".tran 100n 30m"
- note removed: ".options reltol=1e-4"
- note removed: ".tran 100n 40m"
Changed lines of the file:
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@@
 		(rev "V1")
 	)
-	(text ".tran 100n 40m"
+	(text ".tran 100n 30m"
 		(exclude_from_sim no)
 		(at 27.94 161.29 0)
@@
 		)
 	)
-	(text ".options reltol=1e-4"
+	(text ".options reltol=1e-3 itl4=100 gmin=1e-10"
 		(exclude_from_sim no)
 		(at 27.94 168.91 0)
@@
 		)
 	)
-	(embedded_fonts no)
 )

Commit message: Jfhjh
Parts:
- removed V1: 60V, symbol Simulation_SPICE:VDC
Changed lines of the file:
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@@
 	)
 	(junction
-		(at 43.18 46.99)
-		(diameter 0)
-		(color 0 0 0 0)
-	)
-	(junction
 		(at 97.79 92.71)
 		(diameter 0)
@@
 	(wire
 		(pts
-			(xy 43.18 57.15) (xy 43.18 46.99)
-		)
-		(stroke
-			(width 0)
-			(type default)
-		)
-	)
-	(wire
-		(pts
 			(xy 167.64 111.76) (xy 175.26 111.76)
 		)
@@
 	)
 	(symbol
-		(lib_id "Simulation_SPICE:VDC")
-		(at 43.18 62.23 0)
-		(unit 1)
-		(body_style 1)
-		(exclude_from_sim yes)
-		(in_bom no)
-		(on_board no)
-		(in_pos_files no)
-		(dnp no)
-		(property "Reference" "V1"
-			(at 45.72 60.96 0)
-			(show_name no)
-			(do_not_autoplace no)
-			(effects
-				(font
-					(size 1.27 1.27)
-				)
-				(justify left)
-			)
-		)
-		(property "Value" "60V"
-			(at 45.72 63.5 0)
-			(show_name no)
-			(do_not_autoplace no)
-			(effects
-				(font
-					(size 1.27 1.27)
-				)
-				(justify left)
-			)
-		)
-		(property "Footprint" ""
-			(at 43.18 62.23 0)
-			(hide yes)
-			(show_name no)
-			(do_not_autoplace no)
-			(effects
-				(font
-					(size 1.27 1.27)
-				)
-			)
-		)
-		(property "Datasheet" "https://ngspice.sourceforge.io/docs/ngspice-html-manual/manual.xhtml#sec_Independent_Sources_for"
-			(at 43.18 62.23 0)
-			(hide yes)
-			(show_name no)
-			(do_not_autoplace no)
-			(effects
-				(font
-					(size 1.27 1.27)
-				)
-			)
-		)
-		(property "Description" "Voltage source, DC"
-			(at 43.18 62.23 0)
-			(hide yes)
-			(show_name no)
-			(do_not_autoplace no)
-			(effects
-				(font
-					(size 1.27 1.27)
-				)
-			)
-		)
-		(property "Sim.Device" "V"
-			(at 43.18 62.23 0)
-			(hide yes)
-			(show_name no)
-			(do_not_autoplace no)
-			(effects
-				(font
-					(size 1.27 1.27)
-				)
-			)
-		)
-		(property "Sim.Type" "DC"
-			(at 43.18 62.23 0)
-			(hide yes)
-			(show_name no)
-			(do_not_autoplace no)
-			(effects
-				(font
-					(size 1.27 1.27)
-				)
-			)
-		)
-		(property "Sim.Pins" "1=+ 2=-"
-			(at 43.18 62.23 0)
-			(hide yes)
-			(show_name no)
-			(do_not_autoplace no)
-			(effects
-				(font
-					(size 1.27 1.27)
-				)
-			)
-		)
-		(property "Sim.Params" "dc=60"
-			(at 43.18 62.23 0)
-			(hide yes)
-			(show_name no)
-			(do_not_autoplace no)
-			(effects
-				(font
-					(size 1.27 1.27)
-				)
-			)
-		)
-		(pin "1"
-		)
-		(pin "2"
-		)
-		(instances
-			(project "V1"
-				(path "/ac43abac-3a45-4cc0-8cc7-86391d0cc456/678b09c8-7c6d-4a51-9277-3bee220bddeb"
-					(reference "V1")
-					(unit 1)
-				)
-			)
-		)
-	)
-	(symbol
 		(lib_id "Device:C_Small")
 		(at 132.08 91.44 0)
@@
 	)
 	(symbol
-		(lib_id "power:GND")
-		(at 43.18 67.31 0)
-		(unit 1)
-		(body_style 1)
-		(exclude_from_sim no)
-		(in_bom no)
-		(on_board no)
-		(in_pos_files no)
-		(dnp no)
-		(property "Reference" "#PWR02"
-			(at 43.18 67.31 0)
-			(hide yes)
-			(show_name no)
-			(do_not_autoplace no)
-			(effects
-				(font
-					(size 1.27 1.27)
-				)
-			)
-		)
-		(property "Value" "GND"
-			(at 43.18 71.12 0)
-			(show_name no)
-			(do_not_autoplace no)
-			(effects
-				(font
-					(size 1.27 1.27)
-				)
-			)
-		)
-		(property "Footprint" ""
-			(at 43.18 67.31 0)
-			(hide yes)
-			(show_name no)
-			(do_not_autoplace no)
-			(effects
-				(font
-					(size 1.27 1.27)
-				)
-			)
-		)
-		(property "Datasheet" ""
-			(at 43.18 67.31 0)
-			(hide yes)
-			(show_name no)
-			(do_not_autoplace no)
-			(effects
-				(font
-					(size 1.27 1.27)
-				)
-			)
-		)
-		(property "Description" ""
-			(at 43.18 67.31 0)
-			(hide yes)
-			(show_name no)
-			(do_not_autoplace no)
-			(effects
-				(font
-					(size 1.27 1.27)
-				)
-			)
-		)
-		(pin "1"
-		)
-		(instances
-			(project "V1"
-				(path "/ac43abac-3a45-4cc0-8cc7-86391d0cc456/678b09c8-7c6d-4a51-9277-3bee220bddeb"
-					(reference "#PWR02")
-					(unit 1)
-				)
-			)
-		)
-	)
-	(symbol
 		(lib_id "Device:R_Small")
 		(at 165.1 111.76 90)
@@
 		)
 	)
+	(embedded_fonts no)
 )

Commit message: Jfhaha
Other:
- note added: ".tran 100n 9m"
- note removed: ".tran 100n 30m"
Changed lines of the file:
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@@
 		(rev "V1")
 	)
-	(text ".tran 100n 30m"
+	(text ".tran 100n 9m"
 		(exclude_from_sim no)
 		(at 27.94 161.29 0)
@@
 		)
 	)
-	(embedded_fonts no)
 )
